Commit message: Added meshes for wheels and base

File: carl_description/urdf/carl.urdf (robot description, URDF)
Before this commit: robot carl, 5 links, 4 joints
Links:
- removed link jaco
- removed link left_wheel
- removed link right_wheel
- removed link top_plate
- added link LeftWheel_link; collision mesh filename=package://carl_description/meshes/FullRobot - RMP_210-2 Sta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; visual mesh filename=package://carl_description/meshes/FullRobot - RMP_210-2 Sta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
- link base_link: geometry collision mesh filename=package://carl_description/meshes/FullRobot - RMP_210-1 RMP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; visual mesh filename=package://carl_description/meshes/FullRobot - RMP_210-1 RMP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
Joints:
- removed joint base_to_left_wheel
- removed joint base_to_plate
- removed joint base_to_right_wheel
- removed joint plate_to_jaco
- added joint BaseToLeftWheel: type continuous, parent base_link, child LeftWheel_link, origin xyz=0.32 0.02 0 rpy=0 0 0, axis 0 1 0

Commit message: Added more links

File: carl_description/urdf/carl.urdf (robot description, URDF)
Before this commit: robot carl, 2 links, 1 joints
Links:
- added link CameraLift_link; collision mesh filename=package://carl_description/meshes/FullRobot - tempHorizonta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; visual mesh filename=package://carl_description/meshes/FullRobot - tempHorizonta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
- added link CameraTilt_link; collision mesh filename=package://carl_description/meshes/FullRobot - tempPlate-1.S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; visual mesh filename=package://carl_description/meshes/FullRobot - tempPlate-1.S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
- added link Caster_link; collision mesh filename=package://carl_description/meshes/FullRobot - RMP_210-1 Cas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; visual mesh filename=package://carl_description/meshes/FullRobot - RMP_210-1 Cas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
- added link Hokuyo_link; collision mesh filename=package://carl_description/meshes/FullRobot - hokuyo-1.STL; visual mesh filename=package://carl_description/meshes/FullRobot - hokuyo-1.STL
- added link JacoMount_link; collision mesh filename=package://carl_description/meshes/FullRobot - SuperStructur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; visual mesh filename=package://carl_description/meshes/FullRobot - SuperStructur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
- added link RearLeftStrut_link; collision mesh filename=package://carl_description/meshes/FullRobot - SuperStructur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; visual mesh filename=package://carl_description/meshes/FullRobot - SuperStructur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
- added link RearRightStrut_link; collision mesh filename=package://carl_description/meshes/FullRobot - SuperStructur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; visual mesh filename=package://carl_description/meshes/FullRobot - SuperStructur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
- added link RightWheel_link; collision mesh filename=package://carl_description/meshes/FullRobot - RMP_210-1 Sta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; visual mesh filename=package://carl_description/meshes/FullRobot - RMP_210-1 Sta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
- added link TopPlate_link; collision mesh filename=package://carl_description/meshes/FullRobot - SuperStructur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; visual mesh filename=package://carl_description/meshes/FullRobot - SuperStructur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
- link LeftWheel_link: geometry collision mesh filename=package://carl_description/meshes/FullRobot - RMP_210-1 Sta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; visual mesh filename=package://carl_description/meshes/FullRobot - RMP_210-1 Sta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
Joints:
- added joint BaseToCaster: type fixed, parent base_link, child Caster_link, origin xyz=0 0 0 rpy=0 0 0
- added joint BaseToRearLeftStrut: type fixed, parent base_link, child RearLeftStrut_link, origin xyz=0.20 0.19 0.22 rpy=0 0 0
- added joint BaseToRearRightStrut: type fixed, parent base_link, child RearRightStrut_link, origin xyz=-0.20 0.19 0.22 rpy=0 0 0
- added joint BaseToRightWheel: type continuous, parent base_link, child RightWheel_link, origin xyz=-0.32 0.02 0 rpy=0 0 0, axis 0 -1 0
- added joint CameraLiftToCameraTilt: type fixed, parent CameraLift_link, child CameraTilt_link, origin xyz=0 -0.07 -0.02 rpy=0.707 0 0
- added joint CasterToHokuyo: type fixed, parent Caster_link, child Hokuyo_link, origin xyz=0 -0.36 0 rpy=0 0 0
- added joint RearLeftStrutToCameraLift: type fixed, parent RearRightStrut_link, child CameraLift_link, origin xyz=0.20 0.01 1.17 rpy=0 0 0
- added joint RearLeftStrutToTopPlate: type fixed, parent RearRightStrut_link, child TopPlate_link, origin xyz=0.20 -0.30 0.30 rpy=0 0 0
- added joint TopPlateToJacoMount: type fixed, parent TopPlate_link, child JacoMount_link, origin xyz=0 -0.13 -0.22 rpy=0 0 0

Commit message: Fixed rotation axis for camera tilt link

File: carl_description/urdf/carl.urdf (robot description, URDF)
Before this commit: robot carl, 11 links, 10 joints
Links:
- removed link CameraTilt_link
- added link CameraTiltBracket_link; collision mesh filename=package://carl_description/meshes/FullRobot - tempSwivelBas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; visual mesh filename=package://carl_description/meshes/FullRobot - tempSwivelBas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
- added link CameraTiltPlate_link; collision mesh filename=package://carl_description/meshes/FullRobot - tempPlate-1.S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; visual mesh filename=package://carl_description/meshes/FullRobot - tempPlate-1.S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
Joints:
- removed joint CameraLiftToCameraTilt
- added joint CameraLiftBracketToCameraTiltPlate: type fixed, parent CameraTiltBracket_link, child CameraTiltPlate_link, origin xyz=0.10 -0.11 0.0 rpy=0 0 0
- added joint CameraLiftToCameraTiltBracket: type continuous, parent CameraLift_link, child CameraTiltBracket_link, origin xyz=-0.10 -0.03  0 rpy=0 0 0, axis 1 0 0
- joint BaseToLeftWheel: axis 0 1 0 -> 1 0 0
- joint BaseToRightWheel: axis 0 -1 0 -> -1 0 0

Commit message: Fixed origins for visualization.

File: carl_description/urdf/carl.urdf (robot description, URDF)
Before this commit: robot carl, 12 links, 11 joints
Links:
- link CameraTiltBracket_link: geometry collision mesh filename=package://carl_description/meshes/FullRobot - tempSwivelMou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

Commit message: Fixed collision origins

File: carl_description/urdf/carl.urdf (robot description, URDF)
Before this commit: robot carl, 12 links, 11 joints
Joints:
- joint TopPlateToJacoMount: origin xyz=0 -0.13 -0.22 rpy=0 0 0 -> xyz=0 -0.13 -0.216 rpy=0 0 0

Commit message: Fixed origin of STLs and reoriented axis of urdf

File: carl_description/urdf/carl.urdf (robot description, URDF)
Before this commit: robot carl, 12 links, 11 joints
Joints:
- joint BaseToLeftWheel: axis 1 0 0 -> 0 0 1; origin xyz=0.32 0.02 0 rpy=0 0 0 -> xyz=0.02 0.32 0 rpy=-1.5708 0 0
- joint BaseToRearLeftStrut: origin xyz=0.20 0.19 0.22 rpy=0 0 0 -> xyz=-0.19 0.20 0.22 rpy=0 0 0
- joint BaseToRearRightStrut: origin xyz=-0.20 0.19 0.22 rpy=0 0 0 -> xyz=-0.19 -0.20 0.22 rpy=0 0 0
- joint BaseToRightWheel: axis -1 0 0 -> 0 0 1; origin xyz=-0.32 0.02 0 rpy=0 0 0 -> xyz=0.02 -0.32 0 rpy=1.5708 0 0
- joint CameraLiftBracketToCameraTiltPlate: origin xyz=0.10 -0.11 0.0 rpy=0 0 0 -> xyz=0.11 0 -0.10 rpy=0 0 0
- joint CameraLiftToCameraTiltBracket: axis 1 0 0 -> 0 0 1; origin xyz=-0.10 -0.03  0 rpy=0 0 0 -> xyz=0.03 -0.10 0 rpy=1.5708 0 0
- joint CasterToHokuyo: origin xyz=0 -0.36 0 rpy=0 0 0 -> xyz=0.36 0 0 rpy=0 0 0
- joint RearLeftStrutToCameraLift: origin xyz=0.20 0.01 1.17 rpy=0 0 0 -> xyz=0.01 0.20 1.17 rpy=0 0 0
- joint RearLeftStrutToTopPlate: origin xyz=0.20 -0.30 0.30 rpy=0 0 0 -> xyz=0.30 0.20 0.30 rpy=0 0 0
- joint TopPlateToJacoMount: origin xyz=0 -0.13 -0.216 rpy=0 0 0 -> xyz=0.216 0 -0.13 rpy=0 0 0

Commit message: Removed spaces from mesh file names

File: carl_description/urdf/carl.urdf (robot description, URDF)
Before this commit: robot carl, 12 links, 11 joints
Links:
- link CameraLift_link: geometry collision mesh filename=package://carl_description/meshes/FullRobot_-_tempHorizonta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; visual mesh filename=package://carl_description/meshes/FullRobot_-_tempHorizonta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
- link CameraTiltBracket_link: geometry collision mesh filename=package://carl_description/meshes/FullRobot_-_tempSwivelMou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
- link CameraTiltPlate_link: geometry collision mesh filename=package://carl_description/meshes/FullRobot_-_tempPlate-1.S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; visual mesh filename=package://carl_description/meshes/FullRobot_-_tempPlate-1.S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
- link Caster_link: geometry collision mesh filename=package://carl_description/meshes/FullRobot_-_RMP_210-1_Cas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; visual mesh filename=package://carl_description/meshes/FullRobot_-_RMP_210-1_Cas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
- link Hokuyo_link: geometry collision mesh filename=package://carl_description/meshes/FullRobot_-_hokuyo-1.STL; visual mesh filename=package://carl_description/meshes/FullRobot_-_hokuyo-1.STL
- link JacoMount_link: geometry collision mesh filename=package://carl_description/meshes/FullRobot_-_SuperStructur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; visual mesh filename=package://carl_description/meshes/FullRobot_-_SuperStructur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
- link LeftWheel_link: geometry collision mesh filename=package://carl_description/meshes/FullRobot_-_RMP_210-1_Sta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; visual mesh filename=package://carl_description/meshes/FullRobot_-_RMP_210-1_Sta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
- link RearLeftStrut_link: geometry collision mesh filename=package://carl_description/meshes/FullRobot_-_SuperStructur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; visual mesh filename=package://carl_description/meshes/FullRobot_-_SuperStructur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
- link RearRightStrut_link: geometry collision mesh filename=package://carl_description/meshes/FullRobot_-_SuperStructur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; visual mesh filename=package://carl_description/meshes/FullRobot_-_SuperStructur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
- link RightWheel_link: geometry collision mesh filename=package://carl_description/meshes/FullRobot_-_RMP_210-1_Sta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; visual mesh filename=package://carl_description/meshes/FullRobot_-_RMP_210-1_Sta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
- link TopPlate_link: geometry collision mesh filename=package://carl_description/meshes/FullRobot_-_SuperStructur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; visual mesh filename=package://carl_description/meshes/FullRobot_-_SuperStructur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
- link base_link: geometry collision mesh filename=package://carl_description/meshes/FullRobot_-_RMP_210-1_RMP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; visual mesh filename=package://carl_description/meshes/FullRobot_-_RMP_210-1_RMP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

Commit message: Switched to xacro format. Added jaco arm to model.

File: carl_description/urdf/carl.urdf (robot description, URDF)
Before this commit: robot carl, 12 links, 11 joints
Links:
- added link jaco_link_1; collision mesh filename=package://jaco_model/meshes/jaco_link_1.dae; visual mesh filename=package://jaco_model/meshes/jaco_link_1.dae
- added link jaco_link_2; collision mesh filename=package://jaco_model/meshes/jaco_link_2.dae; visual mesh filename=package://jaco_model/meshes/jaco_link_2.dae
- added link jaco_link_3; collision mesh filename=package://jaco_model/meshes/jaco_link_3.dae; visual mesh filename=package://jaco_model/meshes/jaco_link_3.dae
- added link jaco_link_4; collision mesh filename=package://jaco_model/meshes/jaco_link_4.dae; visual mesh filename=package://jaco_model/meshes/jaco_link_4.dae
- added link jaco_link_5; collision mesh filename=package://jaco_model/meshes/jaco_link_5.dae; visual mesh filename=package://jaco_model/meshes/jaco_link_5.dae
- added link jaco_link_base; collision mesh filename=package://jaco_model/meshes/jaco_link_base.dae; visual mesh filename=package://jaco_model/meshes/jaco_link_base.dae
- added link jaco_link_finger_1; collision mesh filename=package://jaco_model/meshes/jaco_link_finger_1.dae; visual mesh filename=package://jaco_model/meshes/jaco_link_finger_1.dae
- added link jaco_link_finger_2; collision mesh filename=package://jaco_model/meshes/jaco_link_finger_2.dae; visual mesh filename=package://jaco_model/meshes/jaco_link_finger_2.dae
- added link jaco_link_finger_3; collision mesh filename=package://jaco_model/meshes/jaco_link_finger_3.dae; visual mesh filename=package://jaco_model/meshes/jaco_link_finger_3.dae
- added link jaco_link_hand; collision mesh filename=package://jaco_model/meshes/jaco_link_hand.dae; visual mesh filename=package://jaco_model/meshes/jaco_link_hand.dae
- link CameraTiltBracket_link: geometry 
Joints:
- added joint jaco_joint_1: type continuous, parent jaco_link_base, child jaco_link_1, origin xyz=0 0 0.1535 rpy=3.14159265359 0 0, axis 0 0 1
- added joint jaco_joint_2: type continuous, parent jaco_link_1, child jaco_link_2, origin xyz=0 0 -0.1185 rpy=-1.57079632679 -1.57079632679 0, axis 0 0 1
- added joint jaco_joint_3: type continuous, parent jaco_link_2, child jaco_link_3, origin xyz=0.41 0 0 rpy=3.14159265359 0 3.14159265359, axis 0 0 1
- added joint jaco_joint_4: type continuous, parent jaco_link_3, child jaco_link_4, origin xyz=0.207 0 -0.01125 rpy=0 -1.57079632679 0, axis 0 0 1
- added joint jaco_joint_5: type continuous, parent jaco_link_4, child jaco_link_5, origin xyz=0.0343 0 -0.06588 rpy=0 0.959931088597 3.14159265359, axis 0 0 1
- added joint jaco_joint_6: type continuous, parent jaco_link_5, child jaco_link_hand, origin xyz=0.0343 0 -0.06588 rpy=0 0.959931088597 3.14159265359, axis 0 0 1
- added joint jaco_joint_base: type fixed, parent JacoMount_link, child jaco_link_base, origin xyz=0 0 0 rpy=0 0 0, axis 0 0 0
- added joint jaco_joint_finger_1: type revolute, parent jaco_link_hand, child jaco_link_finger_1, origin xyz=-0.03978 0 -0.10071 rpy=-1.7983 1.117 3.1416, axis 0 0 1, limit lower=0 upper=0.698131700798 effort=30 velocity=5
- added joint jaco_joint_finger_2: type revolute, parent jaco_link_hand, child jaco_link_finger_2, origin xyz=0.03569 -0.0216 -0.10071 rpy=-1.6222 1.117 -0.23615, axis 0 0 1, limit lower=0 upper=0.698131700798 effort=30 velocity=5
- added joint jaco_joint_finger_3: type revolute, parent jaco_link_hand, child jaco_link_finger_3, origin xyz=0.03569 0.0216 -0.10071 rpy=-1.5161 1.1459 0.23978, axis 0 0 1, limit lower=0 upper=0.698131700798 effort=30 velocity=5
- joint BaseToRearLeftStrut: origin xyz=-0.19 0.20 0.22 rpy=0 0 0 -> xyz=-0.222 0.20 0.194 rpy=0 0 0
- joint BaseToRearRightStrut: origin xyz=-0.19 -0.20 0.22 rpy=0 0 0 -> xyz=-0.222 -0.20 0.194 rpy=0 0 0

Commit message: Simplifications to collision model

File: carl_description/urdf/carl.urdf (robot description, URDF)
Before this commit: robot carl, 22 links, 21 joints
Links:
- link CameraLift_link: geometry visual mesh filename=package://carl_description/meshes/FullRobot_-_tempHorizonta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
- link CameraTiltPlate_link: geometry visual mesh filename=package://carl_description/meshes/FullRobot_-_tempPlate-1.S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
- link Caster_link: geometry visual mesh filename=package://carl_description/meshes/FullRobot_-_RMP_210-1_Cas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
- link Hokuyo_link: geometry visual mesh filename=package://carl_description/meshes/FullRobot_-_hokuyo-1.STL
- link JacoMount_link: geometry visual mesh filename=package://carl_description/meshes/FullRobot_-_SuperStructur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
- link LeftWheel_link: geometry collision cylinder length=0.090 radius=0.25; visual mesh filename=package://carl_description/meshes/FullRobot_-_RMP_210-1_Sta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
- link RearLeftStrut_link: geometry collision box size=0.025 0.051 1.055; visual mesh filename=package://carl_description/meshes/FullRobot_-_SuperStructur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
- link RearRightStrut_link: geometry collision box size=0.025 0.051 1.055; visual mesh filename=package://carl_description/meshes/FullRobot_-_SuperStructur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
- link RightWheel_link: geometry collision cylinder length=0.090 radius=0.25; visual mesh filename=package://carl_description/meshes/FullRobot_-_RMP_210-1_Sta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
- link TopPlate_link: geometry collision box size=0.465 0.584 0.6; visual mesh filename=package://carl_description/meshes/FullRobot_-_SuperStructur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
- link base_link: geometry visual mesh filename=package://carl_description/meshes/FullRobot_-_RMP_210-1_RMP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

File: carl_description/urdf/carl.xacro (robot description, xacro)
@@ -1,5 +1,5 @@
 <?xml version="1.0"?>
 <robot xmlns:xacro="http://www.ros.org/wiki/xacro" name="carl">
-<xacro:include filename="$(find jaco_model)/urdf/jaco_arm.xacro" />
+  <xacro:include filename="$(find jaco_model)/urdf/jaco_arm.xacro" />
   <link name="base_link">
    <visual>
@@ -9,10 +9,4 @@
       </geometry>
     </visual>
-    <collision>
-      <origin xyz="0 0 0" rpy="0 0 0"/>
-      <geometry>
-        <mesh filename="package://carl_description/meshes/FullRobot_-_RMP_210-1_RMP_Powerbase-1.STL"/>
-      </geometry>
-    </collision>
   </link>
   <link name="LeftWheel_link">
@@ -24,7 +18,7 @@
     </visual>
     <collision>
-      <origin xyz="0 0.02 -0.32" rpy="1.5708 0 0" />
+      <origin xyz="0 0 -0.045" rpy="0 0 0" />
       <geometry>
-        <mesh filename="package://carl_description/meshes/FullRobot_-_RMP_210-1_StandardWheel-2.STL"/>
+        <cylinder radius="0.25" length="0.090" />
       </geometry>
     </collision>
@@ -38,7 +32,7 @@
     </visual>
     <collision>
-      <origin xyz="0 -0.02 -0.32" rpy="-1.5708 0 0" />
+      <origin xyz="0 0 -0.045" rpy="0 0 0" />
       <geometry>
-        <mesh filename="package://carl_description/meshes/FullRobot_-_RMP_210-1_StandardWheel-1.STL"/>
+        <cylinder radius="0.25" length="0.090" />
       </geometry>
     </collision>
@@ -51,10 +45,4 @@
       </geometry>
     </visual>
-    <collision>
-      <origin xyz="0 0 0" rpy="0 0 0"/>
-      <geometry>
-        <mesh filename="package://carl_description/meshes/FullRobot_-_RMP_210-1_CasterAssembly-1.STL"/>
-      </geometry>
-    </collision>
   </link>
   <link name="RearLeftStrut_link">
@@ -66,8 +54,8 @@
     </visual>
     <collision>
-      <origin xyz="0.222 0.20 -0.194" rpy="0 0 0" />
+      <origin xyz="0 -0.40 0.24" rpy="0 0 0" />
       <geometry>
-        <mesh filename="package://carl_description/meshes/FullRobot_-_SuperStructure-1_RearVerticalStrut-1.STL"/>
-      </geometry>
+        <box size="0.025 0.051 1.055" />
+       </geometry>
     </collision>
   </link>
@@ -80,7 +68,7 @@
     </visual>
     <collision>
-      <origin xyz="0.222 0.20 -0.194" rpy="0 0 0" />
+      <origin xyz="0 0.40 0.24" rpy="0 0 0" />
       <geometry>
-        <mesh filename="package://carl_description/meshes/FullRobot_-_SuperStructure-1_RearVerticalStrut-2.STL"/>
+        <box size="0.025 0.051 1.055" />
       </geometry>
     </collision>
@@ -94,7 +82,7 @@
     </visual>
     <collision>
-      <origin xyz="-.08 0 -0.495" rpy="0 0 0" />
+      <origin xyz="-.055 0 -0.295" rpy="0 0 0" />
       <geometry>
-        <mesh filename="package://carl_description/meshes/FullRobot_-_SuperStructure-1_Table_Plate-1.STL"/>
+        <box size="0.465 0.584 0.6" />
       </geometry>
     </collision>
@@ -107,24 +95,7 @@
       </geometry>
     </visual>
-    <collision>
-      <origin xyz="0.22 0 -1.36" rpy="0 0 0" />
-      <geometry>
-        <mesh filename="package://carl_description/meshes/FullRobot_-_tempHorizontal-1.STL"/>
-      </geometry>
-    </collision>
   </link>
-    <link name="CameraTiltBracket_link">
-    <!--<visual>
-      <origin xyz="0 0 0" rpy="0 0 0"/>
-      <geometry>
-        <mesh filename="package://carl_description/meshes/FullRobot_-_tempSwivelMount-1.STL" />
-      </geometry>
-    </visual>
-    <collision>
-      <origin xyz="0 0 0" rpy="0 0 0"/>
-      <geometry>
-        <mesh filename="package://carl_description/meshes/FullRobot_-_tempSwivelMount-1.STL"/>
-      </geometry>
-    </collision>-->
+  <link name="CameraTiltBracket_link">
+	<!--exists to move center of rotation for camera mount-->
   </link>
   <link name="CameraTiltPlate_link">
@@ -135,10 +106,4 @@
       </geometry>
     </visual>
-    <collision>
-      <origin xyz="-1.24 .54 0 " rpy="-1.5708 0 -2.1" />
-      <geometry>
-        <mesh filename="package://carl_description/meshes/FullRobot_-_tempPlate-1.STL"/>
-      </geometry>
-    </collision>
   </link>
   <link name="JacoMount_link">
@@ -149,10 +114,4 @@
       </geometry>
     </visual>
-    <collision>
-      <origin xyz="-0.3 0 -0.36" rpy="0 0 0" />
-      <geometry>
-        <mesh filename="package://carl_description/meshes/FullRobot_-_SuperStructure-1_ArmMountHoriz-1.STL"/>
-      </geometry>
-    </collision>
   </link>
   <link name="Hokuyo_link">
@@ -163,10 +122,4 @@
       </geometry>
     </visual>
-    <collision>
-      <origin xyz="-0.36 0 0" rpy="0 0 0" />
-      <geometry>
-        <mesh filename="package://carl_description/meshes/FullRobot_-_hokuyo-1.STL"/>
-      </geometry>
-    </collision>
   </link>
   <joint name="BaseToLeftWheel" type="continuous">

Commit message: Added side walls

File: carl_description/urdf/carl.urdf (robot description, URDF)
Before this commit: robot carl, 22 links, 21 joints
Links:
- added link LeftSideWall_link; visual mesh filename=package://carl_description/meshes/FullRobot_-_sideWall-1.STL
- added link RightSideWall_link; visual mesh filename=package://carl_description/meshes/FullRobot_-_sideWall-1.STL
Joints:
- added joint RearLeftStrutToLeftSideWall: type fixed, parent RearLeftStrut_link, child LeftSideWall_link, origin xyz=0.229 0.025 0.078 rpy=0 0 0
- added joint RearRightStrutToRightSideWall: type fixed, parent RearRightStrut_link, child RightSideWall_link, origin xyz=0.229 -0.025 0.078 rpy=0 0 0

File: carl_description/urdf/carl.xacro (robot description, xacro)
@@ -123,4 +123,20 @@
     </visual>
   </link>
+   <link name="LeftSideWall_link">
+    <visual>
+      <origin xyz="0 -.225 -.27" rpy="0 0 0" />
+      <geometry>
+        <mesh filename="package://carl_description/meshes/FullRobot_-_sideWall-1.STL" />
+      </geometry>
+    </visual>
+  </link>
+   <link name="RightSideWall_link">
+    <visual>
+      <origin xyz="0 -.225 -.27" rpy="0 0 0" />
+      <geometry>
+        <mesh filename="package://carl_description/meshes/FullRobot_-_sideWall-1.STL" />
+      </geometry>
+    </visual>
+  </link>
   <joint name="BaseToLeftWheel" type="continuous">
     <parent link="base_link"/>
@@ -181,4 +197,14 @@
     <origin xyz="0.36 0 0" rpy="0 0 0" />
   </joint>
+  <joint name="RearLeftStrutToLeftSideWall" type="fixed">
+    <parent link="RearLeftStrut_link"/>
+    <child link="LeftSideWall_link"/>
+    <origin xyz="0.229 0.025 0.078" rpy="0 0 0" />
+  </joint>
+  <joint name="RearRightStrutToRightSideWall" type="fixed">
+    <parent link="RearRightStrut_link"/>
+    <child link="RightSideWall_link"/>
+    <origin xyz="0.229 -0.025 0.078" rpy="0 0 0" />
+  </joint>
   <xacro:jaco_arm  parent="JacoMount_link"/>
 </robot>
