Commit message: Added front plate

File: carl_description/urdf/carl.urdf (robot description, URDF)
Before this commit: robot carl, 24 links, 23 joints
Links:
- added link FrontCover_link; collision mesh filename=package://carl_description/meshes/FrontCoverCollision.STL; visual mesh filename=package://carl_description/meshes/FullRobot_-_FrontCover-1.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
- link TopPlate_link: geometry collision box size=0.483 0.584 0.6; visual mesh filename=package://carl_description/meshes/FullRobot_-_SuperStructur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
Joints:
- added joint BaseToFrontCover: type fixed, parent base_link, child FrontCover_link, origin xyz=0 0 0.012 rpy=0 0 0

File: carl_description/urdf/carl.xacro (robot description, xacro)
@@ -82,7 +82,9 @@
     </visual>
     <collision>
-      <origin xyz="-.055 0 -0.295" rpy="0 0 0" />
-      <geometry>
-        <box size="0.465 0.584 0.6" />
+      <!--<origin xyz="-.055 0 -0.295" rpy="0 0 0" />-->
+      <origin xyz="-.068 0 -0.295" rpy="0 0 0" />
+      <geometry>
+        <!--<box size="0.465 0.584 0.6" />-->
+        <box size="0.483 0.584 0.6" />
       </geometry>
     </collision>
@@ -138,4 +140,18 @@
       </geometry>
     </visual>
+  </link>
+  <link name="FrontCover_link">
+    <visual>
+      <origin xyz="0 0 -.012" rpy="0 0 0" />
+      <geometry>
+        <mesh filename="package://carl_description/meshes/FullRobot_-_FrontCover-1.STL" />
+      </geometry>
+    </visual>
+    <collision>
+      <origin xyz="0 0 -.012" rpy="0 0 0" />
+      <geometry>
+        <mesh filename="package://carl_description/meshes/FrontCoverCollision.STL" />
+      </geometry>
+    </collision>
   </link>
   <joint name="BaseToLeftWheel" type="continuous">
@@ -207,4 +223,9 @@
     <origin xyz="0.229 -0.025 0.078" rpy="0 0 0" />
   </joint>
+  <joint name="BaseToFrontCover" type="fixed">
+    <parent link="base_link"/>
+    <child link="FrontCover_link"/>
+    <origin xyz="0 0 0.012" rpy="0 0 0" />
+  </joint>
   <xacro:jaco_arm  parent="JacoMount_link"/>
 </robot>

Commit message: Added collision for caster

File: carl_description/urdf/carl.urdf (robot description, URDF)
Before this commit: robot carl, 25 links, 24 joints
Links:
- link Caster_link: geometry collision cylinder length=0.213 radius=0.116; visual mesh filename=package://carl_description/meshes/FullRobot_-_RMP_210-1_Cas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

File: carl_description/urdf/carl.xacro (robot description, xacro)
@@ -45,4 +45,10 @@
       </geometry>
     </visual>
+    <collision>
+      <origin xyz="0.31 0 -0.12" rpy="0 0 0" />
+      <geometry>
+        <cylinder radius="0.116" length="0.213" />
+       </geometry>
+    </collision>
   </link>
   <link name="RearLeftStrut_link">

Commit message: Added back cover

File: carl_description/urdf/carl.urdf (robot description, URDF)
Before this commit: robot carl, 25 links, 24 joints
Links:
- added link BackCover_link; visual box size=0.005 0.45 0.6
Joints:
- added joint BaseToBackCover: type fixed, parent base_link, child BackCover_link, origin xyz=0 0 -0.012 rpy=0 0 0

File: carl_description/urdf/carl.xacro (robot description, xacro)
@@ -88,8 +88,6 @@
     </visual>
     <collision>
-      <!--<origin xyz="-.055 0 -0.295" rpy="0 0 0" />-->
       <origin xyz="-.068 0 -0.295" rpy="0 0 0" />
       <geometry>
-        <!--<box size="0.465 0.584 0.6" />-->
         <box size="0.483 0.584 0.6" />
       </geometry>
@@ -160,4 +158,12 @@
       </geometry>
     </collision>
+  </link>
+    <link name="BackCover_link">
+    <visual>
+      <origin xyz="-.237 0 .208" rpy="0 0 0" />
+      <geometry>
+      	<box size="0.005 0.45 0.6" />
+      </geometry>
+    </visual>
   </link>
   <joint name="BaseToLeftWheel" type="continuous">
@@ -234,4 +240,9 @@
     <origin xyz="0 0 0.012" rpy="0 0 0" />
   </joint>
+  <joint name="BaseToBackCover" type="fixed">
+    <parent link="base_link"/>
+    <child link="BackCover_link"/>
+    <origin xyz="0 0 -0.012" rpy="0 0 0" />
+  </joint>
   <xacro:jaco_arm  parent="JacoMount_link"/>
 </robot>

Commit message: Replaced STLs with Collada files.

File: carl_description/urdf/carl.urdf (robot description, URDF)
Before this commit: robot carl, 26 links, 25 joints
Links:
- added link CasterPlate_link; collision cylinder length=0.213 radius=0.116; visual mesh filename=package://carl_description/meshes/casterPlate.dae
- link BackCover_link: geometry visual mesh filename=package://carl_description/meshes/BackCover.dae
- link CameraLift_link: geometry visual mesh filename=package://carl_description/meshes/CameraLift.dae
- link CameraTiltPlate_link: geometry visual mesh filename=package://carl_description/meshes/CameraPlate.dae
- link Caster_link: geometry collision cylinder length=0.213 radius=0.116; visual mesh filename=package://carl_description/meshes/caster.dae
- link FrontCover_link: geometry collision mesh filename=package://carl_description/meshes/FrontCoverCollision.STL; visual mesh filename=package://carl_description/meshes/FrontCover.dae
- link Hokuyo_link: geometry visual mesh filename=package://carl_description/meshes/Hokuyo.dae
- link JacoMount_link: geometry visual mesh filename=package://carl_description/meshes/JacoMount.dae
- link LeftSideWall_link: geometry visual mesh filename=package://carl_description/meshes/SideWall.dae
- link LeftWheel_link: geometry collision cylinder length=0.090 radius=0.25; visual mesh filename=package://carl_description/meshes/Wheel.dae
- link RearLeftStrut_link: geometry collision box size=0.025 0.051 1.055; visual mesh filename=package://carl_description/meshes/RearStrut.dae
- link RearRightStrut_link: geometry collision box size=0.025 0.051 1.055; visual mesh filename=package://carl_description/meshes/RearStrut.dae
- link RightSideWall_link: geometry visual mesh filename=package://carl_description/meshes/SideWall.dae
- link RightWheel_link: geometry collision cylinder length=0.090 radius=0.25; visual mesh filename=package://carl_description/meshes/Wheel.dae
- link TopPlate_link: geometry collision box size=0.483 0.584 0.6; visual mesh filename=package://carl_description/meshes/TablePlate.dae
- link base_link: geometry visual mesh filename=package://carl_description/meshes/Base.dae
Joints:
- removed joint BaseToCaster
- added joint BaseToCasterPlate: type fixed, parent base_link, child CasterPlate_link, origin xyz=0.2883 0 0 rpy=0 0 0
- added joint CasterPlateToCaster: type fixed, parent CasterPlate_link, child Caster_link, origin xyz=0.0267 0 -0.024 rpy=0 0 0
- joint BaseToFrontCover: origin xyz=0 0 0.012 rpy=0 0 0 -> xyz=.247 0 0.242 rpy=0 0 0
- joint BaseToRearLeftStrut: origin xyz=-0.222 0.20 0.194 rpy=0 0 0 -> xyz=-0.222 0.200 -0.102 rpy=0 0 0
- joint BaseToRearRightStrut: origin xyz=-0.222 -0.20 0.194 rpy=0 0 0 -> xyz=-0.222 -0.200 -0.102 rpy=0 0 0
- joint CasterToHokuyo: origin xyz=0.36 0 0 rpy=0 0 0 -> xyz=0.07 0 0.035 rpy=0 0 0; parent Caster_link -> CasterPlate_link
- joint RearLeftStrutToCameraLift: origin xyz=0.01 0.20 1.17 rpy=0 0 0 -> xyz=0.01 0.20 1.461 rpy=0 0 0
- joint RearLeftStrutToTopPlate: origin xyz=0.30 0.20 0.30 rpy=0 0 0 -> xyz=0.516 0.20 0.598 rpy=0 0 0
- joint TopPlateToJacoMount: origin xyz=0.216 0 -0.13 rpy=0 0 0 -> xyz=0 0 -0.13 rpy=0 0 0

File: carl_description/urdf/carl.xacro (robot description, xacro)
@@ -1,3 +1,6 @@
 <?xml version="1.0"?>
+<!--
+If you are reading this, it means I forgot to update the collision model. Remind me.
+-->
 <robot xmlns:xacro="http://www.ros.org/wiki/xacro" name="carl">
   <xacro:include filename="$(find jaco_model)/urdf/jaco_arm.xacro" />
@@ -6,5 +9,5 @@
       <origin xyz="0 0 0" rpy="0 0 0"/>
       <geometry>
-        <mesh filename="package://carl_description/meshes/FullRobot_-_RMP_210-1_RMP_Powerbase-1.STL" />
+        <mesh filename="package://carl_description/meshes/Base.dae" />
       </geometry>
     </visual>
@@ -12,11 +15,11 @@
   <link name="LeftWheel_link">
     <visual>
-      <origin xyz="0 0.02 -0.32" rpy="1.5708 0 0" />
-      <geometry>
-        <mesh filename="package://carl_description/meshes/FullRobot_-_RMP_210-1_StandardWheel-2.STL" />
-      </geometry>
-    </visual>
-    <collision>
-      <origin xyz="0 0 -0.045" rpy="0 0 0" />
+      <origin xyz="0 0 0" rpy="0 0 0" />
+      <geometry>
+        <mesh filename="package://carl_description/meshes/Wheel.dae" />
+      </geometry>
+    </visual>
+    <collision>
+      <origin xyz="0 0 0" rpy="0 0 0" />
       <geometry>
         <cylinder radius="0.25" length="0.090" />
@@ -26,11 +29,11 @@
   <link name="RightWheel_link">
     <visual>
-     <origin xyz="0 -0.02 -0.32" rpy="-1.5708 0 0" />
-      <geometry>
-        <mesh filename="package://carl_description/meshes/FullRobot_-_RMP_210-1_StandardWheel-1.STL" />
-      </geometry>
-    </visual>
-    <collision>
-      <origin xyz="0 0 -0.045" rpy="0 0 0" />
+      <origin xyz="0 0 0" rpy="0 0 0" />
+      <geometry>
+        <mesh filename="package://carl_description/meshes/Wheel.dae" />
+      </geometry>
+    </visual>
+    <collision>
+      <origin xyz="0 0 0" rpy="0 0 0" />
       <geometry>
         <cylinder radius="0.25" length="0.090" />
@@ -38,9 +41,9 @@
     </collision>
   </link>
-  <link name="Caster_link">
-    <visual>
-      <origin xyz="0 0 0" rpy="0 0 0"/>
-      <geometry>
-        <mesh filename="package://carl_description/meshes/FullRobot_-_RMP_210-1_CasterAssembly-1.STL" />
+  <link name="CasterPlate_link">
+    <visual>
+      <origin xyz="0 0 0" rpy="0 0 1.5708"/>
+      <geometry>
+        <mesh filename="package://carl_description/meshes/casterPlate.dae" />
       </geometry>
     </visual>
@@ -52,9 +55,23 @@
     </collision>
   </link>
+    <link name="Caster_link">
+    <visual>
+      <origin xyz="0 0 0" rpy="0 0 1.5708"/>
+      <geometry>
+        <mesh filename="package://carl_description/meshes/caster.dae" />
+      </geometry>
+    </visual>
+    <collision>
+      <origin xyz="0.31 0 -0.12" rpy="0 0 0" />
+      <geometry>
+        <cylinder radius="0.116" length="0.213" />
+       </geometry>
+    </collision>
+  </link>
   <link name="RearLeftStrut_link">
     <visual>
-      <origin xyz="0.222 -0.20 -0.194" rpy="0 0 0" />
-      <geometry>
-        <mesh filename="package://carl_description/meshes/FullRobot_-_SuperStructure-1_RearVerticalStrut-1.STL" />
+      <origin xyz="0 0 0" rpy="0 0 -1.5708" />
+      <geometry>
+        <mesh filename="package://carl_description/meshes/RearStrut.dae" />
       </geometry>
     </visual>
@@ -68,7 +85,7 @@
   <link name="RearRightStrut_link">
     <visual>
-      <origin xyz="0.222 0.20 -0.194" rpy="0 0 0" />
-      <geometry>
-        <mesh filename="package://carl_description/meshes/FullRobot_-_SuperStructure-1_RearVerticalStrut-2.STL" />
+      <origin xyz="0 0 0" rpy="0 0 -1.5708" />
+      <geometry>
+        <mesh filename="package://carl_description/meshes/RearStrut.dae" />
       </geometry>
     </visual>
@@ -82,7 +99,7 @@
   <link name="TopPlate_link">
     <visual>
-      <origin xyz="-.08 0 -0.495" rpy="0 0 0" />
-      <geometry>
-        <mesh filename="package://carl_description/meshes/FullRobot_-_SuperStructure-1_Table_Plate-1.STL" />
+      <origin xyz="0 0 0" rpy="0 0 -1.5708" />
+      <geometry>
+        <mesh filename="package://carl_description/meshes/TablePlate.dae" />
       </geometry>
     </visual>
@@ -96,7 +113,7 @@
   <link name="CameraLift_link">
     <visual>
-      <origin xyz="0.22 0 -1.36" rpy="0 0 0" />
-      <geometry>
-        <mesh filename="package://carl_description/meshes/FullRobot_-_tempHorizontal-1.STL" />
+      <origin xyz="0 0 0" rpy="0 0 1.5708" />
+      <geometry>
+        <mesh filename="package://carl_description/meshes/CameraLift.dae" />
       </geometry>
     </visual>
@@ -107,7 +124,7 @@
   <link name="CameraTiltPlate_link">
     <visual>
-      <origin xyz="-1.24 .54 0 " rpy="-1.5708 0 -2.1" />
-      <geometry>
-        <mesh filename="package://carl_description/meshes/FullRobot_-_tempPlate-1.STL" />
+      <origin xyz="0 0 0" rpy="0 1.5708 0" />
+      <geometry>
+        <mesh filename="package://carl_description/meshes/CameraPlate.dae" />
       </geometry>
     </visual>
@@ -115,7 +132,7 @@
   <link name="JacoMount_link">
     <visual>
-      <origin xyz="-0.295 0 -0.367" rpy="0 0 0" />
-      <geometry>
-        <mesh filename="package://carl_description/meshes/FullRobot_-_SuperStructure-1_ArmMountHoriz-1.STL" />
+      <origin xyz="0 0 0" rpy="0 0 1.5708" />
+      <geometry>
+        <mesh filename="package://carl_description/meshes/JacoMount.dae" />
       </geometry>
     </visual>
@@ -123,7 +140,7 @@
   <link name="Hokuyo_link">
     <visual>
-      <origin xyz="-0.36 0 0" rpy="0 0 0" />
-      <geometry>
-        <mesh filename="package://carl_description/meshes/FullRobot_-_hokuyo-1.STL" />
+      <origin xyz="0 0 0" rpy="0 0 0" />
+      <geometry>
+        <mesh filename="package://carl_description/meshes/Hokuyo.dae" />
       </geometry>
     </visual>
@@ -131,7 +148,7 @@
    <link name="LeftSideWall_link">
     <visual>
-      <origin xyz="0 -.225 -.27" rpy="0 0 0" />
-      <geometry>
-        <mesh filename="package://carl_description/meshes/FullRobot_-_sideWall-1.STL" />
+      <origin xyz="0 0 0" rpy="0 0 1.5708" />
+      <geometry>
+        <mesh filename="package://carl_description/meshes/SideWall.dae" />
       </geometry>
     </visual>
@@ -139,7 +156,7 @@
    <link name="RightSideWall_link">
     <visual>
-      <origin xyz="0 -.225 -.27" rpy="0 0 0" />
-      <geometry>
-        <mesh filename="package://carl_description/meshes/FullRobot_-_sideWall-1.STL" />
+      <origin xyz="0 0 0" rpy="0 0 1.5708" />
+      <geometry>
+        <mesh filename="package://carl_description/meshes/SideWall.dae" />
       </geometry>
     </visual>
@@ -147,11 +164,11 @@
   <link name="FrontCover_link">
     <visual>
-      <origin xyz="0 0 -.012" rpy="0 0 0" />
-      <geometry>
-        <mesh filename="package://carl_description/meshes/FullRobot_-_FrontCover-1.STL" />
-      </geometry>
-    </visual>
-    <collision>
-      <origin xyz="0 0 -.012" rpy="0 0 0" />
+      <origin xyz="0 0 0" rpy="0 0 1.5708" />
+      <geometry>
+        <mesh filename="package://carl_description/meshes/FrontCover.dae" />
+      </geometry>
+    </visual>
+    <collision>
+      <origin xyz="0 0 0" rpy="0 0 1.5708" />
       <geometry>
         <mesh filename="package://carl_description/meshes/FrontCoverCollision.STL" />
@@ -159,9 +176,10 @@
     </collision>
   </link>
-    <link name="BackCover_link">
-    <visual>
-      <origin xyz="-.237 0 .208" rpy="0 0 0" />
-      <geometry>
-      	<box size="0.005 0.45 0.6" />
+  <link name="BackCover_link">
+    <visual>
+      <origin xyz="0 0 0" rpy="0 0 0" />
+      <geometry>
+      	<!--<box size="0.005 0.45 0.6" />-->
+      	<mesh filename="package://carl_description/meshes/BackCover.dae" />
       </geometry>
     </visual>
@@ -179,28 +197,33 @@
     <axis xyz="0 0 1" />
   </joint>
-  <joint name="BaseToCaster" type="fixed">
-    <parent link="base_link"/>
+  <joint name="BaseToCasterPlate" type="fixed">
+    <parent link="base_link"/>
+    <child link="CasterPlate_link"/>
+    <origin xyz="0.2883 0 0" rpy="0 0 0" />
+  </joint>
+  <joint name="CasterPlateToCaster" type="fixed">
+    <parent link="CasterPlate_link"/>
     <child link="Caster_link"/>
-    <origin xyz="0 0 0" rpy="0 0 0" />
+    <origin xyz="0.0267 0 -0.024" rpy="0 0 0" />
   </joint>
   <joint name="BaseToRearLeftStrut" type="fixed">
     <parent link="base_link"/>
     <child link="RearLeftStrut_link"/>
-    <origin xyz="-0.222 0.20 0.194" rpy="0 0 0" />
+    <origin xyz="-0.222 0.200 -0.102" rpy="0 0 0" />
   </joint>
   <joint name="BaseToRearRightStrut" type="fixed">
     <parent link="base_link"/>
     <child link="RearRightStrut_link"/>
-    <origin xyz="-0.222 -0.20 0.194" rpy="0 0 0" />
+    <origin xyz="-0.222 -0.200 -0.102" rpy="0 0 0" />
   </joint>
   <joint name="RearLeftStrutToTopPlate" type="fixed">
     <parent link="RearRightStrut_link"/>
     <child link="TopPlate_link"/>
-    <origin xyz="0.30 0.20 0.30" rpy="0 0 0" />
+    <origin xyz="0.516 0.20 0.598" rpy="0 0 0" />
   </joint>
   <joint name="RearLeftStrutToCameraLift" type="fixed">
     <parent link="RearRightStrut_link"/>
     <child link="CameraLift_link"/>
-    <origin xyz="0.01 0.20 1.17" rpy="0 0 0" />
+    <origin xyz="0.01 0.20 1.461" rpy="0 0 0" />
   </joint>
     <joint name="CameraLiftToCameraTiltBracket" type="continuous">
@@ -218,10 +241,10 @@
     <parent link="TopPlate_link"/>
     <child link="JacoMount_link"/>
-    <origin xyz="0.216 0 -0.13" rpy="0 0 0" />
+    <origin xyz="0 0 -0.13" rpy="0 0 0" />
   </joint>
   <joint name="CasterToHokuyo" type="fixed">
-    <parent link="Caster_link"/>
+    <parent link="CasterPlate_link"/>
     <child link="Hokuyo_link"/>
-    <origin xyz="0.36 0 0" rpy="0 0 0" />
+    <origin xyz="0.07 0 0.035" rpy="0 0 0" />
   </joint>
   <joint name="RearLeftStrutToLeftSideWall" type="fixed">
@@ -238,5 +261,5 @@
     <parent link="base_link"/>
     <child link="FrontCover_link"/>
-    <origin xyz="0 0 0.012" rpy="0 0 0" />
+    <origin xyz=".247 0 0.242" rpy="0 0 0" />
   </joint>
   <joint name="BaseToBackCover" type="fixed">

Commit message: Fixed transforms to match origins of new meshes

File: carl_description/urdf/carl.urdf (robot description, URDF)
Before this commit: robot carl, 27 links, 26 joints
Joints:
- joint BaseToBackCover: origin xyz=0 0 -0.012 rpy=0 0 0 -> xyz=-.237 0 -0.102 rpy=0 0 0
- joint RearLeftStrutToLeftSideWall: origin xyz=0.229 0.025 0.078 rpy=0 0 0 -> xyz=0.229 0.026 0.447 rpy=0 0 0
- joint RearRightStrutToRightSideWall: origin xyz=0.229 -0.025 0.078 rpy=0 0 0 -> xyz=0.229 -0.026 0.447 rpy=0 0 0

File: carl_description/urdf/carl.xacro (robot description, xacro)
@@ -251,10 +251,10 @@
     <parent link="RearLeftStrut_link"/>
     <child link="LeftSideWall_link"/>
-    <origin xyz="0.229 0.025 0.078" rpy="0 0 0" />
+    <origin xyz="0.229 0.026 0.447" rpy="0 0 0" />
   </joint>
   <joint name="RearRightStrutToRightSideWall" type="fixed">
     <parent link="RearRightStrut_link"/>
     <child link="RightSideWall_link"/>
-    <origin xyz="0.229 -0.025 0.078" rpy="0 0 0" />
+    <origin xyz="0.229 -0.026 0.447" rpy="0 0 0" />
   </joint>
   <joint name="BaseToFrontCover" type="fixed">
@@ -266,5 +266,5 @@
     <parent link="base_link"/>
     <child link="BackCover_link"/>
-    <origin xyz="0 0 -0.012" rpy="0 0 0" />
+    <origin xyz="-.237 0 -0.102" rpy="0 0 0" />
   </joint>
   <xacro:jaco_arm  parent="JacoMount_link"/>
