Commit message: Updates to collision model

File: carl_description/urdf/carl.urdf (robot description, URDF)
Before this commit: robot carl, 27 links, 26 joints
Links:
- link CameraLift_link: geometry collision mesh filename=package://carl_description/meshes/CameraLift.dae; visual mesh filename=package://carl_description/meshes/CameraLift.dae
- link CameraTiltPlate_link: geometry collision mesh filename=package://carl_description/meshes/CameraPlate.dae; visual mesh filename=package://carl_description/meshes/CameraPlate.dae
- link CasterPlate_link: geometry visual mesh filename=package://carl_description/meshes/casterPlate.dae
- link LeftWheel_link: geometry collision cylinder length=0.1 radius=0.25; visual mesh filename=package://carl_description/meshes/Wheel.dae
- link RearLeftStrut_link: geometry collision box size=0.027 0.054 1.055; visual mesh filename=package://carl_description/meshes/RearStrut.dae
- link RearRightStrut_link: geometry collision box size=0.027 0.054 1.055; visual mesh filename=package://carl_description/meshes/RearStrut.dae
- link RightWheel_link: geometry collision cylinder length=0.1 radius=0.25; visual mesh filename=package://carl_description/meshes/Wheel.dae
- link TopPlate_link: geometry collision box size=0.495 0.59 0.65; visual mesh filename=package://carl_description/meshes/TablePlate.dae
Joints:
- joint BaseToLeftWheel: origin xyz=0.02 0.32 0 rpy=-1.5708 0 0 -> xyz=0 0.25 0 rpy=-1.5708 0 0
- joint BaseToRightWheel: origin xyz=0.02 -0.32 0 rpy=1.5708 0 0 -> xyz=0 -0.25 0 rpy=1.5708 0 0
- joint CasterPlateToCaster: axis (none) -> 0 0 1; type fixed -> continuous

File: carl_description/urdf/carl.xacro (robot description, xacro)
@@ -1,6 +1,3 @@
 <?xml version="1.0"?>
-<!--
-If you are reading this, it means I forgot to update the collision model. Remind me.
--->
 <robot xmlns:xacro="http://www.ros.org/wiki/xacro" name="carl">
   <xacro:include filename="$(find jaco_model)/urdf/jaco_arm.xacro" />
@@ -21,7 +18,7 @@
     </visual>
     <collision>
-      <origin xyz="0 0 0" rpy="0 0 0" />
-      <geometry>
-        <cylinder radius="0.25" length="0.090" />
+      <origin xyz="0 0 .025" rpy="0 0 0" />
+      <geometry>
+        <cylinder radius="0.25" length="0.1" />
       </geometry>
     </collision>
@@ -35,7 +32,7 @@
     </visual>
     <collision>
-      <origin xyz="0 0 0" rpy="0 0 0" />
-      <geometry>
-        <cylinder radius="0.25" length="0.090" />
+      <origin xyz="0 0 .025" rpy="0 0 0" />
+      <geometry>
+        <cylinder radius="0.25" length="0.1" />
       </geometry>
     </collision>
@@ -48,6 +45,14 @@
       </geometry>
     </visual>
-    <collision>
-      <origin xyz="0.31 0 -0.12" rpy="0 0 0" />
+  </link>
+  <link name="Caster_link">
+    <visual>
+      <origin xyz="0 0 0" rpy="0 0 1.5708"/>
+      <geometry>
+        <mesh filename="package://carl_description/meshes/caster.dae" />
+      </geometry>
+    </visual>
+    <collision>
+      <origin xyz="0 0 -0.09" rpy="0 0 0" />
       <geometry>
         <cylinder radius="0.116" length="0.213" />
@@ -55,19 +60,19 @@
     </collision>
   </link>
-    <link name="Caster_link">
-    <visual>
-      <origin xyz="0 0 0" rpy="0 0 1.5708"/>
-      <geometry>
-        <mesh filename="package://carl_description/meshes/caster.dae" />
-      </geometry>
-    </visual>
-    <collision>
-      <origin xyz="0.31 0 -0.12" rpy="0 0 0" />
-      <geometry>
-        <cylinder radius="0.116" length="0.213" />
+  <link name="RearLeftStrut_link">
+    <visual>
+      <origin xyz="0 0 0" rpy="0 0 -1.5708" />
+      <geometry>
+        <mesh filename="package://carl_description/meshes/RearStrut.dae" />
+      </geometry>
+    </visual>
+    <collision>
+      <origin xyz="0 -0.4 0.5275" rpy="0 0 0" />
+      <geometry>
+        <box size="0.027 0.054 1.055" />
        </geometry>
     </collision>
   </link>
-  <link name="RearLeftStrut_link">
+  <link name="RearRightStrut_link">
     <visual>
       <origin xyz="0 0 0" rpy="0 0 -1.5708" />
@@ -77,35 +82,21 @@
     </visual>
     <collision>
-      <origin xyz="0 -0.40 0.24" rpy="0 0 0" />
-      <geometry>
-        <box size="0.025 0.051 1.055" />
-       </geometry>
-    </collision>
-  </link>
-  <link name="RearRightStrut_link">
+      <origin xyz="0 0.4 0.5275" rpy="0 0 0" />
+      <geometry>
+        <box size="0.027 0.054 1.055" />
+      </geometry>
+    </collision>
+  </link>
+  <link name="TopPlate_link">
     <visual>
       <origin xyz="0 0 0" rpy="0 0 -1.5708" />
       <geometry>
-        <mesh filename="package://carl_description/meshes/RearStrut.dae" />
-      </geometry>
-    </visual>
-    <collision>
-      <origin xyz="0 0.40 0.24" rpy="0 0 0" />
-      <geometry>
-        <box size="0.025 0.051 1.055" />
-      </geometry>
-    </collision>
-  </link>
-  <link name="TopPlate_link">
-    <visual>
-      <origin xyz="0 0 0" rpy="0 0 -1.5708" />
-      <geometry>
         <mesh filename="package://carl_description/meshes/TablePlate.dae" />
       </geometry>
     </visual>
     <collision>
-      <origin xyz="-.068 0 -0.295" rpy="0 0 0" />
-      <geometry>
-        <box size="0.483 0.584 0.6" />
+      <origin xyz="-.29 0 -0.299" rpy="0 0 0" />
+      <geometry>
+        <box size="0.495 0.59 0.65" />
       </geometry>
     </collision>
@@ -118,4 +109,10 @@
       </geometry>
     </visual>
+    <collision>
+      <origin xyz="0 0 0" rpy="0 0 1.5708" />
+      <geometry>
+        <mesh filename="package://carl_description/meshes/CameraLift.dae" />
+      </geometry>
+    </collision>
   </link>
   <link name="CameraTiltBracket_link">
@@ -129,4 +126,10 @@
       </geometry>
     </visual>
+    <collision>
+      <origin xyz="0 0 0" rpy="0 1.5708 0" />
+      <geometry>
+        <mesh filename="package://carl_description/meshes/CameraPlate.dae" />
+      </geometry>
+    </collision>
   </link>
   <link name="JacoMount_link">
@@ -170,5 +173,5 @@
     </visual>
     <collision>
-      <origin xyz="0 0 0" rpy="0 0 1.5708" />
+      <origin xyz="-.245 0 -.241" rpy="0 0 0" />
       <geometry>
         <mesh filename="package://carl_description/meshes/FrontCoverCollision.STL" />
@@ -188,5 +191,5 @@
     <parent link="base_link"/>
     <child link="LeftWheel_link"/>
-    <origin xyz="0.02 0.32 0" rpy="-1.5708 0 0" />
+    <origin xyz="0 0.25 0" rpy="-1.5708 0 0" />
     <axis xyz="0 0 1" />
   </joint>
@@ -194,5 +197,5 @@
     <parent link="base_link"/>
     <child link="RightWheel_link"/>
-    <origin xyz="0.02 -0.32 0" rpy="1.5708 0 0" />
+    <origin xyz="0 -0.25 0" rpy="1.5708 0 0" />
     <axis xyz="0 0 1" />
   </joint>
@@ -202,8 +205,9 @@
     <origin xyz="0.2883 0 0" rpy="0 0 0" />
   </joint>
-  <joint name="CasterPlateToCaster" type="fixed">
+  <joint name="CasterPlateToCaster" type="continuous">
     <parent link="CasterPlate_link"/>
     <child link="Caster_link"/>
     <origin xyz="0.0267 0 -0.024" rpy="0 0 0" />
+    <axis xyz="0 0 1" />
   </joint>
   <joint name="BaseToRearLeftStrut" type="fixed">

Commit message: Added lettering

File: carl_description/urdf/carl.urdf (robot description, URDF)
Before this commit: robot carl, 27 links, 26 joints
Links:
- added link RearLeftStrutInside_link; visual box size=0.02 0.045 1
- added link RearRightStrutInside_link; visual box size=0.02 0.045 1
Joints:
- added joint RearLeftStrutToRearLeftStutInside: type fixed, parent RearLeftStrut_link, child RearLeftStrutInside_link, origin xyz=0 0 0 rpy=0 0 0
- added joint RearRightStrutToRearRightStutInside: type fixed, parent RearRightStrut_link, child RearRightStrutInside_link, origin xyz=0 0 0 rpy=0 0 0

File: carl_description/urdf/carl.xacro (robot description, xacro)
@@ -88,4 +88,20 @@
     </collision>
   </link>
+  <link name="RearLeftStrutInside_link">
+    <visual>
+     <origin xyz="0 0 0.5275" rpy="0 0 0" />
+      <geometry>
+        <box size="0.02 0.045 1" />
+      </geometry>
+    </visual>
+  </link>
+  <link name="RearRightStrutInside_link">
+    <visual>
+     <origin xyz="0 0 0.5275" rpy="0 0 0" />
+      <geometry>
+        <box size="0.02 0.045 1" />
+      </geometry>
+    </visual>
+  </link>
   <link name="TopPlate_link">
     <visual>
@@ -221,4 +237,14 @@
     <origin xyz="-0.222 -0.200 -0.102" rpy="0 0 0" />
   </joint>
+  <joint name="RearRightStrutToRearRightStutInside" type="fixed">
+    <parent link="RearRightStrut_link"/>
+    <child link="RearRightStrutInside_link"/>
+    <origin xyz="0 0 0" rpy="0 0 0" />
+  </joint>
+  <joint name="RearLeftStrutToRearLeftStutInside" type="fixed">
+    <parent link="RearLeftStrut_link"/>
+    <child link="RearLeftStrutInside_link"/>
+    <origin xyz="0 0 0" rpy="0 0 0" />
+  </joint>
   <joint name="RearLeftStrutToTopPlate" type="fixed">
     <parent link="RearRightStrut_link"/>

Commit message: Renamed a couple meshes.

File: carl_description/urdf/carl.urdf (robot description, URDF)
Before this commit: robot carl, 29 links, 28 joints
Links:
- link CasterPlate_link: geometry visual mesh filename=package://carl_description/meshes/CasterPlate.dae
- link Caster_link: geometry collision cylinder length=0.213 radius=0.116; visual mesh filename=package://carl_description/meshes/Caster.dae

File: carl_description/urdf/carl.xacro (robot description, xacro)
@@ -42,5 +42,5 @@
       <origin xyz="0 0 0" rpy="0 0 1.5708"/>
       <geometry>
-        <mesh filename="package://carl_description/meshes/casterPlate.dae" />
+        <mesh filename="package://carl_description/meshes/CasterPlate.dae" />
       </geometry>
     </visual>
@@ -50,5 +50,5 @@
       <origin xyz="0 0 0" rpy="0 0 1.5708"/>
       <geometry>
-        <mesh filename="package://carl_description/meshes/caster.dae" />
+        <mesh filename="package://carl_description/meshes/Caster.dae" />
       </geometry>
     </visual>

Commit message: Renamed meshes to follow ROS conventions

File: carl_description/urdf/carl.urdf (robot description, URDF)
Before this commit: robot carl, 29 links, 28 joints
Links:
- removed link LeftSideWall_link
- removed link RightSideWall_link
- added link LeftSideCover_link; visual mesh filename=package://carl_description/meshes/side_cover.dae
- added link RightSideCover_link; visual mesh filename=package://carl_description/meshes/side_cover.dae
- link BackCover_link: geometry visual mesh filename=package://carl_description/meshes/back_cover.dae
- link CameraLift_link: geometry collision mesh filename=package://carl_description/meshes/camera_lift.dae; visual mesh filename=package://carl_description/meshes/camera_lift.dae
- link CameraTiltPlate_link: geometry collision mesh filename=package://carl_description/meshes/camera_plate.dae; visual mesh filename=package://carl_description/meshes/camera_plate.dae
- link CasterPlate_link: geometry visual mesh filename=package://carl_description/meshes/caster_plate.dae
- link Caster_link: geometry collision cylinder length=0.213 radius=0.116; visual mesh filename=package://carl_description/meshes/caster.dae
- link FrontCover_link: geometry collision mesh filename=package://carl_description/meshes/front_cover_collision.stl; visual mesh filename=package://carl_description/meshes/front_cover.dae
- link Hokuyo_link: geometry visual mesh filename=package://carl_description/meshes/hokuyo.dae
- link JacoMount_link: geometry visual mesh filename=package://carl_description/meshes/jaco_mount.dae
- link LeftWheel_link: geometry collision cylinder length=0.1 radius=0.25; visual mesh filename=package://carl_description/meshes/wheel.dae
- link RearLeftStrut_link: geometry collision box size=0.027 0.054 1.055; visual mesh filename=package://carl_description/meshes/rear_strut.dae
- link RearRightStrut_link: geometry collision box size=0.027 0.054 1.055; visual mesh filename=package://carl_description/meshes/rear_strut.dae
- link RightWheel_link: geometry collision cylinder length=0.1 radius=0.25; visual mesh filename=package://carl_description/meshes/wheel.dae
- link TopPlate_link: geometry collision box size=0.495 0.59 0.65; visual mesh filename=package://carl_description/meshes/table_plate.dae
- link base_link: geometry visual mesh filename=package://carl_description/meshes/base.dae
Joints:
- removed joint RearLeftStrutToLeftSideWall
- removed joint RearRightStrutToRightSideWall
- added joint RearLeftStrutToLeftSideCover: type fixed, parent RearLeftStrut_link, child LeftSideCover_link, origin xyz=0.229 0.026 0.447 rpy=0 0 0
- added joint RearRightStrutToRightSideCover: type fixed, parent RearRightStrut_link, child RightSideCover_link, origin xyz=0.229 -0.026 0.447 rpy=0 0 0

File: carl_description/urdf/carl.xacro (robot description, xacro)
@@ -6,5 +6,5 @@
       <origin xyz="0 0 0" rpy="0 0 0"/>
       <geometry>
-        <mesh filename="package://carl_description/meshes/Base.dae" />
+        <mesh filename="package://carl_description/meshes/base.dae" />
       </geometry>
     </visual>
@@ -14,5 +14,5 @@
       <origin xyz="0 0 0" rpy="0 0 0" />
       <geometry>
-        <mesh filename="package://carl_description/meshes/Wheel.dae" />
+        <mesh filename="package://carl_description/meshes/wheel.dae" />
       </geometry>
     </visual>
@@ -28,5 +28,5 @@
       <origin xyz="0 0 0" rpy="0 0 0" />
       <geometry>
-        <mesh filename="package://carl_description/meshes/Wheel.dae" />
+        <mesh filename="package://carl_description/meshes/wheel.dae" />
       </geometry>
     </visual>
@@ -42,5 +42,5 @@
       <origin xyz="0 0 0" rpy="0 0 1.5708"/>
       <geometry>
-        <mesh filename="package://carl_description/meshes/CasterPlate.dae" />
+        <mesh filename="package://carl_description/meshes/caster_plate.dae" />
       </geometry>
     </visual>
@@ -50,5 +50,5 @@
       <origin xyz="0 0 0" rpy="0 0 1.5708"/>
       <geometry>
-        <mesh filename="package://carl_description/meshes/Caster.dae" />
+        <mesh filename="package://carl_description/meshes/caster.dae" />
       </geometry>
     </visual>
@@ -64,5 +64,5 @@
       <origin xyz="0 0 0" rpy="0 0 -1.5708" />
       <geometry>
-        <mesh filename="package://carl_description/meshes/RearStrut.dae" />
+        <mesh filename="package://carl_description/meshes/rear_strut.dae" />
       </geometry>
     </visual>
@@ -78,5 +78,5 @@
       <origin xyz="0 0 0" rpy="0 0 -1.5708" />
       <geometry>
-        <mesh filename="package://carl_description/meshes/RearStrut.dae" />
+        <mesh filename="package://carl_description/meshes/rear_strut.dae" />
       </geometry>
     </visual>
@@ -108,5 +108,5 @@
       <origin xyz="0 0 0" rpy="0 0 -1.5708" />
       <geometry>
-        <mesh filename="package://carl_description/meshes/TablePlate.dae" />
+        <mesh filename="package://carl_description/meshes/table_plate.dae" />
       </geometry>
     </visual>
@@ -122,11 +122,11 @@
       <origin xyz="0 0 0" rpy="0 0 1.5708" />
       <geometry>
-        <mesh filename="package://carl_description/meshes/CameraLift.dae" />
-      </geometry>
-    </visual>
-    <collision>
-      <origin xyz="0 0 0" rpy="0 0 1.5708" />
-      <geometry>
-        <mesh filename="package://carl_description/meshes/CameraLift.dae" />
+        <mesh filename="package://carl_description/meshes/camera_lift.dae" />
+      </geometry>
+    </visual>
+    <collision>
+      <origin xyz="0 0 0" rpy="0 0 1.5708" />
+      <geometry>
+        <mesh filename="package://carl_description/meshes/camera_lift.dae" />
       </geometry>
     </collision>
@@ -139,5 +139,5 @@
       <origin xyz="0 0 0" rpy="0 1.5708 0" />
       <geometry>
-        <mesh filename="package://carl_description/meshes/CameraPlate.dae" />
+        <mesh filename="package://carl_description/meshes/camera_plate.dae" />
       </geometry>
     </visual>
@@ -145,5 +145,5 @@
       <origin xyz="0 0 0" rpy="0 1.5708 0" />
       <geometry>
-        <mesh filename="package://carl_description/meshes/CameraPlate.dae" />
+        <mesh filename="package://carl_description/meshes/camera_plate.dae" />
       </geometry>
     </collision>
@@ -153,5 +153,5 @@
       <origin xyz="0 0 0" rpy="0 0 1.5708" />
       <geometry>
-        <mesh filename="package://carl_description/meshes/JacoMount.dae" />
+        <mesh filename="package://carl_description/meshes/jaco_mount.dae" />
       </geometry>
     </visual>
@@ -161,21 +161,21 @@
       <origin xyz="0 0 0" rpy="0 0 0" />
       <geometry>
-        <mesh filename="package://carl_description/meshes/Hokuyo.dae" />
-      </geometry>
-    </visual>
-  </link>
-   <link name="LeftSideWall_link">
-    <visual>
-      <origin xyz="0 0 0" rpy="0 0 1.5708" />
-      <geometry>
-        <mesh filename="package://carl_description/meshes/SideWall.dae" />
-      </geometry>
-    </visual>
-  </link>
-   <link name="RightSideWall_link">
-    <visual>
-      <origin xyz="0 0 0" rpy="0 0 1.5708" />
-      <geometry>
-        <mesh filename="package://carl_description/meshes/SideWall.dae" />
+        <mesh filename="package://carl_description/meshes/hokuyo.dae" />
+      </geometry>
+    </visual>
+  </link>
+   <link name="LeftSideCover_link">
+    <visual>
+      <origin xyz="0 0 0" rpy="0 0 1.5708" />
+      <geometry>
+        <mesh filename="package://carl_description/meshes/side_cover.dae" />
+      </geometry>
+    </visual>
+  </link>
+   <link name="RightSideCover_link">
+    <visual>
+      <origin xyz="0 0 0" rpy="0 0 1.5708" />
+      <geometry>
+        <mesh filename="package://carl_description/meshes/side_cover.dae" />
       </geometry>
     </visual>
@@ -185,5 +185,5 @@
       <origin xyz="0 0 0" rpy="0 0 1.5708" />
       <geometry>
-        <mesh filename="package://carl_description/meshes/FrontCover.dae" />
+        <mesh filename="package://carl_description/meshes/front_cover.dae" />
       </geometry>
     </visual>
@@ -191,5 +191,5 @@
       <origin xyz="-.245 0 -.241" rpy="0 0 0" />
       <geometry>
-        <mesh filename="package://carl_description/meshes/FrontCoverCollision.STL" />
+        <mesh filename="package://carl_description/meshes/front_cover_collision.stl" />
       </geometry>
     </collision>
@@ -200,5 +200,5 @@
       <geometry>
       	<!--<box size="0.005 0.45 0.6" />-->
-      	<mesh filename="package://carl_description/meshes/BackCover.dae" />
+      	<mesh filename="package://carl_description/meshes/back_cover.dae" />
       </geometry>
     </visual>
@@ -278,12 +278,12 @@
     <origin xyz="0.07 0 0.035" rpy="0 0 0" />
   </joint>
-  <joint name="RearLeftStrutToLeftSideWall" type="fixed">
+  <joint name="RearLeftStrutToLeftSideCover" type="fixed">
     <parent link="RearLeftStrut_link"/>
-    <child link="LeftSideWall_link"/>
+    <child link="LeftSideCover_link"/>
     <origin xyz="0.229 0.026 0.447" rpy="0 0 0" />
   </joint>
-  <joint name="RearRightStrutToRightSideWall" type="fixed">
+  <joint name="RearRightStrutToRightSideCover" type="fixed">
     <parent link="RearRightStrut_link"/>
-    <child link="RightSideWall_link"/>
+    <child link="RightSideCover_link"/>
     <origin xyz="0.229 -0.026 0.447" rpy="0 0 0" />
   </joint>
