Commit message: used cylinder for wheel collision model

File: carl_description/urdf/components/carl_wheel.urdf.xacro (robot description, xacro)
@@ -17,5 +17,8 @@
         <origin xyz="0 0 0" rpy="0 0 0" />
         <geometry>
+          <!--
           <mesh scale="${M_SCALE} ${M_SCALE} ${M_SCALE}" filename="package://carl_description/meshes/wheel.stl" />
+          -->
+          <cylinder radius="0.25" length="0.11"/>
         </geometry>
       </collision>
