Commit message: caster

File: carl_description/urdf/components/carl_caster_assembly.urdf.xacro (robot description, xacro)
@@ -41,7 +41,7 @@
       </visual>
       <collision>
-        <origin xyz="0 0 0" rpy="0 0 0" />
+        <origin xyz="-0.0381 0 -0.0929" rpy="0 0 0" />
         <geometry>
-          <mesh scale="${M_SCALE} ${M_SCALE} ${M_SCALE}" filename="package://carl_description/meshes/caster.stl" />
+          <box size="0.17 0.0636 0.1858"/>
         </geometry>
       </collision>
