Commit message: servo

File: carl_description/urdf/components/carl_asus_camera.urdf.xacro (robot description, xacro)
@@ -23,7 +23,7 @@
       </visual>
       <collision>
-        <origin xyz="0 0 0" rpy="0 0 0" />
+        <origin xyz="0.0279 0.0 0.0" rpy="0 0 0" />
         <geometry>
-          <mesh scale="${M_SCALE} ${M_SCALE} ${M_SCALE}" filename="package://carl_description/meshes/servo_mount.stl" />
+          <box size="0.057 0.0508 0.089"/>
         </geometry>
       </collision>
@@ -42,7 +42,7 @@
       </visual>
       <collision>
-        <origin xyz="0 0 0" rpy="0 0 0" />
+        <origin xyz="0.01344 -0.0184 0" rpy="0 0 0" />
         <geometry>
-          <mesh scale="${M_SCALE} ${M_SCALE} ${M_SCALE}" filename="package://carl_description/meshes/servo.stl" />
+          <box size="0.05 0.0382 0.032"/>
         </geometry>
       </collision>

Commit message: servo arm, caster plate

File: carl_description/urdf/components/carl_asus_camera.urdf.xacro (robot description, xacro)
@@ -62,7 +62,7 @@
       </visual>
       <collision>
-        <origin xyz="0 0 0" rpy="0 0 0" />
+        <origin xyz="0 -0.021 -0.02405" rpy="0 0 0" />
         <geometry>
-          <mesh scale="${M_SCALE} ${M_SCALE} ${M_SCALE}" filename="package://carl_description/meshes/servo_arm.stl" />
+          <box size="0.029 0.067 0.049"/>
         </geometry>
       </collision>

File: carl_description/urdf/components/carl_caster_assembly.urdf.xacro (robot description, xacro)
@@ -21,7 +21,7 @@
       </visual>
       <collision>
-        <origin xyz="0 0 0" rpy="0 0 ${M_PI/2}" />
+        <origin xyz="0.005 0 -0.04145" rpy="0 0 ${M_PI/2}" />
         <geometry>
-          <mesh scale="${M_SCALE} ${M_SCALE} ${M_SCALE}" filename="package://carl_description/meshes/caster_plate.stl" />
+          <box size="0.552 0.174 0.0949"/>
         </geometry>
       </collision>

Commit message: Updated transform between asus mount and asus; added carl_tools for miscellaneous packages, currently including calibration for the asus camera transform.

File: carl_description/urdf/components/carl_asus_camera.urdf.xacro (robot description, xacro)
@@ -88,5 +88,8 @@
     </link>
     <xacro:sensor_asus_xtion_pro parent="asus_mount_link">
-      <origin xyz="-0.016 -0.008 0.018" rpy="0 -${M_PI/2} 0" />
+      <!-- hand measured -->
+      <!--<origin xyz="-0.016 -0.008 0.018" rpy="0 -${M_PI/2} 0" />-->
+      <!-- calibrated -->
+      <origin xyz="-0.021523 -0.003366 0.021402" rpy="0.0 -1.508124 0.0" />
     </xacro:sensor_asus_xtion_pro>
   </xacro:macro>

Commit message: Orientation filter ignores accelerometer measurements when anything more than the gravity vector is detected

File: carl_description/urdf/components/carl_asus_camera.urdf.xacro (robot description, xacro)
@@ -89,7 +89,7 @@
     <xacro:sensor_asus_xtion_pro parent="asus_mount_link">
       <!-- hand measured -->
-      <!--<origin xyz="-0.016 -0.008 0.018" rpy="0 -${M_PI/2} 0" />-->
+      <origin xyz="-0.016 -0.008 0.018" rpy="0 -${M_PI/2} 0" />
       <!-- calibrated -->
-      <origin xyz="-0.021523 -0.003366 0.021402" rpy="0.0 -1.508124 0.0" />
+      <!--<origin xyz="-0.021523 -0.003366 0.021402" rpy="0.0 -1.508124 0.0" />-->
     </xacro:sensor_asus_xtion_pro>
   </xacro:macro>

Commit message: New camera calibrations

File: carl_description/urdf/components/carl_asus_camera.urdf.xacro (robot description, xacro)
@@ -91,5 +91,5 @@
       <origin xyz="-0.016 -0.008 0.018" rpy="0 -${M_PI/2} 0" />
       <!-- calibrated -->
-      <!--<origin xyz="-0.021523 -0.003366 0.021402" rpy="0.0 -1.508124 0.0" />-->
+      <!--<origin xyz="-0.005275 -0.001578 0.014353" rpy="-1.061086 -1.545 1.0" />-->
     </xacro:sensor_asus_xtion_pro>
   </xacro:macro>
