Commit message: Fixed indentation

File: carl_description/urdf/carl_base/carl_camera_mount.urdf.xacro (robot description, xacro)
@@ -7,6 +7,6 @@
   <xacro:macro name="carl_camera_mount">
     <xacro:sensor_asus_xtion_pro parent="camera_tilt_plate_link">
-	      <origin xyz=".025 -.02 -.02" rpy="-1.5708 0 -1.5708" />
-	</xacro:sensor_asus_xtion_pro>
+      <origin xyz=".025 -.02 -.02" rpy="-1.5708 0 -1.5708" />
+    </xacro:sensor_asus_xtion_pro>
     <link name="camera_lift_link">
       <visual>

Commit message: Changed default camera angle

File: carl_description/urdf/carl_base/carl_camera_mount.urdf.xacro (robot description, xacro)
@@ -48,5 +48,5 @@
       <parent link="camera_lift_link"/>
       <child link="camera_tilt_bracket_link"/>
-      <origin xyz="0.03 -0.10 0" rpy="1.5708 0 0" />
+      <origin xyz="0.03 -0.10 0" rpy="1.5708 -1.5708 0" />
       <axis xyz="0 0 1" />
     </joint>

Commit message: Added newly machined components to urdf

File: carl_description/urdf/carl_base/carl_camera_mount.urdf.xacro (robot description, xacro)
@@ -11,14 +11,14 @@
     <link name="camera_lift_link">
       <visual>
-        <origin xyz="0 0 0" rpy="0 0 1.5708" />
+        <origin xyz="0 0 0" rpy="0 1.5708 1.5708" />
         <geometry>
           <mesh filename="package://carl_description/meshes/camera_lift.dae" />
         </geometry>
       </visual>
-      <collision>
-        <origin xyz="0 0 0" rpy="0 0 1.5708" />
+	  <collision>
+        <origin xyz="0.0127 0 0" rpy="0 0 0" />
         <geometry>
-          <mesh filename="package://carl_description/meshes/camera_lift.dae" />
-        </geometry>
+          <box size="0.027 0.454 0.054" />
+         </geometry>
       </collision>
     </link>
@@ -30,5 +30,5 @@
         <origin xyz="0 0 0" rpy="0 1.5708 0" />
         <geometry>
-          <mesh filename="package://carl_description/meshes/camera_plate.dae" />
+          <mesh filename="package://carl_description/meshes/camera_mount.dae" />
         </geometry>
       </visual>
@@ -36,5 +36,5 @@
         <origin xyz="0 0 0" rpy="0 1.5708 0" />
         <geometry>
-          <mesh filename="package://carl_description/meshes/camera_plate.dae" />
+          <mesh filename="package://carl_description/meshes/camera_mount.dae" />
         </geometry>
       </collision>
@@ -43,5 +43,5 @@
       <parent link="right_rear_strut_link"/>
       <child link="camera_lift_link"/>
-      <origin xyz="0.01 0.20 1.461" rpy="0 0 0" />
+      <origin xyz="0.013 0.20 1.538" rpy="0 0 0" />
     </joint>
     <joint name="camera_lift_camera_tilt_bracket_joint" type="continuous">

File: carl_description/urdf/components/carl_rear_strut.urdf.xacro (robot description, xacro)
@@ -11,4 +11,9 @@
    	  <child link="${suffix}_rear_strut_inside_link"/>
       <origin xyz="0 0 0" rpy="0 0 0" />
+    </joint>
+    <joint name="${suffix}_rear_strut_link_${suffix}_rear_strut_top_link_joint" type="fixed">
+      <parent link="${suffix}_rear_strut_link"/>
+   	  <child link="${suffix}_rear_strut_top_link"/>
+      <origin xyz="0 0.001 1.055" rpy="0 0 0" />
     </joint>
     <link name="${suffix}_rear_strut_inside_link">
@@ -34,4 +39,18 @@
       </collision>
     </link>
+    <link name="${suffix}_rear_strut_top_link">
+      <visual>
+        <origin xyz="0 0 0" rpy="0 0 -1.5708" />
+        <geometry>
+          <mesh filename="package://carl_description/meshes/rear_strut_top.dae" />
+        </geometry>
+      </visual>
+      <collision>
+        <origin xyz="0 -0.001 0.2285" rpy="0 0 0" />
+        <geometry>
+          <box size="0.027 0.054 0.4575" />
+         </geometry>
+      </collision>
+    </link>
   </xacro:macro>
 </root>

Commit message: Added new servo mount to model

File: carl_description/urdf/carl_base/carl_camera_mount.urdf.xacro (robot description, xacro)
@@ -6,6 +6,6 @@
   <xacro:include filename="$(find carl_description)/urdf/sensors/asus_xtion_pro.urdf.xacro" />
   <xacro:macro name="carl_camera_mount">
-    <xacro:sensor_asus_xtion_pro parent="camera_tilt_plate_link">
-      <origin xyz=".025 -.02 -.02" rpy="-1.5708 0 -1.5708" />
+    <xacro:sensor_asus_xtion_pro parent="camera_mount_link">
+      <origin xyz="-0.016 -0.008 0.018" rpy="0 -1.5708 0" />
     </xacro:sensor_asus_xtion_pro>
     <link name="camera_lift_link">
@@ -23,8 +23,5 @@
       </collision>
     </link>
-    <link name="camera_tilt_bracket_link">
-	  <!--exists to move center of rotation for camera mount-->
-    </link>
-    <link name="camera_tilt_plate_link">
+    <link name="camera_mount_link">
       <visual>
         <origin xyz="0 0 0" rpy="0 1.5708 0" />
@@ -40,4 +37,52 @@
       </collision>
     </link>
+    <link name="servo_mount_link">
+      <visual>
+        <origin xyz="0 0 0" rpy="0 0 0" />
+        <geometry>
+          <mesh filename="package://carl_description/meshes/servo_mount.dae" />
+        </geometry>
+      </visual>
+      <!--
+      <collision>
+        <origin xyz="0 0 0" rpy="0 1.5708 0" />
+        <geometry>
+          <mesh filename="package://carl_description/meshes/servo_mount.dae" />
+        </geometry>
+      </collision>
+      -->
+    </link>
+    <link name="servo_link">
+      <visual>
+        <origin xyz="0 0 0" rpy="0 0 0" />
+        <geometry>
+          <mesh filename="package://carl_description/meshes/servo.dae" />
+        </geometry>
+      </visual>
+      <!--
+      <collision>
+        <origin xyz="0 0 0" rpy="0 0 0" />
+        <geometry>
+          <mesh filename="package://carl_description/meshes/servo.dae" />
+        </geometry>
+      </collision>
+      -->
+    </link>
+    <link name="servo_arm_link">
+      <visual>
+        <origin xyz="0 0 0" rpy="0 0 0" />
+        <geometry>
+          <mesh filename="package://carl_description/meshes/servo_arm.dae" />
+        </geometry>
+      </visual>
+      <!--
+      <collision>
+        <origin xyz="0 0 0" rpy="0 0 0" />
+        <geometry>
+          <mesh filename="package://carl_description/meshes/servo_arm.dae" />
+        </geometry>
+      </collision>
+      -->
+    </link>
     <joint name="left_rear_strut_camera_lift_joint" type="fixed">
       <parent link="right_rear_strut_link"/>
@@ -45,14 +90,25 @@
       <origin xyz="0.013 0.20 1.538" rpy="0 0 0" />
     </joint>
-    <joint name="camera_lift_camera_tilt_bracket_joint" type="continuous">
+    <joint name="camera_lift_servo_mount_joint" type="fixed">
       <parent link="camera_lift_link"/>
-      <child link="camera_tilt_bracket_link"/>
-      <origin xyz="0.03 -0.10 0" rpy="1.5708 -1.5708 0" />
+      <child link="servo_mount_link"/>
+      <origin xyz="0 0 0" rpy="1.5708 0 0" />
       <axis xyz="0 0 1" />
     </joint>
-    <joint name="camera_lift_bracket_camera_tilt_plate_joint" type="fixed">
-      <parent link="camera_tilt_bracket_link"/>
-      <child link="camera_tilt_plate_link"/>
-      <origin xyz="0.11 0 -0.10" rpy="0 0 0" />
+    <joint name="servo_mount_servo_joint" type="fixed">
+      <parent link="servo_mount_link"/>
+      <child link="servo_link"/>
+      <origin xyz="0.073 0.013 0.0187" rpy="1.5708 0 3.92699" />
+    </joint>
+    <joint name="servo_servo_arm_joint" type="continuous">
+      <parent link="servo_link"/>
+      <child link="servo_arm_link"/>
+      <origin xyz="0 -0.042 0" rpy="1.5708 1.5708 0" />
+      <axis xyz="0 0 1" />
+    </joint>
+    <joint name="servo_arm_camera_mount_joint" type="fixed">
+      <parent link="servo_arm_link"/>
+      <child link="camera_mount_link"/>
+      <origin xyz="0 -0.053 -0.016" rpy="1.5708 0 1.5708" />
     </joint>
   </xacro:macro>

Commit message: Updated collision model

File: carl_description/urdf/carl_base/carl_camera_mount.urdf.xacro (robot description, xacro)
@@ -6,7 +6,4 @@
   <xacro:include filename="$(find carl_description)/urdf/sensors/asus_xtion_pro.urdf.xacro" />
   <xacro:macro name="carl_camera_mount">
-    <xacro:sensor_asus_xtion_pro parent="camera_mount_link">
-      <origin xyz="-0.016 -0.008 0.018" rpy="0 -1.5708 0" />
-    </xacro:sensor_asus_xtion_pro>
     <link name="camera_lift_link">
       <visual>
@@ -17,5 +14,5 @@
       </visual>
 	  <collision>
-        <origin xyz="0.0127 0 0" rpy="0 0 0" />
+        <origin xyz="-0.0127 0 0" rpy="0 0 0" />
         <geometry>
           <box size="0.027 0.454 0.054" />
@@ -30,10 +27,4 @@
         </geometry>
       </visual>
-      <collision>
-        <origin xyz="0 0 0" rpy="0 1.5708 0" />
-        <geometry>
-          <mesh filename="package://carl_description/meshes/camera_mount.dae" />
-        </geometry>
-      </collision>
     </link>
     <link name="servo_mount_link">
@@ -44,12 +35,10 @@
         </geometry>
       </visual>
-      <!--
-      <collision>
-        <origin xyz="0 0 0" rpy="0 1.5708 0" />
+	  <collision>
+        <origin xyz="0.023 0 0" rpy="0 0 0" />
         <geometry>
-          <mesh filename="package://carl_description/meshes/servo_mount.dae" />
-        </geometry>
+          <box size="0.08 0.055 0.09" />
+         </geometry>
       </collision>
-      -->
     </link>
     <link name="servo_link">
@@ -60,12 +49,10 @@
         </geometry>
       </visual>
-      <!--
-      <collision>
-        <origin xyz="0 0 0" rpy="0 0 0" />
+	  <collision>
+        <origin xyz="0.01 -0.021 0" rpy="0 0 0" />
         <geometry>
-          <mesh filename="package://carl_description/meshes/servo.dae" />
-        </geometry>
+          <box size="0.06 0.05 0.035" />
+         </geometry>
       </collision>
-      -->
     </link>
     <link name="servo_arm_link">
@@ -76,13 +63,14 @@
         </geometry>
       </visual>
-      <!--
-      <collision>
-        <origin xyz="0 0 0" rpy="0 0 0" />
+	  <collision>
+        <origin xyz="0 -0.01 -0.02" rpy="0 0 0" />
         <geometry>
-          <mesh filename="package://carl_description/meshes/servo_arm.dae" />
-        </geometry>
+          <box size="0.035 0.05 0.06" />
+         </geometry>
       </collision>
-      -->
     </link>
+    <xacro:sensor_asus_xtion_pro parent="camera_mount_link">
+      <origin xyz="-0.016 -0.008 0.018" rpy="0 -1.5708 0" />
+    </xacro:sensor_asus_xtion_pro>
     <joint name="left_rear_strut_camera_lift_joint" type="fixed">
       <parent link="right_rear_strut_link"/>

File: carl_description/urdf/sensors/asus_xtion_pro.urdf.xacro (robot description, xacro)
@@ -23,5 +23,5 @@
         <origin xyz="0.0 0.0 0.0" rpy="0 0 0" />
         <geometry>
-        <box size="0.0730 .2760 0.0720"/>
+        <box size="0.0830 .2760 0.0720"/>
       </geometry>
       </collision>

Commit message: Rotated right_rear_strut 180 degrees

File: carl_description/urdf/carl_base/carl_camera_mount.urdf.xacro (robot description, xacro)
@@ -73,8 +73,8 @@
       <origin xyz="-0.016 -0.008 0.018" rpy="0 -1.5708 0" />
     </xacro:sensor_asus_xtion_pro>
-    <joint name="left_rear_strut_camera_lift_joint" type="fixed">
+    <joint name="right_rear_strut_camera_lift_joint" type="fixed">
       <parent link="right_rear_strut_link" />
       <child link="camera_lift_link" />
-      <origin xyz="0.013 0.20 1.538" rpy="0 0 0" />
+      <origin xyz="-0.013 -0.20 1.538" rpy="0 0 3.1415926536" />
     </joint>
     <joint name="camera_lift_servo_mount_joint" type="fixed">

File: carl_description/urdf/carl_base/carl_covers.urdf.xacro (robot description, xacro)
@@ -8,5 +8,5 @@
     <!-- right side cover -->
     <xacro:carl_side_cover suffix="right" parent="right_rear_strut_link">
-      <origin xyz="0.229 -0.026 0.447" rpy="0 0 0" />
+      <origin xyz="-0.229 -0.026 0.447" rpy="0 0 0" />
     </xacro:carl_side_cover>
     <!-- left side cover -->

File: carl_description/urdf/carl_base/carl_superstructure.urdf.xacro (robot description, xacro)
@@ -12,10 +12,10 @@
     <!-- right rear strut -->
     <xacro:carl_rear_strut suffix="right" parent="${name}_link">
-      <origin xyz="-0.222 -0.200 -0.102" rpy="0 0 0" />
+      <origin xyz="-0.222 -0.200 -0.102" rpy="0 0 3.1415926536" />
     </xacro:carl_rear_strut>
     <joint name="left_rear_strut_top_plate_joint" type="fixed">
       <parent link="right_rear_strut_link" />
       <child link="top_plate_link" />
-      <origin xyz="0.516 0.20 0.598" rpy="0 0 0" />
+      <origin xyz="-0.516 -0.20 0.598" rpy="0 0 3.14159265" />
     </joint>
     <joint name="top_plate_jaco_mount" type="fixed">
@@ -32,5 +32,5 @@
       </visual>
       <collision>
-        <origin xyz="-.29 0 -0.299" rpy="0 0 0" />
+        <origin xyz="-.29 0 -0.299" rpy="0 0 3.1415926536" />
         <geometry>
           <box size="0.495 0.59 0.65" />
