Commit message: Added creative camera

File: carl_description/urdf/carl_base/carl_creative_camera_mount.urdf.xacro (robot description, xacro)
@@ -5,4 +5,5 @@
        xmlns:xacro="http://ros.org/wiki/xacro">
   <xacro:include filename="$(find carl_description)/urdf/sensors/creative_camera.urdf.xacro" />
+  <!-- TODO FIX COLLISISION MODEL -->
   <xacro:macro name="carl_creative_camera_mount">
     <link name="creative_mount_link">
@@ -45,8 +46,27 @@
         <origin xyz="0 -0.01 -0.02" rpy="0 0 0" />
         <geometry>
+          <box size="0.035 0.09 0.06" />
+         </geometry>
+      </collision>
+    </link>
+    <link name="creative_plate_link">
+      <visual>
+        <origin xyz="0 0 0" rpy="0 0 0" />
+        <geometry>
+          <mesh filename="package://carl_description/meshes/creative_plate.min.dae" />
+        </geometry>
+      </visual>
+      <!--
+	  <collision>
+        <origin xyz="0 -0.01 -0.02" rpy="0 0 0" />
+        <geometry>
           <box size="0.035 0.05 0.06" />
          </geometry>
       </collision>
+      -->
     </link>
+    <xacro:sensor_creative_camera parent="creative_plate_link">
+      <origin xyz="0 0.0 0.012" rpy="0 0 0" />
+    </xacro:sensor_creative_camera>
     <joint name="top_plate_creative_mount_joint" type="fixed">
       <parent link="top_plate_link" />
@@ -65,16 +85,9 @@
       <axis xyz="0 0 1" />
     </joint>
-<!--
--->
-    <!--
-    <xacro:sensor_creative_xtion_pro parent="creative_mount_link">
-      <origin xyz="-0.016 -0.008 0.018" rpy="0 -1.5708 0" />
-    </xacro:sensor_creative_xtion_pro>
-    <joint name="creative_servo_arm_creative_mount_joint" type="fixed">
+    <joint name="creative_servo_arm_creative_plate_joint" type="fixed">
       <parent link="creative_servo_arm_link" />
-      <child link="creative_mount_link" />
-      <origin xyz="0 -0.053 -0.016" rpy="1.5708 0 1.5708" />
+      <child link="creative_plate_link" />
+      <origin xyz="0 -0.057 -0.024" rpy="1.5708 1.5708 0" />
     </joint>
-    -->
   </xacro:macro>
 </robot>

File: carl_description/urdf/sensors/creative_camera.urdf.xacro (robot description, xacro)
@@ -1,5 +1,5 @@
 <?xml version="1.0"?>
 <root xmlns:xacro="http://ros.org/wiki/xacro">
-  <xacro:macro name="creative_camera" params="parent *origin">
+  <xacro:macro name="sensor_creative_camera" params="parent *origin">
     <joint name="${parent}_creative_camera_joint" type="fixed">
       <xacro:insert_block name="origin" />
@@ -14,4 +14,12 @@
         </geometry>
       </visual>
+      <!--
+      <collision>
+      	<origin xyz="0.0 0.0 0.0" rpy="0 0 0" />
+        <geometry>
+        	<box size="0.0830 .2760 0.0720" />
+      	</geometry>
+      </collision>
+      -->
     </link>
   </xacro:macro>

Commit message: Updated Collision Model

File: carl_description/urdf/carl_base/carl_creative_camera_mount.urdf.xacro (robot description, xacro)
@@ -5,5 +5,4 @@
        xmlns:xacro="http://ros.org/wiki/xacro">
   <xacro:include filename="$(find carl_description)/urdf/sensors/creative_camera.urdf.xacro" />
-  <!-- TODO FIX COLLISISION MODEL -->
   <xacro:macro name="carl_creative_camera_mount">
     <link name="creative_mount_link">
@@ -14,11 +13,4 @@
         </geometry>
       </visual>
-	  <!--<collision>
-        <origin xyz="-0.0127 0 0" rpy="0 0 0" />
-        <geometry>
-          <box size="0.027 0.454 0.054" />
-         </geometry>
-      </collision>
-      -->
     </link>
     <link name="creative_servo_link">
@@ -57,12 +49,4 @@
         </geometry>
       </visual>
-      <!--
-	  <collision>
-        <origin xyz="0 -0.01 -0.02" rpy="0 0 0" />
-        <geometry>
-          <box size="0.035 0.05 0.06" />
-         </geometry>
-      </collision>
-      -->
     </link>
     <xacro:sensor_creative_camera parent="creative_plate_link">

File: carl_description/urdf/sensors/creative_camera.urdf.xacro (robot description, xacro)
@@ -14,12 +14,10 @@
         </geometry>
       </visual>
-      <!--
       <collision>
-      	<origin xyz="0.0 0.0 0.0" rpy="0 0 0" />
+      	<origin xyz="0.0 0.0 0.0" rpy="0 0 1.5708" />
         <geometry>
-        	<box size="0.0830 .2760 0.0720" />
+        	<box size="0.04 .14 0.04" />
       	</geometry>
       </collision>
-      -->
     </link>
   </xacro:macro>
