Commit message: Added meshes for creative camera

File: carl_description/urdf/carl_base/carl_asus_camera_mount.urdf.xacro (robot description, xacro)
@@ -5,6 +5,6 @@
        xmlns:xacro="http://ros.org/wiki/xacro">
   <xacro:include filename="$(find carl_description)/urdf/sensors/asus_xtion_pro.urdf.xacro" />
-  <xacro:macro name="carl_camera_mount">
-    <link name="camera_lift_link">
+  <xacro:macro name="carl_asus_camera_mount">
+    <link name="asus_lift_link">
       <visual>
         <origin xyz="0 0 0" rpy="0 1.5708 1.5708" />
@@ -20,5 +20,5 @@
       </collision>
     </link>
-    <link name="camera_mount_link">
+    <link name="asus_mount_link">
       <visual>
         <origin xyz="0 0 0" rpy="0 1.5708 0" />
@@ -28,5 +28,5 @@
       </visual>
     </link>
-    <link name="servo_mount_link">
+    <link name="asus_servo_mount_link">
       <visual>
         <origin xyz="0 0 0" rpy="0 0 0" />
@@ -42,5 +42,5 @@
       </collision>
     </link>
-    <link name="servo_link">
+    <link name="asus_servo_link">
       <visual>
         <origin xyz="0 0 0" rpy="0 0 0" />
@@ -56,5 +56,5 @@
       </collision>
     </link>
-    <link name="servo_arm_link">
+    <link name="asus_servo_arm_link">
       <visual>
         <origin xyz="0 0 0" rpy="0 0 0" />
@@ -70,32 +70,32 @@
       </collision>
     </link>
-    <xacro:sensor_asus_xtion_pro parent="camera_mount_link">
+    <xacro:sensor_asus_xtion_pro parent="asus_mount_link">
       <origin xyz="-0.016 -0.008 0.018" rpy="0 -1.5708 0" />
     </xacro:sensor_asus_xtion_pro>
-    <joint name="right_rear_strut_camera_lift_joint" type="fixed">
+    <joint name="right_rear_strut_asus_lift_joint" type="fixed">
       <parent link="right_rear_strut_link" />
-      <child link="camera_lift_link" />
+      <child link="asus_lift_link" />
       <origin xyz="-0.013 -0.20 1.538" rpy="0 0 3.1415926536" />
     </joint>
-    <joint name="camera_lift_servo_mount_joint" type="fixed">
-      <parent link="camera_lift_link" />
-      <child link="servo_mount_link" />
+    <joint name="asus_lift_asus_servo_mount_joint" type="fixed">
+      <parent link="asus_lift_link" />
+      <child link="asus_servo_mount_link" />
       <origin xyz="0 0 0" rpy="1.5708 0 0" />
       <axis xyz="0 0 1" />
     </joint>
-    <joint name="servo_mount_servo_joint" type="fixed">
-      <parent link="servo_mount_link" />
-      <child link="servo_link" />
+    <joint name="asus_servo_mount_asus_servo_joint" type="fixed">
+      <parent link="asus_servo_mount_link" />
+      <child link="asus_servo_link" />
       <origin xyz="0.073 0.013 0.0187" rpy="1.5708 0 3.92699" />
     </joint>
-    <joint name="servo_servo_arm_joint" type="continuous">
-      <parent link="servo_link" />
-      <child link="servo_arm_link" />
+    <joint name="asus_servo_asus_servo_arm_joint" type="continuous">
+      <parent link="asus_servo_link" />
+      <child link="asus_servo_arm_link" />
       <origin xyz="0 -0.042 0" rpy="1.5708 1.5708 0" />
       <axis xyz="0 0 1" />
     </joint>
-    <joint name="servo_arm_camera_mount_joint" type="fixed">
-      <parent link="servo_arm_link" />
-      <child link="camera_mount_link" />
+    <joint name="asus_servo_arm_asus_mount_joint" type="fixed">
+      <parent link="asus_servo_arm_link" />
+      <child link="asus_mount_link" />
       <origin xyz="0 -0.053 -0.016" rpy="1.5708 0 1.5708" />
     </joint>

File: carl_description/urdf/carl_base/carl_base.urdf.xacro (robot description, xacro)
@@ -9,8 +9,10 @@
   <xacro:include filename="$(find carl_description)/urdf/carl_base/carl_superstructure.urdf.xacro" />
   <xacro:include filename="$(find carl_description)/urdf/carl_base/carl_covers.urdf.xacro" />
-  <xacro:include filename="$(find carl_description)/urdf/carl_base/carl_camera_mount.urdf.xacro" />
+  <xacro:include filename="$(find carl_description)/urdf/carl_base/carl_asus_camera_mount.urdf.xacro" />
+  <xacro:include filename="$(find carl_description)/urdf/carl_base/carl_creative_camera_mount.urdf.xacro" />
   <xacro:macro name="carl_base" params="name">
     <xacro:carl_superstructure />
-    <xacro:carl_camera_mount />
+    <xacro:carl_asus_camera_mount />
+    <xacro:carl_creative_camera_mount />
     <xacro:carl_covers name="${name}" />
     <!-- base footprint -->

Commit message: added calibration files for the asus

File: carl_description/urdf/carl_base/carl_asus_camera_mount.urdf.xacro (robot description, xacro)
@@ -72,5 +72,5 @@
     <xacro:sensor_asus_xtion_pro parent="asus_mount_link">
       <!-- <origin xyz="-0.016 -0.008 0.018" rpy="0 -1.5708 0" /> -->
-      <origin xyz="-0.016 -0.008 0.018" rpy="0 -1.53 0" />
+      <origin xyz="-0.016 -0.008 0.018" rpy="0 -1.54 0" />
     </xacro:sensor_asus_xtion_pro>
     <joint name="right_rear_strut_asus_lift_joint" type="fixed">

Commit message: new collision test

File: carl_description/urdf/carl_base/carl_asus_camera_mount.urdf.xacro (robot description, xacro)
@@ -13,9 +13,9 @@
         </geometry>
       </visual>
-	  <collision>
-        <origin xyz="-0.0127 0 0" rpy="0 0 0" />
+      <collision>
+        <origin xyz="0 0 0" rpy="0 1.5708 1.5708" />
         <geometry>
-          <box size="0.027 0.454 0.054" />
-         </geometry>
+          <mesh filename="package://carl_description/meshes/camera_lift.min.dae" />
+        </geometry>
       </collision>
     </link>
@@ -27,4 +27,10 @@
         </geometry>
       </visual>
+      <collision>
+        <origin xyz="0 0 0" rpy="0 1.5708 0" />
+        <geometry>
+          <mesh filename="package://carl_description/meshes/camera_mount.min.dae" />
+        </geometry>
+      </collision>
     </link>
     <link name="asus_servo_mount_link">
@@ -35,9 +41,9 @@
         </geometry>
       </visual>
-	  <collision>
-        <origin xyz="0.023 0 0" rpy="0 0 0" />
+      <collision>
+        <origin xyz="0 0 0" rpy="0 0 0" />
         <geometry>
-          <box size="0.08 0.055 0.09" />
-         </geometry>
+          <mesh filename="package://carl_description/meshes/servo_mount.min.dae" />
+        </geometry>
       </collision>
     </link>
@@ -49,9 +55,9 @@
         </geometry>
       </visual>
-	  <collision>
-        <origin xyz="0.01 -0.021 0" rpy="0 0 0" />
+      <collision>
+        <origin xyz="0 0 0" rpy="0 0 0" />
         <geometry>
-          <box size="0.06 0.05 0.035" />
-         </geometry>
+          <mesh filename="package://carl_description/meshes/servo.min.dae" />
+        </geometry>
       </collision>
     </link>
@@ -63,9 +69,9 @@
         </geometry>
       </visual>
-	  <collision>
-        <origin xyz="0 -0.01 -0.02" rpy="0 0 0" />
+      <collision>
+        <origin xyz="0 0 0" rpy="0 0 0" />
         <geometry>
-          <box size="0.035 0.05 0.06" />
-         </geometry>
+          <mesh filename="package://carl_description/meshes/servo_arm.min.dae" />
+        </geometry>
       </collision>
     </link>

File: carl_description/urdf/carl_base/carl_base.urdf.xacro (robot description, xacro)
@@ -26,4 +26,10 @@
         </geometry>
       </visual>
+     <collision>
+        <origin xyz="0 0 0" rpy="0 0 0" />
+        <geometry>
+          <mesh filename="package://carl_description/meshes/base.min.dae" />
+        </geometry>
+      </collision>
     </link>
     <joint name="${name}_footprint_${name}_link_joint" type="fixed">

File: carl_description/urdf/carl_base/carl_covers.urdf.xacro (robot description, xacro)
@@ -32,7 +32,7 @@
       </visual>
       <collision>
-        <origin xyz="-.245 0 -.241" rpy="0 0 0" />
+        <origin xyz="0 0 0" rpy="0 0 1.5708" />
         <geometry>
-          <mesh filename="package://carl_description/meshes/front_cover_collision.stl" />
+          <mesh filename="package://carl_description/meshes/front_cover.min.dae" />
         </geometry>
       </collision>
@@ -42,8 +42,15 @@
         <origin xyz="0 0 0" rpy="0 0 0" />
         <geometry>
-      	  <!--<box size="0.005 0.45 0.6" />-->
-      	  <mesh filename="package://carl_description/meshes/back_cover.min.dae" />
+          <!--<box size="0.005 0.45 0.6" />-->
+          <mesh filename="package://carl_description/meshes/back_cover.min.dae" />
         </geometry>
       </visual>
+      <collision>
+        <origin xyz="0 0 0" rpy="0 0 0" />
+        <geometry>
+          <!--<box size="0.005 0.45 0.6" />-->
+          <mesh filename="package://carl_description/meshes/back_cover.min.dae" />
+        </geometry>
+      </collision>
     </link>
   </xacro:macro>

File: carl_description/urdf/carl_base/carl_creative_camera_mount.urdf.xacro (robot description, xacro)
@@ -13,4 +13,10 @@
         </geometry>
       </visual>
+      <collision>
+        <origin xyz="0 0 0" rpy="0 0 0" />
+        <geometry>
+          <mesh filename="package://carl_description/meshes/creative_mount.min.dae" />
+        </geometry>
+      </collision>
     </link>
     <link name="creative_servo_link">
@@ -21,9 +27,9 @@
         </geometry>
       </visual>
-	  <collision>
-        <origin xyz="0.01 -0.021 0" rpy="0 0 0" />
+      <collision>
+        <origin xyz="0 0 0" rpy="0 0 0" />
         <geometry>
-          <box size="0.06 0.05 0.035" />
-         </geometry>
+          <mesh filename="package://carl_description/meshes/servo.min.dae" />
+        </geometry>
       </collision>
     </link>
@@ -35,9 +41,9 @@
         </geometry>
       </visual>
-	  <collision>
-        <origin xyz="0 -0.01 -0.02" rpy="0 0 0" />
+      <collision>
+        <origin xyz="0 0 0" rpy="0 0 0" />
         <geometry>
-          <box size="0.035 0.09 0.06" />
-         </geometry>
+          <mesh filename="package://carl_description/meshes/servo_arm.min.dae" />
+        </geometry>
       </collision>
     </link>
@@ -49,4 +55,10 @@
         </geometry>
       </visual>
+      <collision>
+        <origin xyz="0 0 0" rpy="0 0 0" />
+        <geometry>
+          <mesh filename="package://carl_description/meshes/creative_plate.min.dae" />
+        </geometry>
+      </collision>
     </link>
     <xacro:sensor_creative_camera parent="creative_plate_link">

File: carl_description/urdf/carl_base/carl_superstructure.urdf.xacro (robot description, xacro)
@@ -32,7 +32,7 @@
       </visual>
       <collision>
-        <origin xyz="-.29 0 -0.299" rpy="0 0 3.1415926536" />
+        <origin xyz="0 0 0" rpy="0 0 -1.5708" />
         <geometry>
-          <box size="0.495 0.59 0.65" />
+          <mesh filename="package://carl_description/meshes/table_plate.min.dae" />
         </geometry>
       </collision>
@@ -45,4 +45,10 @@
         </geometry>
       </visual>
+      <collision>
+        <origin xyz="0 0 0" rpy="0 0 1.5708" />
+        <geometry>
+          <mesh filename="package://carl_description/meshes/jaco_mount.min.dae" />
+        </geometry>
+      </collision>
     </link>
   </xacro:macro>

File: carl_description/urdf/components/carl_caster_assembly.urdf.xacro (robot description, xacro)
@@ -20,4 +20,10 @@
         </geometry>
       </visual>
+      <collision>
+        <origin xyz="0 0 0" rpy="0 0 1.5708" />
+        <geometry>
+          <mesh filename="package://carl_description/meshes/caster_plate.min.dae" />
+        </geometry>
+      </collision>
     </link>
     <link name="caster_link">
@@ -29,8 +35,8 @@
       </visual>
       <collision>
-        <origin xyz="0 0 -0.09" rpy="0 0 0" />
+        <origin xyz="0 0 0" rpy="0 0 0" />
         <geometry>
-          <cylinder radius="0.116" length="0.213" />
-         </geometry>
+          <mesh filename="package://carl_description/meshes/caster.min.dae" />
+        </geometry>
       </collision>
     </link>

File: carl_description/urdf/components/carl_rear_strut.urdf.xacro (robot description, xacro)
@@ -20,8 +20,8 @@
       </visual>
       <collision>
-        <origin xyz="0 0 0.5275" rpy="0 0 0" />
+        <origin xyz="0 0 0" rpy="0 0 -1.5708" />
         <geometry>
-          <box size="0.027 0.054 1.055" />
-         </geometry>
+          <mesh filename="package://carl_description/meshes/rear_strut.min.dae" />
+        </geometry>
       </collision>
     </link>
@@ -34,8 +34,8 @@
       </visual>
       <collision>
-        <origin xyz="0 -0.001 0.2285" rpy="0 0 0" />
+        <origin xyz="0 0 0" rpy="0 0 -1.5708" />
         <geometry>
-          <box size="0.027 0.054 0.4575" />
-         </geometry>
+          <mesh filename="package://carl_description/meshes/rear_strut_top.min.dae" />
+        </geometry>
       </collision>
     </link>

File: carl_description/urdf/components/carl_side_cover.urdf.xacro (robot description, xacro)
@@ -14,4 +14,10 @@
         </geometry>
       </visual>
+      <collision>
+        <origin xyz="0 0 0" rpy="0 0 1.5708" />
+        <geometry>
+          <mesh filename="package://carl_description/meshes/side_cover.min.dae" />
+        </geometry>
+      </collision>
     </link>
   </xacro:macro>

File: carl_description/urdf/components/carl_wheel.urdf.xacro (robot description, xacro)
@@ -16,7 +16,7 @@
       </visual>
       <collision>
-        <origin xyz="0 0 .025" rpy="0 0 0" />
+        <origin xyz="0 0 0" rpy="0 0 0" />
         <geometry>
-          <cylinder radius="0.25" length="0.1" />
+          <mesh filename="package://carl_description/meshes/wheel.min.dae" />
         </geometry>
       </collision>

File: carl_description/urdf/sensors/asus_xtion_pro.urdf.xacro (robot description, xacro)
@@ -25,7 +25,7 @@
     </visual>
     <collision>
-      <origin xyz="0.0 0.0 0.0" rpy="0 0 0" />
+      <origin xyz=" 0 0 0 " rpy="${-M_PI/2} -${M_PI} ${-M_PI/2}" />
       <geometry>
-        <box size="0.0730 .2760 0.0720"/>
+        <mesh filename="package://carl_description/meshes/asus_xtion_pro_live.min.dae" scale="${M_SCALE} ${M_SCALE} ${M_SCALE}" />
       </geometry>
     </collision>

File: carl_description/urdf/sensors/creative_camera.urdf.xacro (robot description, xacro)
@@ -15,8 +15,8 @@
       </visual>
       <collision>
-      	<origin xyz="0.0 0.0 0.0" rpy="0 0 1.5708" />
+        <origin xyz="0 0 0" rpy="0 0 0" />
         <geometry>
-        	<box size="0.04 .14 0.04" />
-      	</geometry>
+          <mesh filename="package://carl_description/meshes/creative_camera.min.dae" />
+        </geometry>
       </collision>
     </link>

File: carl_description/urdf/sensors/hokuyo.urdf.xacro (robot description, xacro)
@@ -14,4 +14,10 @@
         </geometry>
       </visual>
+      <collision>
+        <origin xyz="0 0 0" rpy="0 0 0" />
+        <geometry>
+          <mesh filename="package://carl_description/meshes/hokuyo.min.dae" />
+        </geometry>
+      </collision>
     </link>
   </xacro:macro>
