Commit message: Refactoring.

File: carl_description/urdf/carl_base/carl_base.urdf.xacro (robot description, xacro)
@@ -5,9 +5,11 @@
         xmlns:xacro="http://ros.org/wiki/xacro">
 <xacro:include filename="$(find carl_description)/urdf/components/carl_wheel.urdf.xacro" />
-<xacro:include filename="$(find carl_description)/urdf/components/carl_rear_strut.urdf.xacro" />
 <xacro:include filename="$(find carl_description)/urdf/components/carl_caster_assembly.urdf.xacro" />
-<xacro:include filename="$(find carl_description)/urdf/components/carl_side_cover.urdf.xacro" />
 <xacro:include filename="$(find carl_description)/urdf/sensors/hokuyo.urdf.xacro" />
+<xacro:include filename="$(find carl_description)/urdf/carl_base/carl_superstructure.urdf.xacro" />
+<xacro:include filename="$(find carl_description)/urdf/carl_base/carl_covers.urdf.xacro" />
 <xacro:macro name="carl_base" params="name">
+  <xacro:carl_superstructure/>
+  <xacro:carl_covers name="${name}"/>
   <link name="${name}_link">
    <visual>
@@ -17,18 +19,4 @@
       </geometry>
     </visual>
-  </link>
-  <link name="top_plate_link">
-    <visual>
-      <origin xyz="0 0 0" rpy="0 0 -1.5708" />
-      <geometry>
-        <mesh filename="package://carl_description/meshes/table_plate.dae" />
-      </geometry>
-    </visual>
-    <collision>
-      <origin xyz="-.29 0 -0.299" rpy="0 0 0" />
-      <geometry>
-        <box size="0.495 0.59 0.65" />
-      </geometry>
-    </collision>
   </link>
   <link name="CameraLift_link">
@@ -63,35 +51,4 @@
     </collision>
   </link>
-  <link name="jaco_mount_link">
-    <visual>
-      <origin xyz="0 0 0" rpy="0 0 1.5708" />
-      <geometry>
-        <mesh filename="package://carl_description/meshes/jaco_mount.dae" />
-      </geometry>
-    </visual>
-  </link>
-  <link name="FrontCover_link">
-    <visual>
-      <origin xyz="0 0 0" rpy="0 0 1.5708" />
-      <geometry>
-        <mesh filename="package://carl_description/meshes/front_cover.dae" />
-      </geometry>
-    </visual>
-    <collision>
-      <origin xyz="-.245 0 -.241" rpy="0 0 0" />
-      <geometry>
-        <mesh filename="package://carl_description/meshes/front_cover_collision.stl" />
-      </geometry>
-    </collision>
-  </link>
-  <link name="BackCover_link">
-    <visual>
-      <origin xyz="0 0 0" rpy="0 0 0" />
-      <geometry>
-      	<!--<box size="0.005 0.45 0.6" />-->
-      	<mesh filename="package://carl_description/meshes/back_cover.dae" />
-      </geometry>
-    </visual>
-  </link>
    <!-- left wheel -->
    <xacro:carl_wheel suffix="left" parent="${name}_link">
@@ -106,17 +63,4 @@
      <origin xyz="0.2883 0 0" rpy="0 0 0" />
    </xacro:carl_caster_assembly>
-   <!-- left rear strut -->
-   <xacro:carl_rear_strut suffix="left" parent="${name}_link">
-     <origin xyz="-0.222 0.200 -0.102" rpy="0 0 0" />
-   </xacro:carl_rear_strut>
-   <!-- right rear strut -->
-   <xacro:carl_rear_strut suffix="right" parent="${name}_link">
-     <origin xyz="-0.222 -0.200 -0.102" rpy="0 0 0" />
-   </xacro:carl_rear_strut>
-  <joint name="left_rear_strut_top_plate_joint" type="fixed">
-    <parent link="right_rear_strut_link"/>
-    <child link="top_plate_link"/>
-    <origin xyz="0.516 0.20 0.598" rpy="0 0 0" />
-  </joint>
   <joint name="RearLeftStrutToCameraLift" type="fixed">
     <parent link="right_rear_strut_link"/>
@@ -124,5 +68,5 @@
     <origin xyz="0.01 0.20 1.461" rpy="0 0 0" />
   </joint>
-    <joint name="CameraLiftToCameraTiltBracket" type="continuous">
+  <joint name="CameraLiftToCameraTiltBracket" type="continuous">
     <parent link="CameraLift_link"/>
     <child link="CameraTiltBracket_link"/>
@@ -135,31 +79,8 @@
     <origin xyz="0.11 0 -0.10" rpy="0 0 0" />
   </joint>
-  <joint name="top_plate_jaco_mount" type="fixed">
-    <parent link="top_plate_link"/>
-    <child link="jaco_mount_link"/>
-    <origin xyz="0 0 -0.13" rpy="0 0 0" />
-  </joint>
    <!-- hokuyo -->
    <xacro:hokuyo parent="caster_plate_link">
      <origin xyz="0.07 0 0.035" rpy="0 0 0" />
    </xacro:hokuyo>
-   <!-- right side cover -->
-   <xacro:carl_side_cover suffix="right" parent="right_rear_strut_link">
-     <origin xyz="0.229 -0.026 0.447" rpy="0 0 0" />
-   </xacro:carl_side_cover>
-   <!-- left side cover -->
-   <xacro:carl_side_cover suffix="left" parent="left_rear_strut_link">
-     <origin xyz="0.229 -0.026 0.447" rpy="0 0 0" />
-   </xacro:carl_side_cover>
-  <joint name="${name}_front_cover_joint" type="fixed">
-    <parent link="${name}_link"/>
-    <child link="FrontCover_link"/>
-    <origin xyz=".247 0 0.242" rpy="0 0 0" />
-  </joint>
-  <joint name="${name}_back_cover" type="fixed">
-    <parent link="${name}_link"/>
-    <child link="BackCover_link"/>
-    <origin xyz="-.237 0 -0.102" rpy="0 0 0" />
-  </joint>
 </xacro:macro>
 </robot>

Commit message: Refactoring

File: carl_description/urdf/carl_base/carl_base.urdf.xacro (robot description, xacro)
@@ -22,20 +22,20 @@
       </visual>
     </link>
-     <!-- left wheel -->
-     <xacro:carl_wheel suffix="left" parent="${name}_link">
-       <origin xyz="0 0.25 0" rpy="-1.5708 0 0" />
-     </xacro:carl_wheel>
-     <!-- right wheel -->
-     <xacro:carl_wheel suffix="right" parent="${name}_link">
-       <origin xyz="0 -0.25 0" rpy="1.5708 0 0" />
-     </xacro:carl_wheel>
-     <!-- caster assembly -->
-     <xacro:carl_caster_assembly parent="${name}_link">
-       <origin xyz="0.2883 0 0" rpy="0 0 0" />
-     </xacro:carl_caster_assembly>
-     <!-- hokuyo -->
-     <xacro:hokuyo parent="caster_plate_link">
-       <origin xyz="0.07 0 0.035" rpy="0 0 0" />
-     </xacro:hokuyo>
+    <!-- left wheel -->
+    <xacro:carl_wheel suffix="left" parent="${name}_link">
+      <origin xyz="0 0.25 0" rpy="-1.5708 0 0" />
+    </xacro:carl_wheel>
+    <!-- right wheel -->
+    <xacro:carl_wheel suffix="right" parent="${name}_link">
+      <origin xyz="0 -0.25 0" rpy="1.5708 0 0" />
+    </xacro:carl_wheel>
+    <!-- caster assembly -->
+    <xacro:carl_caster_assembly parent="${name}_link">
+      <origin xyz="0.2883 0 0" rpy="0 0 0" />
+    </xacro:carl_caster_assembly>
+    <!-- hokuyo -->
+    <xacro:hokuyo parent="caster_plate_link">
+      <origin xyz="0.07 0 0.035" rpy="0 0 0" />
+    </xacro:hokuyo>
   </xacro:macro>
 </robot>

File: carl_description/urdf/components/carl_rear_strut.urdf.xacro (robot description, xacro)
@@ -1,4 +1,4 @@
 <?xml version="1.0"?>
-  <root xmlns:xacro="http://ros.org/wiki/xacro">
+<root xmlns:xacro="http://ros.org/wiki/xacro">
   <xacro:macro name="carl_rear_strut" params="suffix parent *origin">
     <joint name="${parent}_${suffix}_rear_strut_joint" type="fixed">
@@ -8,16 +8,16 @@
     </joint>
     <joint name="${suffix}_rear_strut_link_${suffix}_rear_strut_link_inside_joint" type="fixed">
-    	<parent link="${suffix}_rear_strut_link"/>
-    	<child link="${suffix}_rear_strut_inside_link"/>
-    	<origin xyz="0 0 0" rpy="0 0 0" />
-  	</joint>
+      <parent link="${suffix}_rear_strut_link"/>
+   	  <child link="${suffix}_rear_strut_inside_link"/>
+      <origin xyz="0 0 0" rpy="0 0 0" />
+    </joint>
     <link name="${suffix}_rear_strut_inside_link">
-    <visual>
-     <origin xyz="0 0 0.5275" rpy="0 0 0" />
-      <geometry>
-        <box size="0.02 0.045 1" />
-      </geometry>
-    </visual>
- 	</link>
+      <visual>
+        <origin xyz="0 0 0.5275" rpy="0 0 0" />
+        <geometry>
+          <box size="0.02 0.045 1" />
+        </geometry>
+      </visual>
+    </link>
     <link name="${suffix}_rear_strut_link">
       <visual>

Commit message: Added transform to base_footprint

File: carl_description/urdf/carl_base/carl_base.urdf.xacro (robot description, xacro)
@@ -14,4 +14,5 @@
     <xacro:carl_camera_mount/>
     <xacro:carl_covers name="${name}"/>
+  	<!-- base link -->
     <link name="${name}_link">
      <visual>
@@ -22,4 +23,11 @@
       </visual>
     </link>
+    <!-- base footprint -->
+    <link name="${name}_footprint"/>
+    <joint name="${name}_link_${name}_footprint_joint" type="fixed">
+      <parent link="${name}_link"/>
+      <child link="${name}_footprint"/>
+      <origin xyz="0 0 -0.23114" rpy="0 0 0" />
+    </joint>
     <!-- left wheel -->
     <xacro:carl_wheel suffix="left" parent="${name}_link">

Commit message: Fixed base_footprint tf

File: carl_description/urdf/carl_base/carl_base.urdf.xacro (robot description, xacro)
@@ -14,4 +14,6 @@
     <xacro:carl_camera_mount/>
     <xacro:carl_covers name="${name}"/>
+    <!-- base footprint -->
+    <link name="${name}_footprint"/>
   	<!-- base link -->
     <link name="${name}_link">
@@ -23,10 +25,8 @@
       </visual>
     </link>
-    <!-- base footprint -->
-    <link name="${name}_footprint"/>
-    <joint name="${name}_link_${name}_footprint_joint" type="fixed">
-      <parent link="${name}_link"/>
-      <child link="${name}_footprint"/>
-      <origin xyz="0 0 -0.23114" rpy="0 0 0" />
+    <joint name="${name}_footprint_${name}_link_joint" type="fixed">
+      <parent link="${name}_footprint"/>
+      <child link="${name}_link"/>
+      <origin xyz="0 0 0.23114" rpy="0 0 0" />
     </joint>
     <!-- left wheel -->

Commit message: minified XML in Collada modles

File: carl_description/urdf/carl_base/carl_base.urdf.xacro (robot description, xacro)
@@ -21,5 +21,5 @@
         <origin xyz="0 0 0" rpy="0 0 0" />
         <geometry>
-          <mesh filename="package://carl_description/meshes/base.dae" />
+          <mesh filename="package://carl_description/meshes/base.min.dae" />
         </geometry>
       </visual>

File: carl_description/urdf/carl_base/carl_camera_mount.urdf.xacro (robot description, xacro)
@@ -10,5 +10,5 @@
         <origin xyz="0 0 0" rpy="0 1.5708 1.5708" />
         <geometry>
-          <mesh filename="package://carl_description/meshes/camera_lift.dae" />
+          <mesh filename="package://carl_description/meshes/camera_lift.min.dae" />
         </geometry>
       </visual>
@@ -24,5 +24,5 @@
         <origin xyz="0 0 0" rpy="0 1.5708 0" />
         <geometry>
-          <mesh filename="package://carl_description/meshes/camera_mount.dae" />
+          <mesh filename="package://carl_description/meshes/camera_mount.min.dae" />
         </geometry>
       </visual>
@@ -32,5 +32,5 @@
         <origin xyz="0 0 0" rpy="0 0 0" />
         <geometry>
-          <mesh filename="package://carl_description/meshes/servo_mount.dae" />
+          <mesh filename="package://carl_description/meshes/servo_mount.min.dae" />
         </geometry>
       </visual>
@@ -46,5 +46,5 @@
         <origin xyz="0 0 0" rpy="0 0 0" />
         <geometry>
-          <mesh filename="package://carl_description/meshes/servo.dae" />
+          <mesh filename="package://carl_description/meshes/servo.min.dae" />
         </geometry>
       </visual>
@@ -60,5 +60,5 @@
         <origin xyz="0 0 0" rpy="0 0 0" />
         <geometry>
-          <mesh filename="package://carl_description/meshes/servo_arm.dae" />
+          <mesh filename="package://carl_description/meshes/servo_arm.min.dae" />
         </geometry>
       </visual>

File: carl_description/urdf/carl_base/carl_covers.urdf.xacro (robot description, xacro)
@@ -28,5 +28,5 @@
         <origin xyz="0 0 0" rpy="0 0 1.5708" />
         <geometry>
-          <mesh filename="package://carl_description/meshes/front_cover.dae" />
+          <mesh filename="package://carl_description/meshes/front_cover.min.dae" />
         </geometry>
       </visual>
@@ -43,5 +43,5 @@
         <geometry>
       	  <!--<box size="0.005 0.45 0.6" />-->
-      	  <mesh filename="package://carl_description/meshes/back_cover.dae" />
+      	  <mesh filename="package://carl_description/meshes/back_cover.min.dae" />
         </geometry>
       </visual>

File: carl_description/urdf/carl_base/carl_superstructure.urdf.xacro (robot description, xacro)
@@ -28,5 +28,5 @@
         <origin xyz="0 0 0" rpy="0 0 -1.5708" />
         <geometry>
-          <mesh filename="package://carl_description/meshes/table_plate.dae" />
+          <mesh filename="package://carl_description/meshes/table_plate.min.dae" />
         </geometry>
       </visual>
@@ -42,5 +42,5 @@
         <origin xyz="0 0 0" rpy="0 0 1.5708" />
         <geometry>
-          <mesh filename="package://carl_description/meshes/jaco_mount.dae" />
+          <mesh filename="package://carl_description/meshes/jaco_mount.min.dae" />
         </geometry>
       </visual>

File: carl_description/urdf/components/carl_caster_assembly.urdf.xacro (robot description, xacro)
@@ -17,5 +17,5 @@
         <origin xyz="0 0 0" rpy="0 0 1.5708" />
         <geometry>
-          <mesh filename="package://carl_description/meshes/caster_plate.dae" />
+          <mesh filename="package://carl_description/meshes/caster_plate.min.dae" />
         </geometry>
       </visual>
@@ -25,5 +25,5 @@
         <origin xyz="0 0 0" rpy="0 0 0" />
         <geometry>
-          <mesh filename="package://carl_description/meshes/caster.dae" />
+          <mesh filename="package://carl_description/meshes/caster.min.dae" />
         </geometry>
       </visual>

File: carl_description/urdf/components/carl_rear_strut.urdf.xacro (robot description, xacro)
@@ -29,5 +29,5 @@
         <origin xyz="0 0 0" rpy="0 0 -1.5708" />
         <geometry>
-          <mesh filename="package://carl_description/meshes/rear_strut.dae" />
+          <mesh filename="package://carl_description/meshes/rear_strut.min.dae" />
         </geometry>
       </visual>
@@ -43,5 +43,5 @@
         <origin xyz="0 0 0" rpy="0 0 -1.5708" />
         <geometry>
-          <mesh filename="package://carl_description/meshes/rear_strut_top.dae" />
+          <mesh filename="package://carl_description/meshes/rear_strut_top.min.dae" />
         </geometry>
       </visual>

File: carl_description/urdf/components/carl_side_cover.urdf.xacro (robot description, xacro)
@@ -11,5 +11,5 @@
         <origin xyz="0 0 0" rpy="0 0 1.5708" />
         <geometry>
-          <mesh filename="package://carl_description/meshes/side_cover.dae" />
+          <mesh filename="package://carl_description/meshes/side_cover.min.dae" />
         </geometry>
       </visual>

File: carl_description/urdf/components/carl_wheel.urdf.xacro (robot description, xacro)
@@ -12,5 +12,5 @@
         <origin xyz="0 0 0" rpy="0 0 0" />
         <geometry>
-          <mesh filename="package://carl_description/meshes/wheel.dae" />
+          <mesh filename="package://carl_description/meshes/wheel.min.dae" />
         </geometry>
       </visual>

File: carl_description/urdf/sensors/asus_xtion_pro.urdf.xacro (robot description, xacro)
@@ -16,5 +16,5 @@
         <origin xyz="-0.01 0 0" rpy="${-M_PI/2} -${M_PI} ${-M_PI/2}" />
         <geometry>
-          <mesh filename="package://carl_description/meshes/asus_xtion_pro_live.dae" scale="${M_SCALE} ${M_SCALE} ${M_SCALE}" />
+          <mesh filename="package://carl_description/meshes/asus_xtion_pro_live.min.dae" scale="${M_SCALE} ${M_SCALE} ${M_SCALE}" />
         </geometry>
       </visual>

File: carl_description/urdf/sensors/hokuyo.urdf.xacro (robot description, xacro)
@@ -11,5 +11,5 @@
         <origin xyz="0 0 0" rpy="0 0 0" />
         <geometry>
-          <mesh filename="package://carl_description/meshes/hokuyo.dae" />
+          <mesh filename="package://carl_description/meshes/hokuyo.min.dae" />
         </geometry>
       </visual>
