Commit message: moved to minified DAE

File: carl_description/urdf/carl_base/carl_base.urdf.xacro (robot description, xacro)
@@ -22,5 +22,5 @@
         <origin xyz="0 0 0" rpy="0 0 0" />
         <geometry>
-          <mesh scale="${M_SCALE} ${M_SCALE} ${M_SCALE}" filename="package://carl_description/meshes/base.dae" />
+          <mesh scale="${M_SCALE} ${M_SCALE} ${M_SCALE}" filename="package://carl_description/meshes/base.min.dae" />
         </geometry>
       </visual>

File: carl_description/urdf/carl_base/carl_covers.urdf.xacro (robot description, xacro)
@@ -19,5 +19,5 @@
         <origin xyz="0 0 0" rpy="0 0 0" />
         <geometry>
-          <mesh scale="${M_SCALE} ${M_SCALE} ${M_SCALE}" filename="package://carl_description/meshes/front_cover.dae" />
+          <mesh scale="${M_SCALE} ${M_SCALE} ${M_SCALE}" filename="package://carl_description/meshes/front_cover.min.dae" />
         </geometry>
       </visual>
@@ -39,5 +39,5 @@
         <origin xyz="0 0 0" rpy="0 0 0" />
         <geometry>
-          <mesh scale="${M_SCALE} ${M_SCALE} ${M_SCALE}" filename="package://carl_description/meshes/back_cover.dae" />
+          <mesh scale="${M_SCALE} ${M_SCALE} ${M_SCALE}" filename="package://carl_description/meshes/back_cover.min.dae" />
         </geometry>
       </visual>

File: carl_description/urdf/carl_base/carl_frame.urdf.xacro (robot description, xacro)
@@ -26,5 +26,5 @@
         <origin xyz="0 0 0" rpy="0 0 -${M_PI/2}" />
         <geometry>
-          <mesh scale="${M_SCALE} ${M_SCALE} ${M_SCALE}" filename="package://carl_description/meshes/top_plate.dae" />
+          <mesh scale="${M_SCALE} ${M_SCALE} ${M_SCALE}" filename="package://carl_description/meshes/top_plate.min.dae" />
         </geometry>
       </visual>
@@ -46,5 +46,5 @@
         <origin xyz="0 0 0" rpy="0 0 0" />
         <geometry>
-          <mesh scale="${M_SCALE} ${M_SCALE} ${M_SCALE}" filename="package://carl_description/meshes/jaco_mount.dae" />
+          <mesh scale="${M_SCALE} ${M_SCALE} ${M_SCALE}" filename="package://carl_description/meshes/jaco_mount.min.dae" />
         </geometry>
       </visual>
@@ -66,5 +66,5 @@
         <origin xyz="0 0 0" rpy="0 ${M_PI/2} ${M_PI/2}" />
         <geometry>
-          <mesh scale="${M_SCALE} ${M_SCALE} ${M_SCALE}" filename="package://carl_description/meshes/camera_lift.dae" />
+          <mesh scale="${M_SCALE} ${M_SCALE} ${M_SCALE}" filename="package://carl_description/meshes/camera_lift.min.dae" />
         </geometry>
       </visual>

File: carl_description/urdf/components/carl_asus_camera.urdf.xacro (robot description, xacro)
@@ -19,5 +19,5 @@
         <origin xyz="0 0 0" rpy="0 0 0" />
         <geometry>
-          <mesh scale="${M_SCALE} ${M_SCALE} ${M_SCALE}" filename="package://carl_description/meshes/servo_mount.dae" />
+          <mesh scale="${M_SCALE} ${M_SCALE} ${M_SCALE}" filename="package://carl_description/meshes/servo_mount.min.dae" />
         </geometry>
       </visual>
@@ -38,5 +38,5 @@
         <origin xyz="0 0 0" rpy="0 0 0" />
         <geometry>
-          <mesh scale="${M_SCALE} ${M_SCALE} ${M_SCALE}" filename="package://carl_description/meshes/servo.dae" />
+          <mesh scale="${M_SCALE} ${M_SCALE} ${M_SCALE}" filename="package://carl_description/meshes/servo.min.dae" />
         </geometry>
       </visual>
@@ -58,5 +58,5 @@
         <origin xyz="0 0 0" rpy="0 0 0" />
         <geometry>
-          <mesh scale="${M_SCALE} ${M_SCALE} ${M_SCALE}" filename="package://carl_description/meshes/servo_arm.dae" />
+          <mesh scale="${M_SCALE} ${M_SCALE} ${M_SCALE}" filename="package://carl_description/meshes/servo_arm.min.dae" />
         </geometry>
       </visual>
@@ -77,5 +77,5 @@
         <origin xyz="0 0 0" rpy="0 ${M_PI/2} 0" />
         <geometry>
-          <mesh scale="${M_SCALE} ${M_SCALE} ${M_SCALE}" filename="package://carl_description/meshes/camera_mount.dae" />
+          <mesh scale="${M_SCALE} ${M_SCALE} ${M_SCALE}" filename="package://carl_description/meshes/camera_mount.min.dae" />
         </geometry>
       </visual>

File: carl_description/urdf/components/carl_caster_assembly.urdf.xacro (robot description, xacro)
@@ -17,5 +17,5 @@
         <origin xyz="0 0 0" rpy="0 0 ${M_PI/2}" />
         <geometry>
-          <mesh scale="${M_SCALE} ${M_SCALE} ${M_SCALE}" filename="package://carl_description/meshes/caster_plate.dae" />
+          <mesh scale="${M_SCALE} ${M_SCALE} ${M_SCALE}" filename="package://carl_description/meshes/caster_plate.min.dae" />
         </geometry>
       </visual>
@@ -37,5 +37,5 @@
         <origin xyz="0 0 0" rpy="0 0 0" />
         <geometry>
-          <mesh scale="${M_SCALE} ${M_SCALE} ${M_SCALE}" filename="package://carl_description/meshes/caster.dae" />
+          <mesh scale="${M_SCALE} ${M_SCALE} ${M_SCALE}" filename="package://carl_description/meshes/caster.min.dae" />
         </geometry>
       </visual>

File: carl_description/urdf/components/carl_creative_camera.urdf.xacro (robot description, xacro)
@@ -19,5 +19,5 @@
         <origin xyz="0 0 0" rpy="0 0 0" />
         <geometry>
-          <mesh scale="${M_SCALE} ${M_SCALE} ${M_SCALE}" filename="package://carl_description/meshes/creative_mount.dae" />
+          <mesh scale="${M_SCALE} ${M_SCALE} ${M_SCALE}" filename="package://carl_description/meshes/creative_mount.min.dae" />
         </geometry>
       </visual>
@@ -38,5 +38,5 @@
         <origin xyz="0 0 0" rpy="0 0 0" />
         <geometry>
-          <mesh scale="${M_SCALE} ${M_SCALE} ${M_SCALE}" filename="package://carl_description/meshes/servo.dae" />
+          <mesh scale="${M_SCALE} ${M_SCALE} ${M_SCALE}" filename="package://carl_description/meshes/servo.min.dae" />
         </geometry>
       </visual>
@@ -58,5 +58,5 @@
         <origin xyz="0 0 0" rpy="0 0 0" />
         <geometry>
-          <mesh scale="${M_SCALE} ${M_SCALE} ${M_SCALE}" filename="package://carl_description/meshes/servo_arm.dae" />
+          <mesh scale="${M_SCALE} ${M_SCALE} ${M_SCALE}" filename="package://carl_description/meshes/servo_arm.min.dae" />
         </geometry>
       </visual>
@@ -77,5 +77,5 @@
         <origin xyz="0 0 0" rpy="0 0 0" />
         <geometry>
-          <mesh scale="${M_SCALE} ${M_SCALE} ${M_SCALE}" filename="package://carl_description/meshes/creative_plate.dae" />
+          <mesh scale="${M_SCALE} ${M_SCALE} ${M_SCALE}" filename="package://carl_description/meshes/creative_plate.min.dae" />
         </geometry>
       </visual>

File: carl_description/urdf/components/carl_rear_strut.urdf.xacro (robot description, xacro)
@@ -18,5 +18,5 @@
         <origin xyz="0 0 0" rpy="0 0 -${M_PI/2}" />
         <geometry>
-          <mesh scale="${M_SCALE} ${M_SCALE} ${M_SCALE}" filename="package://carl_description/meshes/rear_strut.dae" />
+          <mesh scale="${M_SCALE} ${M_SCALE} ${M_SCALE}" filename="package://carl_description/meshes/rear_strut.min.dae" />
         </geometry>
       </visual>
@@ -38,5 +38,5 @@
         <origin xyz="0 0 0" rpy="0 0 -${M_PI/2}" />
         <geometry>
-          <mesh scale="${M_SCALE} ${M_SCALE} ${M_SCALE}" filename="package://carl_description/meshes/rear_strut_top.dae" />
+          <mesh scale="${M_SCALE} ${M_SCALE} ${M_SCALE}" filename="package://carl_description/meshes/rear_strut_top.min.dae" />
         </geometry>
       </visual>

File: carl_description/urdf/components/carl_side_cover.urdf.xacro (robot description, xacro)
@@ -16,5 +16,5 @@
         <origin xyz="0 0 0" rpy="0 0 0" />
         <geometry>
-          <mesh scale="${M_SCALE} ${M_SCALE} ${M_SCALE}" filename="package://carl_description/meshes/side_cover.dae" />
+          <mesh scale="${M_SCALE} ${M_SCALE} ${M_SCALE}" filename="package://carl_description/meshes/side_cover.min.dae" />
         </geometry>
       </visual>

File: carl_description/urdf/components/carl_wheel.urdf.xacro (robot description, xacro)
@@ -11,5 +11,5 @@
         <origin xyz="0 0 0" rpy="0 0 0" />
         <geometry>
-          <mesh scale="${M_SCALE} ${M_SCALE} ${M_SCALE}" filename="package://carl_description/meshes/wheel.dae" />
+          <mesh scale="${M_SCALE} ${M_SCALE} ${M_SCALE}" filename="package://carl_description/meshes/wheel.min.dae" />
         </geometry>
       </visual>

File: carl_description/urdf/sensors/asus_xtion_pro.urdf.xacro (robot description, xacro)
@@ -21,5 +21,5 @@
         <origin xyz=" 0 0 0 " rpy="${-M_PI/2} -${M_PI} ${-M_PI/2}" />
         <geometry>
-          <mesh filename="package://carl_description/meshes/asus_xtion_pro_live.dae" scale="${M_SCALE*0.001} ${M_SCALE*0.001} ${M_SCALE*0.001}" />
+          <mesh filename="package://carl_description/meshes/asus_xtion_pro_live.min.dae" scale="${M_SCALE*0.001} ${M_SCALE*0.001} ${M_SCALE*0.001}" />
         </geometry>
       </visual>

File: carl_description/urdf/sensors/creative_camera.urdf.xacro (robot description, xacro)
@@ -17,5 +17,5 @@
         <origin xyz="0 0 0" rpy="0 0 0" />
         <geometry>
-          <mesh scale="${M_SCALE} ${M_SCALE} ${M_SCALE}" filename="package://carl_description/meshes/creative_camera.dae" />
+          <mesh scale="${M_SCALE} ${M_SCALE} ${M_SCALE}" filename="package://carl_description/meshes/creative_camera.min.dae" />
         </geometry>
       </visual>

Commit message: base, rear struts< >

File: carl_description/urdf/carl_base/carl_base.urdf.xacro (robot description, xacro)
@@ -26,7 +26,7 @@
       </visual>
      <collision>
-        <origin xyz="0 0 0" rpy="0 0 0" />
+        <origin xyz="0 0 -.0425" rpy="0 0 0" />
         <geometry>
-          <mesh scale="${M_SCALE} ${M_SCALE} ${M_SCALE}" filename="package://carl_description/meshes/base.stl" />
+          <box size="0.4 0.363 0.12"/>
         </geometry>
       </collision>

File: carl_description/urdf/components/carl_rear_strut.urdf.xacro (robot description, xacro)
@@ -22,7 +22,7 @@
       </visual>
       <collision>
-        <origin xyz="0 0 0" rpy="0 0 -${M_PI/2}" />
+        <origin xyz="0 0.001 0.505" rpy="0 0 0"/>
         <geometry>
-          <mesh scale="${M_SCALE} ${M_SCALE} ${M_SCALE}" filename="package://carl_description/meshes/rear_strut.stl" />
+          <box size="0.0255 0.052 1.1 "/>
         </geometry>
       </collision>
@@ -42,7 +42,7 @@
       </visual>
       <collision>
-        <origin xyz="0 0 0" rpy="0 0 -${M_PI/2}" />
+        <origin xyz="0 0 0.229" rpy="0 0 0" />
         <geometry>
-          <mesh scale="${M_SCALE} ${M_SCALE} ${M_SCALE}" filename="package://carl_description/meshes/rear_strut_top.stl" />
+          <box size="0.0255 0.051 0.4572"/>
         </geometry>
       </collision>

File: carl_description/urdf/components/carl_side_cover.urdf.xacro (robot description, xacro)
@@ -22,5 +22,5 @@
         <origin xyz="0 0 0" rpy="0 0 0" />
         <geometry>
-          <mesh scale="${M_SCALE} ${M_SCALE} ${M_SCALE}" filename="package://carl_description/meshes/side_cover.stl" />
+          <box size="0.0008 0.483 0.289"/>
         </geometry>
       </collision>
