Commit message: finished collision models. creative camera,mount,topplate,jacomount,camera lift

File: carl_description/urdf/carl_base/carl_frame.urdf.xacro (robot description, xacro)
@@ -30,7 +30,19 @@
       </visual>
       <collision>
-        <origin xyz="0 0 0" rpy="0 0 -${M_PI/2}" />
+        <origin xyz="-0.28 0.0 -.0031" rpy="0 0 -${M_PI/2}" />
         <geometry>
-          <mesh scale="${M_SCALE} ${M_SCALE} ${M_SCALE}" filename="package://carl_description/meshes/top_plate.stl" />
+          <box size="0.5842 0.5 0.0066"/>
+        </geometry>
+      </collision>
+      <collision>
+        <origin xyz="-.005 0.127 -.0031" rpy="0 0 -1.25" />
+        <geometry>
+          <box size="0.325 0.14 0.0066"/>
+        </geometry>
+      </collision>
+      <collision>
+        <origin xyz="-.005 -0.127 -.0031" rpy="0 0 1.25" />
+        <geometry>
+          <box size="0.325 0.14 0.0066"/>
         </geometry>
       </collision>
@@ -50,7 +62,8 @@
       </visual>
       <collision>
-        <origin xyz="0 0 0" rpy="0 0 0" />
+        <origin xyz="0 0 -0.0127" rpy="0 0 0" />
         <geometry>
-          <mesh scale="${M_SCALE} ${M_SCALE} ${M_SCALE}" filename="package://carl_description/meshes/jaco_mount.stl" />
+         <!-- <mesh scale="${M_SCALE} ${M_SCALE} ${M_SCALE}" filename="package://carl_description/meshes/jaco_mount.stl" /> -->
+         <box size="0.2286 0.0508 0.0254"/>
         </geometry>
       </collision>
@@ -70,7 +83,7 @@
       </visual>
       <collision>
-        <origin xyz="0 0 0" rpy="0 ${M_PI/2} ${M_PI/2}" />
+        <origin xyz="-0.0127 0 0" rpy="0 0 0" />
         <geometry>
-          <mesh scale="${M_SCALE} ${M_SCALE} ${M_SCALE}" filename="package://carl_description/meshes/camera_lift.stl" />
+          <box size="0.027 0.454 0.054" />
         </geometry>
       </collision>

File: carl_description/urdf/components/carl_asus_camera.urdf.xacro (robot description, xacro)
@@ -81,7 +81,7 @@
       </visual>
       <collision>
-        <origin xyz="0 0 0" rpy="0 ${M_PI/2} 0" />
+        <origin xyz="-0.0015875 0 0" rpy="0 ${M_PI/2} 0" />
         <geometry>
-          <mesh scale="${M_SCALE} ${M_SCALE} ${M_SCALE}" filename="package://carl_description/meshes/camera_mount.stl" />
+          <box size="0.041 0.2365 0.0032"/>
         </geometry>
       </collision>

File: carl_description/urdf/components/carl_creative_camera.urdf.xacro (robot description, xacro)
@@ -23,7 +23,7 @@
       </visual>
       <collision>
-        <origin xyz="0 0 0" rpy="0 0 0" />
+        <origin xyz="0.01488 0 0" rpy="0 0 0" />
         <geometry>
-          <mesh scale="${M_SCALE} ${M_SCALE} ${M_SCALE}" filename="package://carl_description/meshes/creative_mount.stl" />
+          <box size="0.0298 0.051 0.051"/>
         </geometry>
       </collision>
@@ -42,7 +42,7 @@
       </visual>
       <collision>
-        <origin xyz="0 0 0" rpy="0 0 0" />
+        <origin xyz="0.01344 -0.0184 0" rpy="0 0 0" />
         <geometry>
-          <mesh scale="${M_SCALE} ${M_SCALE} ${M_SCALE}" filename="package://carl_description/meshes/servo.stl" />
+          <box size="0.05 0.0382 0.032"/>
         </geometry>
       </collision>
@@ -62,7 +62,7 @@
       </visual>
       <collision>
-        <origin xyz="0 0 0" rpy="0 0 0" />
+        <origin xyz="0 -0.021 -0.02405" rpy="0 0 0" />
         <geometry>
-          <mesh scale="${M_SCALE} ${M_SCALE} ${M_SCALE}" filename="package://carl_description/meshes/servo_arm.stl" />
+          <box size="0.029 0.067 0.049"/>
         </geometry>
       </collision>
@@ -81,7 +81,7 @@
       </visual>
       <collision>
-        <origin xyz="0 0 0" rpy="0 0 0" />
+        <origin xyz="0 0 -0.0015875" rpy="0 0 0" />
         <geometry>
-          <mesh scale="${M_SCALE} ${M_SCALE} ${M_SCALE}" filename="package://carl_description/meshes/creative_plate.stl" />
+          <box size="0.13975 0.03815 0.00318"/>
         </geometry>
       </collision>

File: carl_description/urdf/sensors/creative_camera.urdf.xacro (robot description, xacro)
@@ -23,5 +23,5 @@
         <origin xyz="0 0 0" rpy="0 0 0" />
         <geometry>
-          <mesh scale="${M_SCALE} ${M_SCALE} ${M_SCALE}" filename="package://carl_description/meshes/creative_camera.stl" />
+          <box size="0.1070 0.02575 0.026"/>
         </geometry>
       </collision>
