Commit message: wheels, front cover, camera, hokuyo

File: carl_description/urdf/carl_base/carl_covers.urdf.xacro (robot description, xacro)
@@ -23,7 +23,19 @@
       </visual>
       <collision>
-        <origin xyz="0 0 0" rpy="0 0 0" />
+        <origin xyz="-0.2205 -0.034 0" rpy="0 0 -0.52" />
         <geometry>
-          <mesh scale="${M_SCALE} ${M_SCALE} ${M_SCALE}" filename="package://carl_description/meshes/front_cover.stl" />
+          <box size="0.25 0.068 0.508"/>
+        </geometry>
+      </collision>
+      <collision>
+        <origin xyz="0.2205 -0.034 0" rpy="0 0 0.52" />
+        <geometry>
+          <box size="0.25 0.068 0.508"/>
+        </geometry>
+      </collision>
+      <collision>
+        <origin xyz="0 -0.11 0" rpy="0 0 0" />
+        <geometry>
+          <box size="0.25 0.068 0.508"/>
         </geometry>
       </collision>
@@ -47,10 +59,4 @@
           <box size=".05 .45 1.56" />
         </geometry>
-        <!--
-        <origin xyz="0 0 0" rpy="0 0 0" />
-        <geometry>
-          <mesh scale="${M_SCALE} ${M_SCALE} ${M_SCALE}" filename="package://carl_description/meshes/back_cover.stl" />
-        </geometry>
-        -->
       </collision>
     </link>

File: carl_description/urdf/components/carl_wheel.urdf.xacro (robot description, xacro)
@@ -15,10 +15,7 @@
       </visual>
       <collision>
-        <origin xyz="0 0 0" rpy="0 0 0" />
+        <origin xyz="0 0 0.03" rpy="0 0 0" />
         <geometry>
-          <!--
-          <mesh scale="${M_SCALE} ${M_SCALE} ${M_SCALE}" filename="package://carl_description/meshes/wheel.stl" />
-          -->
-          <cylinder radius="0.25" length="0.11"/>
+          <cylinder radius="0.25" length="0.12"/>
         </geometry>
       </collision>

File: carl_description/urdf/sensors/asus_xtion_pro.urdf.xacro (robot description, xacro)
@@ -25,7 +25,7 @@
       </visual>
       <collision>
-        <origin xyz=" 0 0 0 " rpy="${-M_PI/2} -${M_PI} ${-M_PI/2}" />
+        <origin xyz="-0.0071 0.0031 0" rpy="${-M_PI/2} -${M_PI} ${-M_PI/2}" />
         <geometry>
-          <mesh filename="package://carl_description/meshes/asus_xtion_pro_live.stl" scale="${M_SCALE*0.001} ${M_SCALE*0.001} ${M_SCALE*0.001}" />
+          <box size="0.1799 0.0246 0.0362"/>
         </geometry>
       </collision>

File: carl_description/urdf/sensors/hokuyo.urdf.xacro (robot description, xacro)
@@ -20,5 +20,5 @@
         <origin xyz="0 0 0" rpy="0 0 0" />
         <geometry>
-          <mesh filename="package://carl_description/meshes/hokuyo.stl" />
+          <box size="0.05 0.05 0.08"/>
         </geometry>
       </collision>

Commit message: fixed castor plate. added screenshot

File: carl_description/urdf/carl_base/carl_covers.urdf.xacro (robot description, xacro)
@@ -55,5 +55,5 @@
       </visual>
       <collision>
-        <origin xyz=".025 0 .8" rpy="0 0 0" />
+        <origin xyz="-.0025 0 .78" rpy="0 0 0" />
         <geometry>
           <box size=".05 .45 1.56" />

File: carl_description/urdf/components/carl_caster_assembly.urdf.xacro (robot description, xacro)
@@ -21,7 +21,19 @@
       </visual>
       <collision>
-        <origin xyz="0.005 0 -0.04145" rpy="0 0 ${M_PI/2}" />
+        <origin xyz="-.01 -0.12 -0.04145" rpy="0 0 -2" />
         <geometry>
-          <box size="0.552 0.174 0.0949"/>
+          <box size="0.3 0.16 0.0949"/>
+        </geometry>
+      </collision>
+      <collision>
+        <origin xyz="-.01 0.12 -0.04145" rpy="0 0 2" />
+        <geometry>
+          <box size="0.3 0.16 0.0949"/>
+        </geometry>
+      </collision>
+            <collision>
+        <origin xyz="0.003 0 -0.04145" rpy="0 0 0" />
+        <geometry>
+          <box size="0.16 0.16 0.0949"/>
         </geometry>
       </collision>

File: carl_description/urdf/components/carl_side_cover.urdf.xacro (robot description, xacro)
@@ -20,7 +20,7 @@
       </visual>
       <collision>
-        <origin xyz="0 0 0" rpy="0 0 0" />
+        <origin xyz=".0005 0 0" rpy="0 0 0" />
         <geometry>
-          <box size="0.0008 0.483 0.289"/>
+          <box size="0.0015 0.483 0.289"/>
         </geometry>
       </collision>

Commit message: fixed front cover and back strut

File: carl_description/urdf/carl_base/carl_covers.urdf.xacro (robot description, xacro)
@@ -23,13 +23,13 @@
       </visual>
       <collision>
-        <origin xyz="-0.2205 -0.034 0" rpy="0 0 -0.52" />
+        <origin xyz="-0.20 -0.05 0" rpy="0 0 -0.52" />
         <geometry>
-          <box size="0.25 0.068 0.508"/>
+          <box size="0.21 0.068 0.508"/>
         </geometry>
       </collision>
       <collision>
-        <origin xyz="0.2205 -0.034 0" rpy="0 0 0.52" />
+        <origin xyz="0.20 -0.05 0" rpy="0 0 0.52" />
         <geometry>
-          <box size="0.25 0.068 0.508"/>
+          <box size="0.21 0.068 0.508"/>
         </geometry>
       </collision>

File: carl_description/urdf/components/carl_rear_strut.urdf.xacro (robot description, xacro)
@@ -22,7 +22,7 @@
       </visual>
       <collision>
-        <origin xyz="0 0.001 0.505" rpy="0 0 0"/>
+        <origin xyz="0.005 0.001 0.525" rpy="0 0 0"/>
         <geometry>
-          <box size="0.0255 0.052 1.1 "/>
+          <box size="0.0355 0.052 1.07 "/>
         </geometry>
       </collision>
@@ -42,7 +42,7 @@
       </visual>
       <collision>
-        <origin xyz="0 0 0.229" rpy="0 0 0" />
+        <origin xyz="0.005 0 0.229" rpy="0 0 0" />
         <geometry>
-          <box size="0.0255 0.051 0.4572"/>
+          <box size="0.0355 0.051 0.4572"/>
         </geometry>
       </collision>
