Commit message: re-wrote URDF to fix collision problems

File: carl_description/robots/carl.urdf.xacro (robot description, xacro)
@@ -2,6 +2,4 @@
 <robot xmlns:xacro="http://www.ros.org/wiki/xacro" name="carl">
   <xacro:include filename="$(find carl_description)/urdf/carl_base/carl_base.urdf.xacro" />
-  <xacro:include filename="$(find jaco_description)/urdf/jaco_arm.xacro" />
   <xacro:carl_base name="base" />
-  <xacro:jaco_arm  parent="jaco_mount_link" />
 </robot>

File: carl_description/urdf/carl_base/carl_base.urdf.xacro (robot description, xacro)
@@ -4,24 +4,23 @@
        xmlns:interface="http://playerstage.sourceforge.net/gazebo/xmlschema/#interface"
        xmlns:xacro="http://ros.org/wiki/xacro">
+  <!-- Xacro properties -->
+  <xacro:property name="M_SCALE" value="0.0254" />
+  <xacro:property name="M_PI" value="3.1415926535897931" />
   <xacro:include filename="$(find carl_description)/urdf/components/carl_wheel.urdf.xacro" />
   <xacro:include filename="$(find carl_description)/urdf/components/carl_caster_assembly.urdf.xacro" />
+  <xacro:include filename="$(find carl_description)/urdf/components/carl_asus_camera.urdf.xacro" />
+  <xacro:include filename="$(find carl_description)/urdf/components/carl_creative_camera.urdf.xacro" />
   <xacro:include filename="$(find carl_description)/urdf/sensors/hokuyo.urdf.xacro" />
-  <xacro:include filename="$(find carl_description)/urdf/carl_base/carl_superstructure.urdf.xacro" />
+  <xacro:include filename="$(find carl_description)/urdf/carl_base/carl_frame.urdf.xacro" />
   <xacro:include filename="$(find carl_description)/urdf/carl_base/carl_covers.urdf.xacro" />
-  <xacro:include filename="$(find carl_description)/urdf/carl_base/carl_asus_camera_mount.urdf.xacro" />
-  <xacro:include filename="$(find carl_description)/urdf/carl_base/carl_creative_camera_mount.urdf.xacro" />
   <xacro:macro name="carl_base" params="name">
-    <xacro:carl_superstructure />
-    <xacro:carl_asus_camera_mount />
-    <xacro:carl_creative_camera_mount />
-    <xacro:carl_covers name="${name}" />
-    <!-- base footprint -->
+    <!-- base_footprint -->
     <link name="${name}_footprint" />
-  	<!-- base link -->
+  	<!-- base_link -->
     <link name="${name}_link">
      <visual>
         <origin xyz="0 0 0" rpy="0 0 0" />
         <geometry>
-          <mesh filename="package://carl_description/meshes/base.min.dae" />
+          <mesh scale="${M_SCALE} ${M_SCALE} ${M_SCALE}" filename="package://carl_description/meshes/base.dae" />
         </geometry>
       </visual>
@@ -29,8 +28,9 @@
         <origin xyz="0 0 0" rpy="0 0 0" />
         <geometry>
-          <mesh filename="package://carl_description/meshes/base.min.dae" />
+          <mesh scale="${M_SCALE} ${M_SCALE} ${M_SCALE}" filename="package://carl_description/meshes/base.stl" />
         </geometry>
       </collision>
     </link>
+    <!-- base_link to base_footprint -->
     <joint name="${name}_footprint_${name}_link_joint" type="fixed">
       <parent link="${name}_footprint" />
@@ -38,20 +38,28 @@
       <origin xyz="0 0 0.23114" rpy="0 0 0" />
     </joint>
-    <!-- left wheel -->
+    <!-- Wheels -->
     <xacro:carl_wheel suffix="left" parent="${name}_link">
-      <origin xyz="0 0.25 0" rpy="-1.5708 0 0" />
+      <origin xyz="0 0.25 0" rpy="${M_PI/2} 0 0" />
     </xacro:carl_wheel>
-    <!-- right wheel -->
     <xacro:carl_wheel suffix="right" parent="${name}_link">
-      <origin xyz="0 -0.25 0" rpy="1.5708 0 0" />
+      <origin xyz="0 -0.25 0" rpy="-${M_PI/2} 0 0" />
     </xacro:carl_wheel>
-    <!-- caster assembly -->
+    <!-- Caster Assembly -->
     <xacro:carl_caster_assembly parent="${name}_link">
       <origin xyz="0.2883 0 0" rpy="0 0 0" />
     </xacro:carl_caster_assembly>
-    <!-- hokuyo -->
+    <!-- Frame and Covers -->
+    <xacro:carl_frame parent="${name}_link" />
+    <xacro:carl_covers parent="${name}_link" />
+    <!-- Sensors -->
     <xacro:hokuyo parent="caster_plate_link">
       <origin xyz="0.07 0 0.035" rpy="0 0 0" />
     </xacro:hokuyo>
+    <xacro:carl_asus_camera parent="asus_lift_link">
+      <origin xyz="0 0 0" rpy="${M_PI/2} 0 0" />
+    </xacro:carl_asus_camera>
+    <xacro:carl_creative_camera parent="top_plate_link">
+      <origin xyz="0.07 0 -0.03" rpy="0 0 ${M_PI}" />
+    </xacro:carl_creative_camera>
   </xacro:macro>
 </robot>

File: carl_description/urdf/carl_base/carl_covers.urdf.xacro (robot description, xacro)
@@ -4,44 +4,20 @@
        xmlns:interface="http://playerstage.sourceforge.net/gazebo/xmlschema/#interface"
        xmlns:xacro="http://ros.org/wiki/xacro">
+  <!-- Xacro properties -->
+  <xacro:property name="M_SCALE" value="0.0254" />
+  <xacro:property name="M_PI" value="3.1415926535897931" />
   <xacro:include filename="$(find carl_description)/urdf/components/carl_side_cover.urdf.xacro" />
-  <xacro:macro name="carl_covers" params="name">
-    <!-- right side cover -->
-    <xacro:carl_side_cover suffix="right" parent="right_rear_strut_link">
-      <origin xyz="-0.229 -0.026 0.447" rpy="0 0 0" />
-    </xacro:carl_side_cover>
-    <!-- left side cover -->
-    <xacro:carl_side_cover suffix="left" parent="left_rear_strut_link">
-      <origin xyz="0.229 0.026 0.447" rpy="0 0 0" />
-    </xacro:carl_side_cover>
-    <joint name="${name}_front_cover_joint" type="fixed">
-      <parent link="${name}_link" />
-      <child link="FrontCover_link" />
-      <origin xyz=".247 0 0.242" rpy="0 0 0" />
+  <xacro:macro name="carl_covers" params="parent">
+    <!-- Front Cover -->
+    <joint name="${name}_front_cover_link_joint" type="fixed">
+      <parent link="${parent}" />
+      <child link="front_cover_link" />
+      <origin xyz="0.247 0 0.242" rpy="0 0 ${M_PI/2}" />
     </joint>
-    <joint name="${name}_back_cover" type="fixed">
-      <parent link="${name}_link" />
-      <child link="BackCover_link" />
-      <origin xyz="-.237 0 -0.102" rpy="0 0 0" />
-    </joint>
-    <link name="FrontCover_link">
-      <visual>
-        <origin xyz="0 0 0" rpy="0 0 1.5708" />
-        <geometry>
-          <mesh filename="package://carl_description/meshes/front_cover.min.dae" />
-        </geometry>
-      </visual>
-      <collision>
-        <origin xyz="0 0 0" rpy="0 0 1.5708" />
-        <geometry>
-          <mesh filename="package://carl_description/meshes/front_cover.min.dae" />
-        </geometry>
-      </collision>
-    </link>
-    <link name="BackCover_link">
+    <link name="front_cover_link">
       <visual>
         <origin xyz="0 0 0" rpy="0 0 0" />
         <geometry>
-          <!--<box size="0.005 0.45 0.6" />-->
-          <mesh filename="package://carl_description/meshes/back_cover.min.dae" />
+          <mesh scale="${M_SCALE} ${M_SCALE} ${M_SCALE}" filename="package://carl_description/meshes/front_cover.dae" />
         </geometry>
       </visual>
@@ -49,9 +25,35 @@
         <origin xyz="0 0 0" rpy="0 0 0" />
         <geometry>
-          <!--<box size="0.005 0.45 0.6" />-->
-          <mesh filename="package://carl_description/meshes/back_cover.min.dae" />
+          <mesh scale="${M_SCALE} ${M_SCALE} ${M_SCALE}" filename="package://carl_description/meshes/front_cover.stl" />
         </geometry>
       </collision>
     </link>
+    <!-- Back Cover -->
+    <joint name="${name}_back_cover_link_joint" type="fixed">
+      <parent link="${parent}" />
+      <child link="back_cover_link" />
+      <origin xyz="-0.237 0 -0.102" rpy="0 0 0" />
+    </joint>
+    <link name="back_cover_link">
+      <visual>
+        <origin xyz="0 0 0" rpy="0 0 0" />
+        <geometry>
+          <mesh scale="${M_SCALE} ${M_SCALE} ${M_SCALE}" filename="package://carl_description/meshes/back_cover.dae" />
+        </geometry>
+      </visual>
+      <collision>
+        <origin xyz="0 0 0" rpy="0 0 0" />
+        <geometry>
+          <mesh scale="${M_SCALE} ${M_SCALE} ${M_SCALE}" filename="package://carl_description/meshes/back_cover.stl" />
+        </geometry>
+      </collision>
+    </link>
+    <!-- Side Covers -->
+    <xacro:carl_side_cover prefix="right" parent="${parent}">
+      <origin xyz="0.007 -0.226 0.345" rpy="0 0 ${M_PI/2}" />
+    </xacro:carl_side_cover>
+    <xacro:carl_side_cover prefix="left" parent="${parent}">
+      <origin xyz="0.007 0.226 0.345" rpy="0 0 ${M_PI/2}" />
+    </xacro:carl_side_cover>
   </xacro:macro>
 </robot>

File: carl_description/urdf/components/carl_caster_assembly.urdf.xacro (robot description, xacro)
@@ -1,11 +1,31 @@
 <?xml version="1.0"?>
-<root xmlns:xacro="http://ros.org/wiki/xacro">
+<robot xmlns:sensor="http://playerstage.sourceforge.net/gazebo/xmlschema/#sensor"
+       xmlns:controller="http://playerstage.sourceforge.net/gazebo/xmlschema/#controller"
+       xmlns:interface="http://playerstage.sourceforge.net/gazebo/xmlschema/#interface"
+       xmlns:xacro="http://ros.org/wiki/xacro">
+  <!-- Xacro properties -->
+  <xacro:property name="M_SCALE" value="0.0254" />
+  <xacro:property name="M_PI" value="3.1415926535897931" />
   <xacro:macro name="carl_caster_assembly" params="parent *origin">
-    <joint name="${parent}_caster_plate_joint" type="fixed">
+    <joint name="${parent}_caster_plate_link_joint" type="fixed">
       <xacro:insert_block name="origin" />
       <parent link="${parent}" />
       <child link="caster_plate_link" />
     </joint>
-    <joint name="caster_plate__caster_joint" type="continuous">
+    <link name="caster_plate_link">
+      <visual>
+        <origin xyz="0 0 0" rpy="0 0 ${M_PI/2}" />
+        <geometry>
+          <mesh scale="${M_SCALE} ${M_SCALE} ${M_SCALE}" filename="package://carl_description/meshes/caster_plate.dae" />
+        </geometry>
+      </visual>
+      <collision>
+        <origin xyz="0 0 0" rpy="0 0 ${M_PI/2}" />
+        <geometry>
+          <mesh scale="${M_SCALE} ${M_SCALE} ${M_SCALE}" filename="package://carl_description/meshes/caster_plate.stl" />
+        </geometry>
+      </collision>
+    </link>
+    <joint name="caster_plate_link_caster_link_joint" type="continuous">
       <parent link="caster_plate_link" />
       <child link="caster_link" />
@@ -13,23 +33,9 @@
       <axis xyz="0 0 1" />
     </joint>
-    <link name="caster_plate_link">
-      <visual>
-        <origin xyz="0 0 0" rpy="0 0 1.5708" />
-        <geometry>
-          <mesh filename="package://carl_description/meshes/caster_plate.min.dae" />
-        </geometry>
-      </visual>
-      <collision>
-        <origin xyz="0 0 0" rpy="0 0 1.5708" />
-        <geometry>
-          <mesh filename="package://carl_description/meshes/caster_plate.min.dae" />
-        </geometry>
-      </collision>
-    </link>
     <link name="caster_link">
       <visual>
         <origin xyz="0 0 0" rpy="0 0 0" />
         <geometry>
-          <mesh filename="package://carl_description/meshes/caster.min.dae" />
+          <mesh scale="${M_SCALE} ${M_SCALE} ${M_SCALE}" filename="package://carl_description/meshes/caster.dae" />
         </geometry>
       </visual>
@@ -37,8 +43,8 @@
         <origin xyz="0 0 0" rpy="0 0 0" />
         <geometry>
-          <mesh filename="package://carl_description/meshes/caster.min.dae" />
+          <mesh scale="${M_SCALE} ${M_SCALE} ${M_SCALE}" filename="package://carl_description/meshes/caster.stl" />
         </geometry>
       </collision>
     </link>
   </xacro:macro>
-</root>
+</robot>

File: carl_description/urdf/components/carl_rear_strut.urdf.xacro (robot description, xacro)
@@ -1,43 +1,51 @@
 <?xml version="1.0"?>
-<root xmlns:xacro="http://ros.org/wiki/xacro">
-  <xacro:macro name="carl_rear_strut" params="suffix parent *origin">
-    <joint name="${parent}_${suffix}_rear_strut_joint" type="fixed">
+<robot xmlns:sensor="http://playerstage.sourceforge.net/gazebo/xmlschema/#sensor"
+       xmlns:controller="http://playerstage.sourceforge.net/gazebo/xmlschema/#controller"
+       xmlns:interface="http://playerstage.sourceforge.net/gazebo/xmlschema/#interface"
+       xmlns:xacro="http://ros.org/wiki/xacro">
+  <!-- Xacro properties -->
+  <xacro:property name="M_SCALE" value="0.0254" />
+  <xacro:property name="M_PI" value="3.1415926535897931" />
+  <xacro:macro name="carl_rear_strut" params="prefix parent *origin">
+    <!-- Bottom -->
+    <joint name="${parent}_${prefix}_rear_strut_joint" type="fixed">
       <xacro:insert_block name="origin" />
       <parent link="${parent}" />
-      <child link="${suffix}_rear_strut_link" />
+      <child link="${prefix}_rear_strut_link" />
     </joint>
-    <joint name="${suffix}_rear_strut_link_${suffix}_rear_strut_top_link_joint" type="fixed">
-      <parent link="${suffix}_rear_strut_link" />
-        <child link="${suffix}_rear_strut_top_link" />
-      <origin xyz="0 0.001 1.055" rpy="0 0 0" />
-    </joint>
-    <link name="${suffix}_rear_strut_link">
+    <link name="${prefix}_rear_strut_link">
       <visual>
-        <origin xyz="0 0 0" rpy="0 0 -1.5708" />
+        <origin xyz="0 0 0" rpy="0 0 -${M_PI/2}" />
         <geometry>
-          <mesh filename="package://carl_description/meshes/rear_strut.min.dae" />
+          <mesh scale="${M_SCALE} ${M_SCALE} ${M_SCALE}" filename="package://carl_description/meshes/rear_strut.dae" />
         </geometry>
       </visual>
       <collision>
-        <origin xyz="0 0 0" rpy="0 0 -1.5708" />
+        <origin xyz="0 0 0" rpy="0 0 -${M_PI/2}" />
         <geometry>
-          <mesh filename="package://carl_description/meshes/rear_strut.min.dae" />
+          <mesh scale="${M_SCALE} ${M_SCALE} ${M_SCALE}" filename="package://carl_description/meshes/rear_strut.stl" />
         </geometry>
       </collision>
     </link>
-    <link name="${suffix}_rear_strut_top_link">
+    <!-- Top -->
+    <joint name="${prefix}_rear_strut_link_${prefix}_rear_strut_top_link_joint" type="fixed">
+      <parent link="${prefix}_rear_strut_link" />
+      <child link="${prefix}_rear_strut_top_link" />
+      <origin xyz="0 0.001 1.055" rpy="0 0 0" />
+    </joint>
+    <link name="${prefix}_rear_strut_top_link">
       <visual>
-        <origin xyz="0 0 0" rpy="0 0 -1.5708" />
+        <origin xyz="0 0 0" rpy="0 0 -${M_PI/2}" />
         <geometry>
-          <mesh filename="package://carl_description/meshes/rear_strut_top.min.dae" />
+          <mesh scale="${M_SCALE} ${M_SCALE} ${M_SCALE}" filename="package://carl_description/meshes/rear_strut_top.dae" />
         </geometry>
       </visual>
       <collision>
-        <origin xyz="0 0 0" rpy="0 0 -1.5708" />
+        <origin xyz="0 0 0" rpy="0 0 -${M_PI/2}" />
         <geometry>
-          <mesh filename="package://carl_description/meshes/rear_strut_top.min.dae" />
+          <mesh scale="${M_SCALE} ${M_SCALE} ${M_SCALE}" filename="package://carl_description/meshes/rear_strut_top.stl" />
         </geometry>
       </collision>
     </link>
   </xacro:macro>
-</root>
+</robot>

File: carl_description/urdf/components/carl_side_cover.urdf.xacro (robot description, xacro)
@@ -1,24 +1,29 @@
 <?xml version="1.0"?>
-<root xmlns:xacro="http://ros.org/wiki/xacro">
-  <xacro:macro name="carl_side_cover" params="suffix parent *origin">
-    <joint name="${parent}_${suffix}_side_cover_joint" type="fixed">
+<robot xmlns:sensor="http://playerstage.sourceforge.net/gazebo/xmlschema/#sensor"
+       xmlns:controller="http://playerstage.sourceforge.net/gazebo/xmlschema/#controller"
+       xmlns:interface="http://playerstage.sourceforge.net/gazebo/xmlschema/#interface"
+       xmlns:xacro="http://ros.org/wiki/xacro">
+  <!-- Xacro properties -->
+  <xacro:property name="M_SCALE" value="0.0254" />
+  <xacro:macro name="carl_side_cover" params="prefix parent *origin">
+    <joint name="${parent}_${prefix}_side_cover_link_joint" type="fixed">
       <xacro:insert_block name="origin" />
       <parent link="${parent}" />
-      <child link="${suffix}_side_cover_link" />
+      <child link="${prefix}_side_cover_link" />
     </joint>
-    <link name="${suffix}_side_cover_link">
+    <link name="${prefix}_side_cover_link">
       <visual>
-        <origin xyz="0 0 0" rpy="0 0 1.5708" />
+        <origin xyz="0 0 0" rpy="0 0 0" />
         <geometry>
-          <mesh filename="package://carl_description/meshes/side_cover.min.dae" />
+          <mesh scale="${M_SCALE} ${M_SCALE} ${M_SCALE}" filename="package://carl_description/meshes/side_cover.dae" />
         </geometry>
       </visual>
       <collision>
-        <origin xyz="0 0 0" rpy="0 0 1.5708" />
+        <origin xyz="0 0 0" rpy="0 0 0" />
         <geometry>
-          <mesh filename="package://carl_description/meshes/side_cover.min.dae" />
+          <mesh scale="${M_SCALE} ${M_SCALE} ${M_SCALE}" filename="package://carl_description/meshes/side_cover.stl" />
         </geometry>
       </collision>
     </link>
   </xacro:macro>
-</root>
+</robot>

File: carl_description/urdf/components/carl_wheel.urdf.xacro (robot description, xacro)
@@ -1,5 +1,24 @@
 <?xml version="1.0"?>
-<root xmlns:xacro="http://ros.org/wiki/xacro">
+<robot xmlns:sensor="http://playerstage.sourceforge.net/gazebo/xmlschema/#sensor"
+       xmlns:controller="http://playerstage.sourceforge.net/gazebo/xmlschema/#controller"
+       xmlns:interface="http://playerstage.sourceforge.net/gazebo/xmlschema/#interface"
+       xmlns:xacro="http://ros.org/wiki/xacro">
+  <!-- Xacro properties -->
+  <xacro:property name="M_SCALE" value="0.0254" />
   <xacro:macro name="carl_wheel" params="suffix parent *origin">
+    <link name="${suffix}_wheel_link">
+      <visual>
+        <origin xyz="0 0 0" rpy="0 0 0" />
+        <geometry>
+          <mesh scale="${M_SCALE} ${M_SCALE} ${M_SCALE}" filename="package://carl_description/meshes/wheel.dae" />
+        </geometry>
+      </visual>
+      <collision>
+        <origin xyz="0 0 0" rpy="0 0 0" />
+        <geometry>
+          <mesh scale="${M_SCALE} ${M_SCALE} ${M_SCALE}" filename="package://carl_description/meshes/wheel.stl" />
+        </geometry>
+      </collision>
+    </link>
     <joint name="${parent}_${suffix}_wheel_joint" type="continuous">
       <xacro:insert_block name="origin" />
@@ -8,18 +27,4 @@
       <child link="${suffix}_wheel_link" />
     </joint>
-    <link name="${suffix}_wheel_link">
-      <visual>
-        <origin xyz="0 0 0" rpy="0 0 0" />
-        <geometry>
-          <mesh filename="package://carl_description/meshes/wheel.min.dae" />
-        </geometry>
-      </visual>
-      <collision>
-        <origin xyz="0 0 0" rpy="0 0 0" />
-        <geometry>
-          <mesh filename="package://carl_description/meshes/wheel.min.dae" />
-        </geometry>
-      </collision>
-    </link>
   </xacro:macro>
-</root>
+</robot>
