Commit message: re-wrote URDF to fix collision problems

File: carl_description/urdf/sensors/asus_xtion_pro.urdf.xacro (robot description, xacro)
@@ -2,5 +2,5 @@
 <robot name="sensor_asus_xtion_pro" xmlns:xacro="http://ros.org/wiki/xacro">
   <!-- Xacro properties -->
-  <xacro:property name="M_SCALE" value="0.001" />
+  <xacro:property name="M_SCALE" value="0.0254" />
   <xacro:property name="asus_xtion_pro_depth_rel_rgb_py" value="0.0270" />
   <xacro:property name="asus_xtion_pro_cam_rel_rgb_py"   value="-0.0220" />
@@ -12,71 +12,71 @@
       <child link="camera_link" />
     </joint>
-  <link name="camera_link">
-    <inertial>
-      <mass value="0.01" />
-      <origin xyz="0 0 0" />
-      <inertia ixx="0.001" ixy="0.0" ixz="0.0" iyy="0.001" iyz="0.0" izz="0.001" />
-    </inertial>
-    <visual>
-      <origin xyz=" 0 0 0 " rpy="${-M_PI/2} -${M_PI} ${-M_PI/2}" />
-      <geometry>
-        <mesh filename="package://carl_description/meshes/asus_xtion_pro_live.min.dae" scale="${M_SCALE} ${M_SCALE} ${M_SCALE}" />
-      </geometry>
-    </visual>
-    <collision>
-      <origin xyz=" 0 0 0 " rpy="${-M_PI/2} -${M_PI} ${-M_PI/2}" />
-      <geometry>
-        <mesh filename="package://carl_description/meshes/asus_xtion_pro_live.min.dae" scale="${M_SCALE} ${M_SCALE} ${M_SCALE}" />
-      </geometry>
-    </collision>
-  </link>
-  <joint name="camera_depth_joint" type="fixed">
-    <origin xyz="0 0.049 0" rpy="0 0 0" />
-    <parent link="camera_link" />
-    <child link="camera_depth_frame" />
-  </joint>
-  <link name="camera_depth_frame">
-    <inertial>
-      <mass value="0.01" />
-      <origin xyz="0 0 0" />
-      <inertia ixx="0.001" ixy="0.0" ixz="0.0" iyy="0.001" iyz="0.0" izz="0.001" />
-    </inertial>
-  </link>
-  <joint name="camera_depth_optical_joint" type="fixed">
-    <origin xyz="0 0 0" rpy="${-M_PI/2} 0 ${-M_PI/2}" />
-    <parent link="camera_depth_frame" />
-    <child link="camera_depth_optical_frame" />
-  </joint>
-  <link name="camera_depth_optical_frame">
-    <inertial>
-      <mass value="0.001" />
-      <origin xyz="0 0 0" />
-      <inertia ixx="0.0001" ixy="0.0" ixz="0.0" iyy="0.0001" iyz="0.0" izz="0.0001" />
-    </inertial>
-  </link>
-  <joint name="camera_rgb_joint" type="fixed">
-    <origin xyz="0 0.022 0" rpy="0 0 0" />
-    <parent link="camera_link" />
-    <child link="camera_rgb_frame" />
-  </joint>
-  <link name="camera_rgb_frame">
-    <inertial>
-      <mass value="0.001" />
-      <origin xyz="0 0 0" />
-      <inertia ixx="0.0001" ixy="0.0" ixz="0.0" iyy="0.0001" iyz="0.0" izz="0.0001" />
-    </inertial>
-  </link>
-  <joint name="camera_rgb_optical_joint" type="fixed">
-    <origin xyz="0 0 0" rpy="${-M_PI/2} 0 ${-M_PI/2}" />
-    <parent link="camera_rgb_frame" />
-    <child link="camera_rgb_optical_frame" />
-  </joint>
-  <link name="camera_rgb_optical_frame">
-    <inertial>
-      <mass value="0.001" />
-      <origin xyz="0 0 0" />
-      <inertia ixx="0.0001" ixy="0.0" ixz="0.0" iyy="0.0001" iyz="0.0" izz="0.0001" />
-    </inertial>
-  </link>
+    <link name="camera_link">
+      <inertial>
+        <mass value="0.01" />
+        <origin xyz="0 0 0" />
+        <inertia ixx="0.001" ixy="0.0" ixz="0.0" iyy="0.001" iyz="0.0" izz="0.001" />
+      </inertial>
+      <visual>
+        <origin xyz=" 0 0 0 " rpy="${-M_PI/2} -${M_PI} ${-M_PI/2}" />
+        <geometry>
+          <mesh filename="package://carl_description/meshes/asus_xtion_pro_live.dae" scale="${M_SCALE*0.001} ${M_SCALE*0.001} ${M_SCALE*0.001}" />
+        </geometry>
+      </visual>
+      <collision>
+        <origin xyz=" 0 0 0 " rpy="${-M_PI/2} -${M_PI} ${-M_PI/2}" />
+        <geometry>
+          <mesh filename="package://carl_description/meshes/asus_xtion_pro_live.stl" scale="${M_SCALE*0.001} ${M_SCALE*0.001} ${M_SCALE*0.001}" />
+        </geometry>
+      </collision>
+    </link>
+    <joint name="camera_depth_joint" type="fixed">
+      <origin xyz="0 0.049 0" rpy="0 0 0" />
+      <parent link="camera_link" />
+      <child link="camera_depth_frame" />
+    </joint>
+    <link name="camera_depth_frame">
+      <inertial>
+        <mass value="0.01" />
+        <origin xyz="0 0 0" />
+        <inertia ixx="0.001" ixy="0.0" ixz="0.0" iyy="0.001" iyz="0.0" izz="0.001" />
+      </inertial>
+    </link>
+    <joint name="camera_depth_optical_joint" type="fixed">
+      <origin xyz="0 0 0" rpy="${-M_PI/2} 0 ${-M_PI/2}" />
+      <parent link="camera_depth_frame" />
+      <child link="camera_depth_optical_frame" />
+    </joint>
+    <link name="camera_depth_optical_frame">
+      <inertial>
+        <mass value="0.001" />
+        <origin xyz="0 0 0" />
+        <inertia ixx="0.0001" ixy="0.0" ixz="0.0" iyy="0.0001" iyz="0.0" izz="0.0001" />
+      </inertial>
+    </link>
+    <joint name="camera_rgb_joint" type="fixed">
+      <origin xyz="0 0.022 0" rpy="0 0 0" />
+      <parent link="camera_link" />
+      <child link="camera_rgb_frame" />
+    </joint>
+    <link name="camera_rgb_frame">
+      <inertial>
+        <mass value="0.001" />
+        <origin xyz="0 0 0" />
+        <inertia ixx="0.0001" ixy="0.0" ixz="0.0" iyy="0.0001" iyz="0.0" izz="0.0001" />
+      </inertial>
+    </link>
+    <joint name="camera_rgb_optical_joint" type="fixed">
+      <origin xyz="0 0 0" rpy="${-M_PI/2} 0 ${-M_PI/2}" />
+      <parent link="camera_rgb_frame" />
+      <child link="camera_rgb_optical_frame" />
+    </joint>
+    <link name="camera_rgb_optical_frame">
+      <inertial>
+        <mass value="0.001" />
+        <origin xyz="0 0 0" />
+        <inertia ixx="0.0001" ixy="0.0" ixz="0.0" iyy="0.0001" iyz="0.0" izz="0.0001" />
+      </inertial>
+    </link>
   </xacro:macro>
 </robot>

File: carl_description/urdf/sensors/creative_camera.urdf.xacro (robot description, xacro)
@@ -1,6 +1,12 @@
 <?xml version="1.0"?>
-<root xmlns:xacro="http://ros.org/wiki/xacro">
+<robot xmlns:sensor="http://playerstage.sourceforge.net/gazebo/xmlschema/#sensor"
+       xmlns:controller="http://playerstage.sourceforge.net/gazebo/xmlschema/#controller"
+       xmlns:interface="http://playerstage.sourceforge.net/gazebo/xmlschema/#interface"
+       xmlns:xacro="http://ros.org/wiki/xacro">
+  <!-- Xacro properties -->
+  <xacro:property name="M_SCALE" value="0.0254" />
+  <xacro:property name="M_PI" value="3.1415926535897931" />
   <xacro:macro name="sensor_creative_camera" params="parent *origin">
-    <joint name="${parent}_creative_camera_joint" type="fixed">
+    <joint name="${parent}_creative_camera_link_joint" type="fixed">
       <xacro:insert_block name="origin" />
       <parent link="${parent}" />
@@ -11,5 +17,5 @@
         <origin xyz="0 0 0" rpy="0 0 0" />
         <geometry>
-          <mesh filename="package://carl_description/meshes/creative_camera.min.dae" />
+          <mesh scale="${M_SCALE} ${M_SCALE} ${M_SCALE}" filename="package://carl_description/meshes/creative_camera.dae" />
         </geometry>
       </visual>
@@ -17,8 +23,8 @@
         <origin xyz="0 0 0" rpy="0 0 0" />
         <geometry>
-          <mesh filename="package://carl_description/meshes/creative_camera.min.dae" />
+          <mesh scale="${M_SCALE} ${M_SCALE} ${M_SCALE}" filename="package://carl_description/meshes/creative_camera.stl" />
         </geometry>
       </collision>
     </link>
   </xacro:macro>
-</root>
+</robot>

File: carl_description/urdf/sensors/hokuyo.urdf.xacro (robot description, xacro)
@@ -1,6 +1,9 @@
 <?xml version="1.0"?>
-<root xmlns:xacro="http://ros.org/wiki/xacro">
+<robot xmlns:sensor="http://playerstage.sourceforge.net/gazebo/xmlschema/#sensor"
+       xmlns:controller="http://playerstage.sourceforge.net/gazebo/xmlschema/#controller"
+       xmlns:interface="http://playerstage.sourceforge.net/gazebo/xmlschema/#interface"
+       xmlns:xacro="http://ros.org/wiki/xacro">
   <xacro:macro name="hokuyo" params="parent *origin">
-    <joint name="${parent}_hokuyo_joint" type="fixed">
+    <joint name="${parent}_hokuyo_link_joint" type="fixed">
       <xacro:insert_block name="origin" />
       <parent link="${parent}" />
@@ -17,8 +20,8 @@
         <origin xyz="0 0 0" rpy="0 0 0" />
         <geometry>
-          <mesh filename="package://carl_description/meshes/hokuyo.min.dae" />
+          <mesh filename="package://carl_description/meshes/hokuyo.stl" />
         </geometry>
       </collision>
     </link>
   </xacro:macro>
-</root>
+</robot>
