Commit message: Refactoring.

File: carl_description/robots/carl.urdf (robot description, URDF)
Before this commit: robot carl, 29 links, 28 joints
Links:
- removed link CasterPlate_link
- removed link Caster_link
- removed link LeftWheel_link
- removed link RearLeftStrutInside_link
- removed link RearLeftStrut_link
- removed link RearRightStrutInside_link
- removed link RearRightStrut_link
- removed link RightWheel_link
- added link caster_link; collision cylinder length=0.213 radius=0.116; visual mesh filename=package://carl_description/meshes/caster.dae
- added link caster_plate_link; visual mesh filename=package://carl_description/meshes/caster_plate.dae
- added link left_rear_strut_inside_link; visual box size=0.02 0.045 1
- added link left_rear_strut_link; collision box size=0.027 0.054 1.055; visual mesh filename=package://carl_description/meshes/rear_strut.dae
- added link left_wheel_link; collision cylinder length=0.1 radius=0.25; visual mesh filename=package://carl_description/meshes/wheel.dae
- added link right_rear_strut_inside_link; visual box size=0.02 0.045 1
- added link right_rear_strut_link; collision box size=0.027 0.054 1.055; visual mesh filename=package://carl_description/meshes/rear_strut.dae
- added link right_wheel_link; collision cylinder length=0.1 radius=0.25; visual mesh filename=package://carl_description/meshes/wheel.dae
Joints:
- removed joint BaseToBackCover
- removed joint BaseToCasterPlate
- removed joint BaseToFrontCover
- removed joint BaseToLeftWheel
- removed joint BaseToRearLeftStrut
- removed joint BaseToRearRightStrut
- removed joint BaseToRightWheel
- removed joint CasterPlateToCaster
- removed joint CasterToHokuyo
- removed joint RearLeftStrutToLeftSideCover
- removed joint RearLeftStrutToRearLeftStutInside
- removed joint RearRightStrutToRearRightStutInside
- removed joint RearRightStrutToRightSideCover
- added joint base_back_cover: type fixed, parent base_link, child BackCover_link, origin xyz=-.237 0 -0.102 rpy=0 0 0
- added joint base_front_cover_joint: type fixed, parent base_link, child FrontCover_link, origin xyz=.247 0 0.242 rpy=0 0 0
- added joint base_link_caster_plate_joint: type fixed, parent base_link, child caster_plate_link, origin xyz=0.2883 0 0 rpy=0 0 0
- added joint base_link_left_rear_strut_joint: type fixed, parent base_link, child left_rear_strut_link, origin xyz=-0.222 0.200 -0.102 rpy=0 0 0
- added joint base_link_left_wheel_joint: type continuous, parent base_link, child left_wheel_link, origin xyz=0 0.25 0 rpy=-1.5708 0 0, axis 0 0 1
- added joint base_link_right_rear_strut_joint: type fixed, parent base_link, child right_rear_strut_link, origin xyz=-0.222 -0.200 -0.102 rpy=0 0 0
- added joint base_link_right_wheel_joint: type continuous, parent base_link, child right_wheel_link, origin xyz=0 -0.25 0 rpy=1.5708 0 0, axis 0 0 1
- added joint caster_hokuyo_joint: type fixed, parent caster_plate_link, child Hokuyo_link, origin xyz=0.07 0 0.035 rpy=0 0 0
- added joint caster_plate__caster_joint: type continuous, parent caster_plate_link, child caster_link, origin xyz=0.0267 0 -0.024 rpy=0 0 0, axis 0 0 1
- added joint left_rear_strut_left_side_cover_joint: type fixed, parent left_rear_strut_link, child LeftSideCover_link, origin xyz=0.229 0.026 0.447 rpy=0 0 0
- added joint left_rear_strut_link_left_rear_strut_link_inside_joint: type fixed, parent left_rear_strut_link, child left_rear_strut_inside_link, origin xyz=0 0 0 rpy=0 0 0
- added joint right_rear_strut_link_right_rear_strut_link_inside_joint: type fixed, parent right_rear_strut_link, child right_rear_strut_inside_link, origin xyz=0 0 0 rpy=0 0 0
- added joint right_right_strut_right_side_cover: type fixed, parent right_rear_strut_link, child RightSideCover_link, origin xyz=0.229 -0.026 0.447 rpy=0 0 0
- joint RearLeftStrutToCameraLift: parent RearRightStrut_link -> right_rear_strut_link
- joint RearLeftStrutToTopPlate: parent RearRightStrut_link -> right_rear_strut_link

Commit message: Refactoring.

File: carl_description/robots/carl.urdf (robot description, URDF)
Before this commit: robot carl, 29 links, 28 joints
Links:
- removed link Hokuyo_link
- removed link JacoMount_link
- removed link LeftSideCover_link
- removed link RightSideCover_link
- removed link TopPlate_link
- added link hokuyo_link; visual mesh filename=package://carl_description/meshes/hokuyo.dae
- added link jaco_mount_link; visual mesh filename=package://carl_description/meshes/jaco_mount.dae
- added link left_side_cover_link; visual mesh filename=package://carl_description/meshes/side_cover.dae
- added link right_side_cover_link; visual mesh filename=package://carl_description/meshes/side_cover.dae
- added link top_plate_link; collision box size=0.495 0.59 0.65; visual mesh filename=package://carl_description/meshes/table_plate.dae
Joints:
- removed joint RearLeftStrutToTopPlate
- removed joint TopPlateToJacoMount
- removed joint caster_hokuyo_joint
- removed joint left_rear_strut_left_side_cover_joint
- removed joint right_right_strut_right_side_cover
- added joint caster_plate_link_hokuyo_joint: type fixed, parent caster_plate_link, child hokuyo_link, origin xyz=0.07 0 0.035 rpy=0 0 0
- added joint left_rear_strut_link_left_side_cover_joint: type fixed, parent left_rear_strut_link, child left_side_cover_link, origin xyz=0.229 -0.026 0.447 rpy=0 0 0
- added joint left_rear_strut_top_plate_joint: type fixed, parent right_rear_strut_link, child top_plate_link, origin xyz=0.516 0.20 0.598 rpy=0 0 0
- added joint right_rear_strut_link_right_side_cover_joint: type fixed, parent right_rear_strut_link, child right_side_cover_link, origin xyz=0.229 -0.026 0.447 rpy=0 0 0
- added joint top_plate_jaco_mount: type fixed, parent top_plate_link, child jaco_mount_link, origin xyz=0 0 -0.13 rpy=0 0 0
- joint jaco_joint_base: parent JacoMount_link -> jaco_mount_link

File: carl_description/robots/carl.urdf.xacro (robot description, xacro)
@@ -5,4 +5,4 @@
   <xacro:include filename="$(find jaco_model)/urdf/jaco_arm.xacro" />
   <xacro:carl_base name="base"/>
-  <xacro:jaco_arm  parent="JacoMount_link"/>
+  <xacro:jaco_arm  parent="jaco_mount_link"/>
 </robot>

File: carl_description/urdf/carl_base/carl_base.urdf.xacro (robot description, xacro)
@@ -7,4 +7,6 @@
 <xacro:include filename="$(find carl_description)/urdf/components/carl_rear_strut.urdf.xacro" />
 <xacro:include filename="$(find carl_description)/urdf/components/carl_caster_assembly.urdf.xacro" />
+<xacro:include filename="$(find carl_description)/urdf/components/carl_side_cover.urdf.xacro" />
+<xacro:include filename="$(find carl_description)/urdf/sensors/hokuyo.urdf.xacro" />
 <xacro:macro name="carl_base" params="name">
   <link name="${name}_link">
@@ -16,5 +18,5 @@
     </visual>
   </link>
-  <link name="TopPlate_link">
+  <link name="top_plate_link">
     <visual>
       <origin xyz="0 0 0" rpy="0 0 -1.5708" />
@@ -61,33 +63,9 @@
     </collision>
   </link>
-  <link name="JacoMount_link">
+  <link name="jaco_mount_link">
     <visual>
       <origin xyz="0 0 0" rpy="0 0 1.5708" />
       <geometry>
         <mesh filename="package://carl_description/meshes/jaco_mount.dae" />
-      </geometry>
-    </visual>
-  </link>
-  <link name="Hokuyo_link">
-    <visual>
-      <origin xyz="0 0 0" rpy="0 0 0" />
-      <geometry>
-        <mesh filename="package://carl_description/meshes/hokuyo.dae" />
-      </geometry>
-    </visual>
-  </link>
-   <link name="LeftSideCover_link">
-    <visual>
-      <origin xyz="0 0 0" rpy="0 0 1.5708" />
-      <geometry>
-        <mesh filename="package://carl_description/meshes/side_cover.dae" />
-      </geometry>
-    </visual>
-  </link>
-   <link name="RightSideCover_link">
-    <visual>
-      <origin xyz="0 0 0" rpy="0 0 1.5708" />
-      <geometry>
-        <mesh filename="package://carl_description/meshes/side_cover.dae" />
       </geometry>
     </visual>
@@ -136,7 +114,7 @@
      <origin xyz="-0.222 -0.200 -0.102" rpy="0 0 0" />
    </xacro:carl_rear_strut>
-  <joint name="RearLeftStrutToTopPlate" type="fixed">
+  <joint name="left_rear_strut_top_plate_joint" type="fixed">
     <parent link="right_rear_strut_link"/>
-    <child link="TopPlate_link"/>
+    <child link="top_plate_link"/>
     <origin xyz="0.516 0.20 0.598" rpy="0 0 0" />
   </joint>
@@ -157,24 +135,21 @@
     <origin xyz="0.11 0 -0.10" rpy="0 0 0" />
   </joint>
-  <joint name="TopPlateToJacoMount" type="fixed">
-    <parent link="TopPlate_link"/>
-    <child link="JacoMount_link"/>
+  <joint name="top_plate_jaco_mount" type="fixed">
+    <parent link="top_plate_link"/>
+    <child link="jaco_mount_link"/>
     <origin xyz="0 0 -0.13" rpy="0 0 0" />
   </joint>
-  <joint name="caster_hokuyo_joint" type="fixed">
-    <parent link="caster_plate_link"/>
-    <child link="Hokuyo_link"/>
-    <origin xyz="0.07 0 0.035" rpy="0 0 0" />
-  </joint>
-  <joint name="left_rear_strut_left_side_cover_joint" type="fixed">
-    <parent link="left_rear_strut_link"/>
-    <child link="LeftSideCover_link"/>
-    <origin xyz="0.229 0.026 0.447" rpy="0 0 0" />
-  </joint>
-  <joint name="right_right_strut_right_side_cover" type="fixed">
-    <parent link="right_rear_strut_link"/>
-    <child link="RightSideCover_link"/>
-    <origin xyz="0.229 -0.026 0.447" rpy="0 0 0" />
-  </joint>
+   <!-- hokuyo -->
+   <xacro:hokuyo parent="caster_plate_link">
+     <origin xyz="0.07 0 0.035" rpy="0 0 0" />
+   </xacro:hokuyo>
+   <!-- right side cover -->
+   <xacro:carl_side_cover suffix="right" parent="right_rear_strut_link">
+     <origin xyz="0.229 -0.026 0.447" rpy="0 0 0" />
+   </xacro:carl_side_cover>
+   <!-- left side cover -->
+   <xacro:carl_side_cover suffix="left" parent="left_rear_strut_link">
+     <origin xyz="0.229 -0.026 0.447" rpy="0 0 0" />
+   </xacro:carl_side_cover>
   <joint name="${name}_front_cover_joint" type="fixed">
     <parent link="${name}_link"/>

Commit message: Refactoring

File: carl_description/robots/carl.urdf (robot description, URDF)
Before this commit: robot carl, 29 links, 28 joints
Links:
- removed link CameraLift_link
- removed link CameraTiltBracket_link
- removed link CameraTiltPlate_link
- added link camera_lift_link; collision mesh filename=package://carl_description/meshes/camera_lift.dae; visual mesh filename=package://carl_description/meshes/camera_lift.dae
- added link camera_tilt_bracket_link
- added link camera_tilt_plate_link; collision mesh filename=package://carl_description/meshes/camera_plate.dae; visual mesh filename=package://carl_description/meshes/camera_plate.dae
Joints:
- removed joint CameraLiftBracketToCameraTiltPlate
- removed joint CameraLiftToCameraTiltBracket
- removed joint RearLeftStrutToCameraLift
- added joint camera_lift_bracket_camera_tilt_plate_joint: type fixed, parent camera_tilt_bracket_link, child camera_tilt_plate_link, origin xyz=0.11 0 -0.10 rpy=0 0 0
- added joint camera_lift_camera_tilt_bracket_joint: type continuous, parent camera_lift_link, child camera_tilt_bracket_link, origin xyz=0.03 -0.10 0 rpy=1.5708 0 0, axis 0 0 1
- added joint left_rear_strut_camera_lift_joint: type fixed, parent right_rear_strut_link, child camera_lift_link, origin xyz=0.01 0.20 1.461 rpy=0 0 0

File: carl_description/urdf/carl_base/carl_base.urdf.xacro (robot description, xacro)
@@ -4,83 +4,38 @@
         xmlns:interface="http://playerstage.sourceforge.net/gazebo/xmlschema/#interface"
         xmlns:xacro="http://ros.org/wiki/xacro">
-<xacro:include filename="$(find carl_description)/urdf/components/carl_wheel.urdf.xacro" />
-<xacro:include filename="$(find carl_description)/urdf/components/carl_caster_assembly.urdf.xacro" />
-<xacro:include filename="$(find carl_description)/urdf/sensors/hokuyo.urdf.xacro" />
-<xacro:include filename="$(find carl_description)/urdf/carl_base/carl_superstructure.urdf.xacro" />
-<xacro:include filename="$(find carl_description)/urdf/carl_base/carl_covers.urdf.xacro" />
-<xacro:macro name="carl_base" params="name">
-  <xacro:carl_superstructure/>
-  <xacro:carl_covers name="${name}"/>
-  <link name="${name}_link">
-   <visual>
-      <origin xyz="0 0 0" rpy="0 0 0"/>
-      <geometry>
-        <mesh filename="package://carl_description/meshes/base.dae" />
-      </geometry>
-    </visual>
-  </link>
-  <link name="CameraLift_link">
-    <visual>
-      <origin xyz="0 0 0" rpy="0 0 1.5708" />
-      <geometry>
-        <mesh filename="package://carl_description/meshes/camera_lift.dae" />
-      </geometry>
-    </visual>
-    <collision>
-      <origin xyz="0 0 0" rpy="0 0 1.5708" />
-      <geometry>
-        <mesh filename="package://carl_description/meshes/camera_lift.dae" />
-      </geometry>
-    </collision>
-  </link>
-  <link name="CameraTiltBracket_link">
-	<!--exists to move center of rotation for camera mount-->
-  </link>
-  <link name="CameraTiltPlate_link">
-    <visual>
-      <origin xyz="0 0 0" rpy="0 1.5708 0" />
-      <geometry>
-        <mesh filename="package://carl_description/meshes/camera_plate.dae" />
-      </geometry>
-    </visual>
-    <collision>
-      <origin xyz="0 0 0" rpy="0 1.5708 0" />
-      <geometry>
-        <mesh filename="package://carl_description/meshes/camera_plate.dae" />
-      </geometry>
-    </collision>
-  </link>
-   <!-- left wheel -->
-   <xacro:carl_wheel suffix="left" parent="${name}_link">
-     <origin xyz="0 0.25 0" rpy="-1.5708 0 0" />
-   </xacro:carl_wheel>
-   <!-- right wheel -->
-   <xacro:carl_wheel suffix="right" parent="${name}_link">
-     <origin xyz="0 -0.25 0" rpy="1.5708 0 0" />
-   </xacro:carl_wheel>
-   <!-- caster assembly -->
-   <xacro:carl_caster_assembly parent="${name}_link">
-     <origin xyz="0.2883 0 0" rpy="0 0 0" />
-   </xacro:carl_caster_assembly>
-  <joint name="RearLeftStrutToCameraLift" type="fixed">
-    <parent link="right_rear_strut_link"/>
-    <child link="CameraLift_link"/>
-    <origin xyz="0.01 0.20 1.461" rpy="0 0 0" />
-  </joint>
-  <joint name="CameraLiftToCameraTiltBracket" type="continuous">
-    <parent link="CameraLift_link"/>
-    <child link="CameraTiltBracket_link"/>
-    <origin xyz="0.03 -0.10 0" rpy="1.5708 0 0" />
-    <axis xyz="0 0 1" />
-  </joint>
-  <joint name="CameraLiftBracketToCameraTiltPlate" type="fixed">
-    <parent link="CameraTiltBracket_link"/>
-    <child link="CameraTiltPlate_link"/>
-    <origin xyz="0.11 0 -0.10" rpy="0 0 0" />
-  </joint>
-   <!-- hokuyo -->
-   <xacro:hokuyo parent="caster_plate_link">
-     <origin xyz="0.07 0 0.035" rpy="0 0 0" />
-   </xacro:hokuyo>
-</xacro:macro>
+  <xacro:include filename="$(find carl_description)/urdf/components/carl_wheel.urdf.xacro" />
+  <xacro:include filename="$(find carl_description)/urdf/components/carl_caster_assembly.urdf.xacro" />
+  <xacro:include filename="$(find carl_description)/urdf/sensors/hokuyo.urdf.xacro" />
+  <xacro:include filename="$(find carl_description)/urdf/carl_base/carl_superstructure.urdf.xacro" />
+  <xacro:include filename="$(find carl_description)/urdf/carl_base/carl_covers.urdf.xacro" />
+  <xacro:include filename="$(find carl_description)/urdf/carl_base/carl_camera_mount.urdf.xacro" />
+  <xacro:macro name="carl_base" params="name">
+    <xacro:carl_superstructure/>
+    <xacro:carl_camera_mount/>
+    <xacro:carl_covers name="${name}"/>
+    <link name="${name}_link">
+     <visual>
+        <origin xyz="0 0 0" rpy="0 0 0"/>
+        <geometry>
+          <mesh filename="package://carl_description/meshes/base.dae" />
+        </geometry>
+      </visual>
+    </link>
+     <!-- left wheel -->
+     <xacro:carl_wheel suffix="left" parent="${name}_link">
+       <origin xyz="0 0.25 0" rpy="-1.5708 0 0" />
+     </xacro:carl_wheel>
+     <!-- right wheel -->
+     <xacro:carl_wheel suffix="right" parent="${name}_link">
+       <origin xyz="0 -0.25 0" rpy="1.5708 0 0" />
+     </xacro:carl_wheel>
+     <!-- caster assembly -->
+     <xacro:carl_caster_assembly parent="${name}_link">
+       <origin xyz="0.2883 0 0" rpy="0 0 0" />
+     </xacro:carl_caster_assembly>
+     <!-- hokuyo -->
+     <xacro:hokuyo parent="caster_plate_link">
+       <origin xyz="0.07 0 0.035" rpy="0 0 0" />
+     </xacro:hokuyo>
+  </xacro:macro>
 </robot>

Commit message: Added asus xtion.

File: carl_description/robots/carl.urdf (robot description, URDF)
Before this commit: robot carl, 29 links, 28 joints
Links:
- added link camera_depth_frame, mass 0.01
- added link camera_depth_optical_frame, mass 0.001
- added link camera_link, mass 0.01; collision box size=0.0730 .2760 0.0720; visual mesh filename=package://carl_description/meshes/asus_xtion_pro_live.dae scale=0.001 0.001 0.001
- added link camera_rgb_frame, mass 0.001
- added link camera_rgb_optical_frame, mass 0.001
Joints:
- added joint camera_depth_joint: type fixed, parent camera_rgb_frame, child camera_depth_frame, origin xyz=0 0.027 0 rpy=0 0 0
- added joint camera_depth_optical_joint: type fixed, parent camera_depth_frame, child camera_depth_optical_frame, origin xyz=0 0 0 rpy=-1.57079632679 0 -1.57079632679
- added joint camera_joint: type fixed, parent camera_rgb_frame, child camera_link, origin xyz=0 -0.022 0 rpy=0 0 0
- added joint camera_rgb_joint: type fixed, parent camera_tilt_plate_link, child camera_rgb_frame, origin xyz=.025 -.02 -.02 rpy=-1.5708 0 -1.5708
- added joint camera_rgb_optical_joint: type fixed, parent camera_rgb_frame, child camera_rgb_optical_frame, origin xyz=0 0 0 rpy=-1.57079632679 0 -1.57079632679

File: carl_description/urdf/carl_base/carl_camera_mount.urdf.xacro (robot description, xacro)
@@ -4,5 +4,9 @@
         xmlns:interface="http://playerstage.sourceforge.net/gazebo/xmlschema/#interface"
         xmlns:xacro="http://ros.org/wiki/xacro">
+  <xacro:include filename="$(find carl_description)/urdf/sensors/asus_xtion_pro.urdf.xacro" />
   <xacro:macro name="carl_camera_mount">
+    <xacro:sensor_asus_xtion_pro parent="camera_tilt_plate_link">
+	      <origin xyz=".025 -.02 -.02" rpy="-1.5708 0 -1.5708" />
+	</xacro:sensor_asus_xtion_pro>
     <link name="camera_lift_link">
       <visual>

Commit message: Changed initial pose of caster and repositioned cover.

File: carl_description/robots/carl.urdf (robot description, URDF)
Before this commit: robot carl, 34 links, 33 joints
Joints:
- joint left_rear_strut_link_left_side_cover_joint: origin xyz=0.229 -0.026 0.447 rpy=0 0 0 -> xyz=0.229 0.026 0.447 rpy=0 0 0

File: carl_description/urdf/carl_base/carl_covers.urdf.xacro (robot description, xacro)
@@ -12,5 +12,5 @@
     <!-- left side cover -->
     <xacro:carl_side_cover suffix="left" parent="left_rear_strut_link">
-      <origin xyz="0.229 -0.026 0.447" rpy="0 0 0" />
+      <origin xyz="0.229 0.026 0.447" rpy="0 0 0" />
     </xacro:carl_side_cover>
     <joint name="${name}_front_cover_joint" type="fixed">

File: carl_description/urdf/components/carl_caster_assembly.urdf.xacro (robot description, xacro)
@@ -23,5 +23,5 @@
     <link name="caster_link">
       <visual>
-        <origin xyz="0 0 0" rpy="0 0 1.5708"/>
+        <origin xyz="0 0 0" rpy="0 0 0"/>
         <geometry>
           <mesh filename="package://carl_description/meshes/caster.dae" />

Commit message: carl_description updated to use jaco_description instead of jaco_model, more carl_teleop cleanup

File: carl_description/robots/carl.urdf (robot description, URDF)
Before this commit: robot carl, 34 links, 33 joints
Links:
- removed link camera_depth_frame
- removed link camera_depth_optical_frame
- removed link camera_rgb_frame
- removed link camera_rgb_optical_frame
- added link base_footprint
- link jaco_link_1: geometry collision mesh filename=package://jaco_description/meshes/jaco_link_1.dae; visual mesh filename=package://jaco_description/meshes/jaco_link_1.dae
- link jaco_link_2: geometry collision mesh filename=package://jaco_description/meshes/jaco_link_2.dae; visual mesh filename=package://jaco_description/meshes/jaco_link_2.dae
- link jaco_link_3: geometry collision mesh filename=package://jaco_description/meshes/jaco_link_3.dae; visual mesh filename=package://jaco_description/meshes/jaco_link_3.dae
- link jaco_link_4: geometry collision mesh filename=package://jaco_description/meshes/jaco_link_4.dae; visual mesh filename=package://jaco_description/meshes/jaco_link_4.dae
- link jaco_link_5: geometry collision mesh filename=package://jaco_description/meshes/jaco_link_5.dae; visual mesh filename=package://jaco_description/meshes/jaco_link_5.dae
- link jaco_link_base: geometry collision mesh filename=package://jaco_description/meshes/jaco_link_base.dae; visual mesh filename=package://jaco_description/meshes/jaco_link_base.dae
- link jaco_link_finger_1: geometry collision mesh filename=package://jaco_description/meshes/jaco_link_finger_1.dae; visual mesh filename=package://jaco_description/meshes/jaco_link_finger_1.dae
- link jaco_link_finger_2: geometry collision mesh filename=package://jaco_description/meshes/jaco_link_finger_2.dae; visual mesh filename=package://jaco_description/meshes/jaco_link_finger_2.dae
- link jaco_link_finger_3: geometry collision mesh filename=package://jaco_description/meshes/jaco_link_finger_3.dae; visual mesh filename=package://jaco_description/meshes/jaco_link_finger_3.dae
- link jaco_link_hand: geometry collision mesh filename=package://jaco_description/meshes/jaco_link_hand.dae; visual mesh filename=package://jaco_description/meshes/jaco_link_hand.dae
Joints:
- removed joint camera_depth_joint
- removed joint camera_depth_optical_joint
- removed joint camera_rgb_joint
- removed joint camera_rgb_optical_joint
- added joint base_footprint_base_link_joint: type fixed, parent base_footprint, child base_link, origin xyz=0 0 0.23114 rpy=0 0 0
- joint camera_joint: origin xyz=0 -0.022 0 rpy=0 0 0 -> xyz=.025 -.02 -.02 rpy=-1.5708 0 -1.5708; parent camera_rgb_frame -> camera_tilt_plate_link
- joint camera_lift_camera_tilt_bracket_joint: origin xyz=0.03 -0.10 0 rpy=1.5708 0 0 -> xyz=0.03 -0.10 0 rpy=1.5708 -1.5708 0
- joint jaco_joint_1: limit (none) -> lower=-6.28318530718 upper=6.28318530718 effort=30 velocity=5; type continuous -> revolute
- joint jaco_joint_2: limit (none) -> lower=0 upper=6.28318530718 effort=30 velocity=5; type continuous -> revolute
- joint jaco_joint_3: limit (none) -> lower=0 upper=6.28318530718 effort=30 velocity=5; type continuous -> revolute
- joint jaco_joint_4: limit (none) -> lower=-6.28318530718 upper=6.28318530718 effort=30 velocity=5; type continuous -> revolute
- joint jaco_joint_5: limit (none) -> lower=-6.28318530718 upper=6.28318530718 effort=30 velocity=5; type continuous -> revolute
- joint jaco_joint_6: limit (none) -> lower=-6.28318530718 upper=6.28318530718 effort=30 velocity=5; type continuous -> revolute
- joint jaco_joint_base: limit (none) -> lower=-6.28318530718 upper=6.28318530718 effort=30 velocity=5
- joint jaco_joint_finger_2: origin xyz=0.03569 -0.0216 -0.10071 rpy=-1.6222 1.117 -0.23615 -> xyz=0.03569 0.0216 -0.10071 rpy=-1.5161 1.1459 0.23978
- joint jaco_joint_finger_3: origin xyz=0.03569 0.0216 -0.10071 rpy=-1.5161 1.1459 0.23978 -> xyz=0.03569 -0.0216 -0.10071 rpy=-1.6222 1.117 -0.23615
