Commit message: cleanup of carl_description

File: carl_description/robots/carl.urdf (robot description, URDF)
Before this commit: robot carl, 31 links, 30 joints
Links:
- removed link camera_tilt_bracket_link
- removed link camera_tilt_plate_link
- added link camera_mount_link; visual mesh filename=package://carl_description/meshes/camera_mount.dae
- added link left_rear_strut_top_link; collision box size=0.027 0.054 0.4575; visual mesh filename=package://carl_description/meshes/rear_strut_top.dae
- added link right_rear_strut_top_link; collision box size=0.027 0.054 0.4575; visual mesh filename=package://carl_description/meshes/rear_strut_top.dae
- added link servo_arm_link; collision box size=0.035 0.05 0.06; visual mesh filename=package://carl_description/meshes/servo_arm.dae
- added link servo_link; collision box size=0.06 0.05 0.035; visual mesh filename=package://carl_description/meshes/servo.dae
- added link servo_mount_link; collision box size=0.08 0.055 0.09; visual mesh filename=package://carl_description/meshes/servo_mount.dae
- link camera_lift_link: geometry collision box size=0.027 0.454 0.054; visual mesh filename=package://carl_description/meshes/camera_lift.dae
- link camera_link: geometry collision box size=0.0830 .2760 0.0720; visual mesh filename=package://carl_description/meshes/asus_xtion_pro_live.dae scale=0.001 0.001 0.001
Joints:
- removed joint camera_lift_bracket_camera_tilt_plate_joint
- removed joint camera_lift_camera_tilt_bracket_joint
- added joint camera_lift_servo_mount_joint: type fixed, parent camera_lift_link, child servo_mount_link, origin xyz=0 0 0 rpy=1.5708 0 0, axis 0 0 1
- added joint left_rear_strut_link_left_rear_strut_top_link_joint: type fixed, parent left_rear_strut_link, child left_rear_strut_top_link, origin xyz=0 0.001 1.055 rpy=0 0 0
- added joint right_rear_strut_link_right_rear_strut_top_link_joint: type fixed, parent right_rear_strut_link, child right_rear_strut_top_link, origin xyz=0 0.001 1.055 rpy=0 0 0
- added joint servo_arm_camera_mount_joint: type fixed, parent servo_arm_link, child camera_mount_link, origin xyz=0 -0.053 -0.016 rpy=1.5708 0 1.5708
- added joint servo_mount_servo_joint: type fixed, parent servo_mount_link, child servo_link, origin xyz=0.073 0.013 0.0187 rpy=1.5708 0 3.92699
- added joint servo_servo_arm_joint: type continuous, parent servo_link, child servo_arm_link, origin xyz=0 -0.042 0 rpy=1.5708 1.5708 0, axis 0 0 1
- joint camera_joint: origin xyz=.025 -.02 -.02 rpy=-1.5708 0 -1.5708 -> xyz=-0.016 -0.008 0.018 rpy=0 -1.5708 0; parent camera_tilt_plate_link -> camera_mount_link
- joint left_rear_strut_camera_lift_joint: origin xyz=0.01 0.20 1.461 rpy=0 0 0 -> xyz=0.013 0.20 1.538 rpy=0 0 0

File: carl_description/robots/carl.urdf.xacro (robot description, xacro)
@@ -3,5 +3,5 @@
   <xacro:include filename="$(find carl_description)/urdf/carl_base/carl_base.urdf.xacro" />
   <xacro:include filename="$(find jaco_description)/urdf/jaco_arm.xacro" />
-  <xacro:carl_base name="base"/>
-  <xacro:jaco_arm  parent="jaco_mount_link"/>
+  <xacro:carl_base name="base" />
+  <xacro:jaco_arm  parent="jaco_mount_link" />
 </robot>

File: carl_description/urdf/carl_base/carl_base.urdf.xacro (robot description, xacro)
@@ -1,7 +1,7 @@
 <?xml version="1.0"?>
 <robot xmlns:sensor="http://playerstage.sourceforge.net/gazebo/xmlschema/#sensor"
-        xmlns:controller="http://playerstage.sourceforge.net/gazebo/xmlschema/#controller"
-        xmlns:interface="http://playerstage.sourceforge.net/gazebo/xmlschema/#interface"
-        xmlns:xacro="http://ros.org/wiki/xacro">
+       xmlns:controller="http://playerstage.sourceforge.net/gazebo/xmlschema/#controller"
+       xmlns:interface="http://playerstage.sourceforge.net/gazebo/xmlschema/#interface"
+       xmlns:xacro="http://ros.org/wiki/xacro">
   <xacro:include filename="$(find carl_description)/urdf/components/carl_wheel.urdf.xacro" />
   <xacro:include filename="$(find carl_description)/urdf/components/carl_caster_assembly.urdf.xacro" />
@@ -11,13 +11,13 @@
   <xacro:include filename="$(find carl_description)/urdf/carl_base/carl_camera_mount.urdf.xacro" />
   <xacro:macro name="carl_base" params="name">
-    <xacro:carl_superstructure/>
-    <xacro:carl_camera_mount/>
-    <xacro:carl_covers name="${name}"/>
+    <xacro:carl_superstructure />
+    <xacro:carl_camera_mount />
+    <xacro:carl_covers name="${name}" />
     <!-- base footprint -->
-    <link name="${name}_footprint"/>
+    <link name="${name}_footprint" />
   	<!-- base link -->
     <link name="${name}_link">
      <visual>
-        <origin xyz="0 0 0" rpy="0 0 0"/>
+        <origin xyz="0 0 0" rpy="0 0 0" />
         <geometry>
           <mesh filename="package://carl_description/meshes/base.dae" />
@@ -26,6 +26,6 @@
     </link>
     <joint name="${name}_footprint_${name}_link_joint" type="fixed">
-      <parent link="${name}_footprint"/>
-      <child link="${name}_link"/>
+      <parent link="${name}_footprint" />
+      <child link="${name}_link" />
       <origin xyz="0 0 0.23114" rpy="0 0 0" />
     </joint>

File: carl_description/urdf/carl_base/carl_camera_mount.urdf.xacro (robot description, xacro)
@@ -1,7 +1,7 @@
 <?xml version="1.0"?>
 <robot xmlns:sensor="http://playerstage.sourceforge.net/gazebo/xmlschema/#sensor"
-        xmlns:controller="http://playerstage.sourceforge.net/gazebo/xmlschema/#controller"
-        xmlns:interface="http://playerstage.sourceforge.net/gazebo/xmlschema/#interface"
-        xmlns:xacro="http://ros.org/wiki/xacro">
+       xmlns:controller="http://playerstage.sourceforge.net/gazebo/xmlschema/#controller"
+       xmlns:interface="http://playerstage.sourceforge.net/gazebo/xmlschema/#interface"
+       xmlns:xacro="http://ros.org/wiki/xacro">
   <xacro:include filename="$(find carl_description)/urdf/sensors/asus_xtion_pro.urdf.xacro" />
   <xacro:macro name="carl_camera_mount">
@@ -74,28 +74,28 @@
     </xacro:sensor_asus_xtion_pro>
     <joint name="left_rear_strut_camera_lift_joint" type="fixed">
-      <parent link="right_rear_strut_link"/>
-      <child link="camera_lift_link"/>
+      <parent link="right_rear_strut_link" />
+      <child link="camera_lift_link" />
       <origin xyz="0.013 0.20 1.538" rpy="0 0 0" />
     </joint>
     <joint name="camera_lift_servo_mount_joint" type="fixed">
-      <parent link="camera_lift_link"/>
-      <child link="servo_mount_link"/>
+      <parent link="camera_lift_link" />
+      <child link="servo_mount_link" />
       <origin xyz="0 0 0" rpy="1.5708 0 0" />
       <axis xyz="0 0 1" />
     </joint>
     <joint name="servo_mount_servo_joint" type="fixed">
-      <parent link="servo_mount_link"/>
-      <child link="servo_link"/>
+      <parent link="servo_mount_link" />
+      <child link="servo_link" />
       <origin xyz="0.073 0.013 0.0187" rpy="1.5708 0 3.92699" />
     </joint>
     <joint name="servo_servo_arm_joint" type="continuous">
-      <parent link="servo_link"/>
-      <child link="servo_arm_link"/>
+      <parent link="servo_link" />
+      <child link="servo_arm_link" />
       <origin xyz="0 -0.042 0" rpy="1.5708 1.5708 0" />
       <axis xyz="0 0 1" />
     </joint>
     <joint name="servo_arm_camera_mount_joint" type="fixed">
-      <parent link="servo_arm_link"/>
-      <child link="camera_mount_link"/>
+      <parent link="servo_arm_link" />
+      <child link="camera_mount_link" />
       <origin xyz="0 -0.053 -0.016" rpy="1.5708 0 1.5708" />
     </joint>

File: carl_description/urdf/carl_base/carl_covers.urdf.xacro (robot description, xacro)
@@ -1,7 +1,7 @@
 <?xml version="1.0"?>
 <robot xmlns:sensor="http://playerstage.sourceforge.net/gazebo/xmlschema/#sensor"
-        xmlns:controller="http://playerstage.sourceforge.net/gazebo/xmlschema/#controller"
-        xmlns:interface="http://playerstage.sourceforge.net/gazebo/xmlschema/#interface"
-        xmlns:xacro="http://ros.org/wiki/xacro">
+       xmlns:controller="http://playerstage.sourceforge.net/gazebo/xmlschema/#controller"
+       xmlns:interface="http://playerstage.sourceforge.net/gazebo/xmlschema/#interface"
+       xmlns:xacro="http://ros.org/wiki/xacro">
   <xacro:include filename="$(find carl_description)/urdf/components/carl_side_cover.urdf.xacro" />
   <xacro:macro name="carl_covers" params="name">
@@ -15,11 +15,11 @@
     </xacro:carl_side_cover>
     <joint name="${name}_front_cover_joint" type="fixed">
-      <parent link="${name}_link"/>
-      <child link="FrontCover_link"/>
+      <parent link="${name}_link" />
+      <child link="FrontCover_link" />
       <origin xyz=".247 0 0.242" rpy="0 0 0" />
     </joint>
     <joint name="${name}_back_cover" type="fixed">
-      <parent link="${name}_link"/>
-      <child link="BackCover_link"/>
+      <parent link="${name}_link" />
+      <child link="BackCover_link" />
       <origin xyz="-.237 0 -0.102" rpy="0 0 0" />
     </joint>

File: carl_description/urdf/carl_base/carl_superstructure.urdf.xacro (robot description, xacro)
@@ -1,7 +1,7 @@
 <?xml version="1.0"?>
 <robot xmlns:sensor="http://playerstage.sourceforge.net/gazebo/xmlschema/#sensor"
-        xmlns:controller="http://playerstage.sourceforge.net/gazebo/xmlschema/#controller"
-        xmlns:interface="http://playerstage.sourceforge.net/gazebo/xmlschema/#interface"
-        xmlns:xacro="http://ros.org/wiki/xacro">
+       xmlns:controller="http://playerstage.sourceforge.net/gazebo/xmlschema/#controller"
+       xmlns:interface="http://playerstage.sourceforge.net/gazebo/xmlschema/#interface"
+       xmlns:xacro="http://ros.org/wiki/xacro">
   <xacro:include filename="$(find carl_description)/urdf/components/carl_rear_strut.urdf.xacro" />
   <xacro:macro name="carl_superstructure">
@@ -15,11 +15,11 @@
     </xacro:carl_rear_strut>
     <joint name="left_rear_strut_top_plate_joint" type="fixed">
-      <parent link="right_rear_strut_link"/>
-      <child link="top_plate_link"/>
+      <parent link="right_rear_strut_link" />
+      <child link="top_plate_link" />
       <origin xyz="0.516 0.20 0.598" rpy="0 0 0" />
     </joint>
     <joint name="top_plate_jaco_mount" type="fixed">
-      <parent link="top_plate_link"/>
-      <child link="jaco_mount_link"/>
+      <parent link="top_plate_link" />
+      <child link="jaco_mount_link" />
       <origin xyz="0 0 -0.13" rpy="0 0 0" />
     </joint>

File: carl_description/urdf/components/carl_caster_assembly.urdf.xacro (robot description, xacro)
@@ -1,13 +1,13 @@
 <?xml version="1.0"?>
-  <root xmlns:xacro="http://ros.org/wiki/xacro">
+<root xmlns:xacro="http://ros.org/wiki/xacro">
   <xacro:macro name="carl_caster_assembly" params="parent *origin">
     <joint name="${parent}_caster_plate_joint" type="fixed">
       <xacro:insert_block name="origin" />
-      <parent link="${parent}"/>
-      <child link="caster_plate_link"/>
+      <parent link="${parent}" />
+      <child link="caster_plate_link" />
     </joint>
     <joint name="caster_plate__caster_joint" type="continuous">
-      <parent link="caster_plate_link"/>
-      <child link="caster_link"/>
+      <parent link="caster_plate_link" />
+      <child link="caster_link" />
       <origin xyz="0.0267 0 -0.024" rpy="0 0 0" />
       <axis xyz="0 0 1" />
@@ -15,5 +15,5 @@
     <link name="caster_plate_link">
       <visual>
-        <origin xyz="0 0 0" rpy="0 0 1.5708"/>
+        <origin xyz="0 0 0" rpy="0 0 1.5708" />
         <geometry>
           <mesh filename="package://carl_description/meshes/caster_plate.dae" />
@@ -23,5 +23,5 @@
     <link name="caster_link">
       <visual>
-        <origin xyz="0 0 0" rpy="0 0 0"/>
+        <origin xyz="0 0 0" rpy="0 0 0" />
         <geometry>
           <mesh filename="package://carl_description/meshes/caster.dae" />

File: carl_description/urdf/components/carl_rear_strut.urdf.xacro (robot description, xacro)
@@ -8,11 +8,11 @@
     </joint>
     <joint name="${suffix}_rear_strut_link_${suffix}_rear_strut_link_inside_joint" type="fixed">
-      <parent link="${suffix}_rear_strut_link"/>
-   	  <child link="${suffix}_rear_strut_inside_link"/>
+      <parent link="${suffix}_rear_strut_link" />
+   	  <child link="${suffix}_rear_strut_inside_link" />
       <origin xyz="0 0 0" rpy="0 0 0" />
     </joint>
     <joint name="${suffix}_rear_strut_link_${suffix}_rear_strut_top_link_joint" type="fixed">
-      <parent link="${suffix}_rear_strut_link"/>
-   	  <child link="${suffix}_rear_strut_top_link"/>
+      <parent link="${suffix}_rear_strut_link" />
+   	  <child link="${suffix}_rear_strut_top_link" />
       <origin xyz="0 0.001 1.055" rpy="0 0 0" />
     </joint>

File: carl_description/urdf/components/carl_side_cover.urdf.xacro (robot description, xacro)
@@ -1,4 +1,4 @@
 <?xml version="1.0"?>
-  <root xmlns:xacro="http://ros.org/wiki/xacro">
+<root xmlns:xacro="http://ros.org/wiki/xacro">
   <xacro:macro name="carl_side_cover" params="suffix parent *origin">
     <joint name="${parent}_${suffix}_side_cover_joint" type="fixed">

File: carl_description/urdf/components/carl_wheel.urdf.xacro (robot description, xacro)
@@ -1,4 +1,4 @@
 <?xml version="1.0"?>
-  <root xmlns:xacro="http://ros.org/wiki/xacro">
+<root xmlns:xacro="http://ros.org/wiki/xacro">
   <xacro:macro name="carl_wheel" params="suffix parent *origin">
     <joint name="${parent}_${suffix}_wheel_joint" type="continuous">

File: carl_description/urdf/sensors/asus_xtion_pro.urdf.xacro (robot description, xacro)
@@ -1,7 +1,6 @@
 <?xml version="1.0"?>
-<!--borrowed and modified from turtlebot_description-->
 <robot name="sensor_asus_xtion_pro" xmlns:xacro="http://ros.org/wiki/xacro">
   <!-- Xacro properties -->
-  <xacro:property name="M_SCALE" value="0.001"/>
+  <xacro:property name="M_SCALE" value="0.001" />
   <xacro:property name="asus_xtion_pro_depth_rel_rgb_py" value="0.0270" />
   <xacro:property name="asus_xtion_pro_cam_rel_rgb_py"   value="-0.0220" />
@@ -10,12 +9,12 @@
     <joint name="camera_joint" type="fixed">
       <xacro:insert_block name="origin" />
-      <parent link="${parent}"/>
-      <child link="camera_link"/>
+      <parent link="${parent}" />
+      <child link="camera_link" />
     </joint>
     <link name="camera_link">
       <visual>
-        <origin xyz="-0.01 0 0" rpy="${-M_PI/2} -${M_PI} ${-M_PI/2}"/>
+        <origin xyz="-0.01 0 0" rpy="${-M_PI/2} -${M_PI} ${-M_PI/2}" />
         <geometry>
-          <mesh filename="package://carl_description/meshes/asus_xtion_pro_live.dae" scale="${M_SCALE} ${M_SCALE} ${M_SCALE}"/>
+          <mesh filename="package://carl_description/meshes/asus_xtion_pro_live.dae" scale="${M_SCALE} ${M_SCALE} ${M_SCALE}" />
         </geometry>
       </visual>
@@ -23,5 +22,5 @@
         <origin xyz="0.0 0.0 0.0" rpy="0 0 0" />
         <geometry>
-        <box size="0.0830 .2760 0.0720"/>
+        <box size="0.0830 .2760 0.0720" />
       </geometry>
       </collision>
@@ -29,67 +28,7 @@
         <mass value="0.01" />
         <origin xyz="0 0 0" />
-        <inertia ixx="0.001" ixy="0.0" ixz="0.0"
-          iyy="0.001" iyz="0.0"
-          izz="0.001" />
+        <inertia ixx="0.001" ixy="0.0" ixz="0.0" iyy="0.001" iyz="0.0" izz="0.001" />
       </inertial>
     </link>
-<!-- published by oppenni2_launch
-    <joint name="camera_rgb_joint" type="fixed">
-      <origin xyz="0 ${asus_xtion_pro_cam_rel_rgb_py} 0" rpy="0 0 0"/>
-      <parent link="camera_link"/>
-      <child link="camera_rgb_frame" />
-    </joint>
-    <link name="camera_rgb_frame">
-      <inertial>
-        <mass value="0.001" />
-        <origin xyz="0 0 0" />
-        <inertia ixx="0.0001" ixy="0.0" ixz="0.0"
-          iyy="0.0001" iyz="0.0"
-          izz="0.0001" />
-      </inertial>
-    </link>
-    <joint name="camera_rgb_optical_joint" type="fixed">
-      <origin xyz="0 0 0" rpy="${-M_PI/2} 0 ${-M_PI/2}" />
-      <parent link="camera_rgb_frame" />
-      <child link="camera_rgb_optical_frame" />
-    </joint>
-    <link name="camera_rgb_optical_frame">
-      <inertial>
-        <mass value="0.001" />
-        <origin xyz="0 0 0" />
-        <inertia ixx="0.0001" ixy="0.0" ixz="0.0"
-          iyy="0.0001" iyz="0.0"
-          izz="0.0001" />
-      </inertial>
-    </link>
-    <joint name="camera_depth_joint" type="fixed">
-      <origin xyz="0 ${asus_xtion_pro_depth_rel_rgb_py} 0" rpy="0 0 0" />
-      <parent link="camera_link" />
-      <child link="camera_depth_frame" />
-    </joint>
-    <link name="camera_depth_frame">
-      <inertial>
-        <mass value="0.01" />
-        <origin xyz="0 0 0" />
-        <inertia ixx="0.001" ixy="0.0" ixz="0.0"
-          iyy="0.001" iyz="0.0"
-          izz="0.001" />
-      </inertial>
-    </link>
-    <joint name="camera_depth_optical_joint" type="fixed">
-      <origin xyz="0 0 0" rpy="${-M_PI/2} 0 ${-M_PI/2}" />
-      <parent link="camera_depth_frame" />
-      <child link="camera_depth_optical_frame" />
-    </joint>
-    <link name="camera_depth_optical_frame">
-      <inertial>
-        <mass value="0.001" />
-        <origin xyz="0 0 0" />
-        <inertia ixx="0.0001" ixy="0.0" ixz="0.0"
-          iyy="0.0001" iyz="0.0"
-          izz="0.0001" />
-      </inertial>
-    </link>
-	-->
-    </xacro:macro>
+  </xacro:macro>
 </robot>

File: carl_description/urdf/sensors/hokuyo.urdf.xacro (robot description, xacro)
@@ -1,4 +1,4 @@
 <?xml version="1.0"?>
-  <root xmlns:xacro="http://ros.org/wiki/xacro">
+<root xmlns:xacro="http://ros.org/wiki/xacro">
   <xacro:macro name="hokuyo" params="parent *origin">
     <joint name="${parent}_hokuyo_joint" type="fixed">

Commit message: READMEs and Travis build

File: carl_description/robots/carl.urdf (robot description, URDF)
Before this commit: robot carl, 35 links, 34 joints
Links:
- link BackCover_link: geometry visual mesh filename=package://carl_description/meshes/back_cover.min.dae
- link FrontCover_link: geometry collision mesh filename=package://carl_description/meshes/front_cover_collision.stl; visual mesh filename=package://carl_description/meshes/front_cover.min.dae
- link base_link: geometry visual mesh filename=package://carl_description/meshes/base.min.dae
- link camera_lift_link: geometry collision box size=0.027 0.454 0.054; visual mesh filename=package://carl_description/meshes/camera_lift.min.dae
- link camera_link: geometry collision box size=0.0830 .2760 0.0720; visual mesh filename=package://carl_description/meshes/asus_xtion_pro_live.min.d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 scale=0.001 0.001 0.001
- link camera_mount_link: geometry visual mesh filename=package://carl_description/meshes/camera_mount.min.dae
- link caster_link: geometry collision cylinder length=0.213 radius=0.116; visual mesh filename=package://carl_description/meshes/caster.min.dae
- link caster_plate_link: geometry visual mesh filename=package://carl_description/meshes/caster_plate.min.dae
- link hokuyo_link: geometry visual mesh filename=package://carl_description/meshes/hokuyo.min.dae
- link jaco_mount_link: geometry visual mesh filename=package://carl_description/meshes/jaco_mount.min.dae
- link left_rear_strut_link: geometry collision box size=0.027 0.054 1.055; visual mesh filename=package://carl_description/meshes/rear_strut.min.dae
- link left_rear_strut_top_link: geometry collision box size=0.027 0.054 0.4575; visual mesh filename=package://carl_description/meshes/rear_strut_top.min.dae
- link left_side_cover_link: geometry visual mesh filename=package://carl_description/meshes/side_cover.min.dae
- link left_wheel_link: geometry collision cylinder length=0.1 radius=0.25; visual mesh filename=package://carl_description/meshes/wheel.min.dae
- link right_rear_strut_link: geometry collision box size=0.027 0.054 1.055; visual mesh filename=package://carl_description/meshes/rear_strut.min.dae
- link right_rear_strut_top_link: geometry collision box size=0.027 0.054 0.4575; visual mesh filename=package://carl_description/meshes/rear_strut_top.min.dae
- link right_side_cover_link: geometry visual mesh filename=package://carl_description/meshes/side_cover.min.dae
- link right_wheel_link: geometry collision cylinder length=0.1 radius=0.25; visual mesh filename=package://carl_description/meshes/wheel.min.dae
- link servo_arm_link: geometry collision box size=0.035 0.05 0.06; visual mesh filename=package://carl_description/meshes/servo_arm.min.dae
- link servo_link: geometry collision box size=0.06 0.05 0.035; visual mesh filename=package://carl_description/meshes/servo.min.dae
- link servo_mount_link: geometry collision box size=0.08 0.055 0.09; visual mesh filename=package://carl_description/meshes/servo_mount.min.dae
- link top_plate_link: geometry collision box size=0.495 0.59 0.65; visual mesh filename=package://carl_description/meshes/table_plate.min.dae
