Commit message: recompiled URDF

File: carl_description/robots/carl.urdf (robot description, URDF)
Before this commit: robot carl, 35 links, 34 joints
Links:
- added link jaco_link_finger_tip_1; collision mesh filename=package://jaco_description/meshes/jaco_link_finger_tip_1.dae; visual mesh filename=package://jaco_description/meshes/jaco_link_finger_tip_1.dae
- added link jaco_link_finger_tip_2; collision mesh filename=package://jaco_description/meshes/jaco_link_finger_tip_2.dae; visual mesh filename=package://jaco_description/meshes/jaco_link_finger_tip_2.dae
- added link jaco_link_finger_tip_3; collision mesh filename=package://jaco_description/meshes/jaco_link_finger_tip_3.dae; visual mesh filename=package://jaco_description/meshes/jaco_link_finger_tip_3.dae
- added link large_ring_cover_1; collision mesh filename=package://jaco_description/meshes/large_ring_cover.dae; visual mesh filename=package://jaco_description/meshes/large_ring_cover.dae
- added link large_ring_cover_2; collision mesh filename=package://jaco_description/meshes/large_ring_cover.dae; visual mesh filename=package://jaco_description/meshes/large_ring_cover.dae
- added link large_ring_cover_3; collision mesh filename=package://jaco_description/meshes/large_ring_cover.dae; visual mesh filename=package://jaco_description/meshes/large_ring_cover.dae
- added link small_ring_cover_1; collision mesh filename=package://jaco_description/meshes/small_ring_cover.dae; visual mesh filename=package://jaco_description/meshes/small_ring_cover.dae
- added link small_ring_cover_2; collision mesh filename=package://jaco_description/meshes/small_ring_cover.dae; visual mesh filename=package://jaco_description/meshes/small_ring_cover.dae
- added link small_ring_cover_3; collision mesh filename=package://jaco_description/meshes/small_ring_cover.dae; visual mesh filename=package://jaco_description/meshes/small_ring_cover.dae
Joints:
- added joint jaco_joint_finger_tip_1: type revolute, parent jaco_link_finger_1, child jaco_link_finger_tip_1, origin xyz=0.044094 -0.0029 0 rpy=0 0 0, axis 0 0 1, limit lower=0 upper=0.698131700798 effort=30 velocity=5
- added joint jaco_joint_finger_tip_2: type revolute, parent jaco_link_finger_2, child jaco_link_finger_tip_2, origin xyz=0.044094 -0.0029 0 rpy=0 0 0, axis 0 0 1, limit lower=0 upper=0.698131700798 effort=30 velocity=5
- added joint jaco_joint_finger_tip_3: type revolute, parent jaco_link_finger_3, child jaco_link_finger_tip_3, origin xyz=0.044094 -0.0029 0 rpy=0 0 0, axis 0 0 1, limit lower=0 upper=0.698131700798 effort=30 velocity=5
- added joint large_ring_cover_1_joint: type fixed, parent jaco_link_base, child large_ring_cover_1, origin xyz=0 0 0.1535 rpy=3.14159265359 0 0, axis 0 0 1, limit lower=-6.28318530718 upper=6.28318530718 effort=30 velocity=5
- added joint large_ring_cover_2_joint: type fixed, parent jaco_link_1, child large_ring_cover_2, origin xyz=0 0 -0.1185 rpy=-1.57079632679 -1.57079632679 0, axis 0 0 1, limit lower=0 upper=6.28318530718 effort=30 velocity=5
- added joint large_ring_cover_3_joint: type fixed, parent jaco_link_2, child large_ring_cover_3, origin xyz=0.41 0 0 rpy=3.14159265359 0 3.14159265359, axis 0 0 1, limit lower=0 upper=6.28318530718 effort=30 velocity=5
- added joint large_ring_cover_4_joint: type fixed, parent jaco_link_3, child small_ring_cover_1, origin xyz=0.207 0 -0.01125 rpy=0 -1.57079632679 0, axis 0 0 1, limit lower=-6.28318530718 upper=6.28318530718 effort=30 velocity=5
- added joint large_ring_cover_5_joint: type fixed, parent jaco_link_4, child small_ring_cover_2, origin xyz=0.0343 0 -0.06588 rpy=0 0.959931088597 3.14159265359, axis 0 0 1, limit lower=-6.28318530718 upper=6.28318530718 effort=30 velocity=5
- added joint large_ring_cover_6_joint: type fixed, parent jaco_link_5, child small_ring_cover_3, origin xyz=0.0343 0 -0.06588 rpy=0 0.959931088597 3.14159265359, axis 0 0 1, limit lower=-6.28318530718 upper=6.28318530718 effort=30 velocity=5
- joint jaco_joint_finger_1: origin xyz=-0.03978 0 -0.10071 rpy=-1.7983 1.117 3.1416 -> xyz=-0.032578 0.0033 -0.12131 rpy=-1.7983 1.117 3.1416
- joint jaco_joint_finger_2: origin xyz=0.03569 0.0216 -0.10071 rpy=-1.5161 1.1459 0.23978 -> xyz=0.027788 0.0206 -0.12131 rpy=-1.5161 1.1459 0.23978
- joint jaco_joint_finger_3: origin xyz=0.03569 -0.0216 -0.10071 rpy=-1.6222 1.117 -0.23615 -> xyz=0.027788 -0.0206 -0.12131 rpy=-1.6222 1.117 -0.23615

Commit message: updated CARL urdf

File: carl_description/robots/carl.urdf (robot description, URDF)
Before this commit: robot carl, 44 links, 43 joints
Links:
- removed link large_ring_cover_1
- removed link large_ring_cover_2
- removed link large_ring_cover_3
- removed link small_ring_cover_1
- removed link small_ring_cover_2
- removed link small_ring_cover_3
- added link jaco_large_ring_cover_1; collision mesh filename=package://jaco_description/meshes/jaco_large_ring_cover.min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; visual mesh filename=package://jaco_description/meshes/jaco_large_ring_cover.min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
- added link jaco_large_ring_cover_2; collision mesh filename=package://jaco_description/meshes/jaco_large_ring_cover.min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; visual mesh filename=package://jaco_description/meshes/jaco_large_ring_cover.min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
- added link jaco_large_ring_cover_3; collision mesh filename=package://jaco_description/meshes/jaco_large_ring_cover.min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; visual mesh filename=package://jaco_description/meshes/jaco_large_ring_cover.min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
- added link jaco_small_ring_cover_1; collision mesh filename=package://jaco_description/meshes/jaco_small_ring_cover.min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; visual mesh filename=package://jaco_description/meshes/jaco_small_ring_cover.min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
- added link jaco_small_ring_cover_2; collision mesh filename=package://jaco_description/meshes/jaco_small_ring_cover.min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; visual mesh filename=package://jaco_description/meshes/jaco_small_ring_cover.min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
- added link jaco_small_ring_cover_3; collision mesh filename=package://jaco_description/meshes/jaco_small_ring_cover.min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; visual mesh filename=package://jaco_description/meshes/jaco_small_ring_cover.min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
- link jaco_link_1: geometry collision mesh filename=package://jaco_description/meshes/jaco_link_1.min.dae; visual mesh filename=package://jaco_description/meshes/jaco_link_1.min.dae
- link jaco_link_2: geometry collision mesh filename=package://jaco_description/meshes/jaco_link_2.min.dae; visual mesh filename=package://jaco_description/meshes/jaco_link_2.min.dae
- link jaco_link_3: geometry collision mesh filename=package://jaco_description/meshes/jaco_link_3.min.dae; visual mesh filename=package://jaco_description/meshes/jaco_link_3.min.dae
- link jaco_link_4: geometry collision mesh filename=package://jaco_description/meshes/jaco_link_4_5.min.dae; visual mesh filename=package://jaco_description/meshes/jaco_link_4_5.min.dae
- link jaco_link_5: geometry collision mesh filename=package://jaco_description/meshes/jaco_link_4_5.min.dae; visual mesh filename=package://jaco_description/meshes/jaco_link_4_5.min.dae
- link jaco_link_base: geometry collision mesh filename=package://jaco_description/meshes/jaco_link_base.min.dae; visual mesh filename=package://jaco_description/meshes/jaco_link_base.min.dae
- link jaco_link_finger_1: geometry collision mesh filename=package://jaco_description/meshes/jaco_link_finger.min.dae; visual mesh filename=package://jaco_description/meshes/jaco_link_finger.min.dae
- link jaco_link_finger_2: geometry collision mesh filename=package://jaco_description/meshes/jaco_link_finger.min.dae; visual mesh filename=package://jaco_description/meshes/jaco_link_finger.min.dae
- link jaco_link_finger_3: geometry collision mesh filename=package://jaco_description/meshes/jaco_link_finger.min.dae; visual mesh filename=package://jaco_description/meshes/jaco_link_finger.min.dae
- link jaco_link_finger_tip_1: geometry collision mesh filename=package://jaco_description/meshes/jaco_link_finger_tip.min.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; visual mesh filename=package://jaco_description/meshes/jaco_link_finger_tip.min.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
- link jaco_link_finger_tip_2: geometry collision mesh filename=package://jaco_description/meshes/jaco_link_finger_tip.min.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; visual mesh filename=package://jaco_description/meshes/jaco_link_finger_tip.min.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
- link jaco_link_finger_tip_3: geometry collision mesh filename=package://jaco_description/meshes/jaco_link_finger_tip.min.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; visual mesh filename=package://jaco_description/meshes/jaco_link_finger_tip.min.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
- link jaco_link_hand: geometry collision mesh filename=package://jaco_description/meshes/jaco_link_hand.min.dae; visual mesh filename=package://jaco_description/meshes/jaco_link_hand.min.dae
Joints:
- removed joint large_ring_cover_1_joint
- removed joint large_ring_cover_2_joint
- removed joint large_ring_cover_3_joint
- removed joint large_ring_cover_4_joint
- removed joint large_ring_cover_5_joint
- removed joint large_ring_cover_6_joint
- added joint jaco_large_ring_cover_1_joint: type fixed, parent jaco_link_base, child jaco_large_ring_cover_1, origin xyz=0 0 0.1535 rpy=3.14159265359 0 0, axis 0 0 1, limit lower=-6.28318530718 upper=6.28318530718 effort=30 velocity=5
- added joint jaco_large_ring_cover_2_joint: type fixed, parent jaco_link_1, child jaco_large_ring_cover_2, origin xyz=0 0 -0.1185 rpy=-1.57079632679 -1.57079632679 0, axis 0 0 1, limit lower=0 upper=6.28318530718 effort=30 velocity=5
- added joint jaco_large_ring_cover_3_joint: type fixed, parent jaco_link_2, child jaco_large_ring_cover_3, origin xyz=0.41 0 0 rpy=3.14159265359 0 3.14159265359, axis 0 0 1, limit lower=0 upper=6.28318530718 effort=30 velocity=5
- added joint jaco_large_ring_cover_4_joint: type fixed, parent jaco_link_3, child jaco_small_ring_cover_1, origin xyz=0.207 0 -0.01125 rpy=0 -1.57079632679 0, axis 0 0 1, limit lower=-6.28318530718 upper=6.28318530718 effort=30 velocity=5
- added joint jaco_large_ring_cover_5_joint: type fixed, parent jaco_link_4, child jaco_small_ring_cover_2, origin xyz=0.0343 0 -0.06588 rpy=0 0.959931088597 3.14159265359, axis 0 0 1, limit lower=-6.28318530718 upper=6.28318530718 effort=30 velocity=5
- added joint jaco_large_ring_cover_6_joint: type fixed, parent jaco_link_4, child jaco_small_ring_cover_3, origin xyz=0.0343 0 -0.06588 rpy=0 0.959931088597 3.14159265359, axis 0 0 1, limit lower=-6.28318530718 upper=6.28318530718 effort=30 velocity=5

Commit message: updated URDF

File: carl_description/robots/carl.urdf (robot description, URDF)
Before this commit: robot carl, 44 links, 43 joints
Links:
- removed link left_rear_strut_inside_link
- removed link right_rear_strut_inside_link
Joints:
- removed joint left_rear_strut_link_left_rear_strut_link_inside_joint
- removed joint right_rear_strut_link_right_rear_strut_link_inside_joint

Commit message: recompiled URDF

File: carl_description/robots/carl.urdf (robot description, URDF)
Before this commit: robot carl, 42 links, 41 joints
Links:
- removed link camera_lift_link
- removed link camera_mount_link
- removed link servo_arm_link
- removed link servo_link
- removed link servo_mount_link
- added link asus_lift_link; collision box size=0.027 0.454 0.054; visual mesh filename=package://carl_description/meshes/camera_lift.min.dae
- added link asus_mount_link; visual mesh filename=package://carl_description/meshes/camera_mount.min.dae
- added link asus_servo_arm_link; collision box size=0.035 0.05 0.06; visual mesh filename=package://carl_description/meshes/servo_arm.min.dae
- added link asus_servo_link; collision box size=0.06 0.05 0.035; visual mesh filename=package://carl_description/meshes/servo.min.dae
- added link asus_servo_mount_link; collision box size=0.08 0.055 0.09; visual mesh filename=package://carl_description/meshes/servo_mount.min.dae
- added link creative_camera_link; collision box size=0.04 .14 0.04; visual mesh filename=package://carl_description/meshes/creative_camera.min.dae
- added link creative_mount_link; visual mesh filename=package://carl_description/meshes/creative_mount.min.dae
- added link creative_plate_link; visual mesh filename=package://carl_description/meshes/creative_plate.min.dae
- added link creative_servo_arm_link; collision box size=0.035 0.09 0.06; visual mesh filename=package://carl_description/meshes/servo_arm.min.dae
- added link creative_servo_link; collision box size=0.06 0.05 0.035; visual mesh filename=package://carl_description/meshes/servo.min.dae
Joints:
- removed joint camera_lift_servo_mount_joint
- removed joint left_rear_strut_camera_lift_joint
- removed joint servo_arm_camera_mount_joint
- removed joint servo_mount_servo_joint
- removed joint servo_servo_arm_joint
- added joint asus_lift_asus_servo_mount_joint: type fixed, parent asus_lift_link, child asus_servo_mount_link, origin xyz=0 0 0 rpy=1.5708 0 0, axis 0 0 1
- added joint asus_servo_arm_asus_mount_joint: type fixed, parent asus_servo_arm_link, child asus_mount_link, origin xyz=0 -0.053 -0.016 rpy=1.5708 0 1.5708
- added joint asus_servo_asus_servo_arm_joint: type continuous, parent asus_servo_link, child asus_servo_arm_link, origin xyz=0 -0.042 0 rpy=1.5708 1.5708 0, axis 0 0 1
- added joint asus_servo_mount_asus_servo_joint: type fixed, parent asus_servo_mount_link, child asus_servo_link, origin xyz=0.073 0.013 0.0187 rpy=1.5708 0 3.92699
- added joint creative_plate_link_creative_camera_joint: type fixed, parent creative_plate_link, child creative_camera_link, origin xyz=0 0.0 0.012 rpy=0 0 0
- added joint creative_servo_arm_creative_plate_joint: type fixed, parent creative_servo_arm_link, child creative_plate_link, origin xyz=0 -0.057 -0.024 rpy=1.5708 1.5708 0
- added joint creative_servo_creative_servo_arm_joint: type continuous, parent creative_servo_link, child creative_servo_arm_link, origin xyz=0 -0.042 0 rpy=1.5708 1.5708 0, axis 0 0 1
- added joint creative_servo_mount_creative_servo_joint: type fixed, parent creative_mount_link, child creative_servo_link, origin xyz=-0.023 0 -0.01 rpy=1.5708 -0.349065 0
- added joint right_rear_strut_asus_lift_joint: type fixed, parent right_rear_strut_link, child asus_lift_link, origin xyz=-0.013 -0.20 1.538 rpy=0 0 3.1415926536
- added joint top_plate_creative_mount_joint: type fixed, parent top_plate_link, child creative_mount_link, origin xyz=0.07 0 -0.03 rpy=0 0 3.1415926536
- joint base_link_right_rear_strut_joint: origin xyz=-0.222 -0.200 -0.102 rpy=0 0 0 -> xyz=-0.222 -0.200 -0.102 rpy=0 0 3.1415926536
- joint camera_joint: parent camera_mount_link -> asus_mount_link
- joint left_rear_strut_top_plate_joint: origin xyz=0.516 0.20 0.598 rpy=0 0 0 -> xyz=-0.516 -0.20 0.598 rpy=0 0 3.14159265
- joint right_rear_strut_link_right_side_cover_joint: origin xyz=0.229 -0.026 0.447 rpy=0 0 0 -> xyz=-0.229 -0.026 0.447 rpy=0 0 0

Commit message: updated asus URDF

File: carl_description/robots/carl.urdf (robot description, URDF)
Before this commit: robot carl, 47 links, 46 joints
Links:
- added link camera_depth_frame, mass 0.01
- added link camera_depth_optical_frame, mass 0.001
- added link camera_rgb_frame, mass 0.001
- added link camera_rgb_optical_frame, mass 0.001
- link camera_link: geometry collision box size=0.0730 .2760 0.0720; visual mesh filename=package://carl_description/meshes/asus_xtion_pro_live.min.d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 scale=0.001 0.001 0.001
Joints:
- added joint camera_depth_joint: type fixed, parent camera_link, child camera_depth_frame, origin xyz=0 0.049 0 rpy=0 0 0
- added joint camera_depth_optical_joint: type fixed, parent camera_depth_frame, child camera_depth_optical_frame, origin xyz=0 0 0 rpy=-1.57079632679 0 -1.57079632679
- added joint camera_rgb_joint: type fixed, parent camera_link, child camera_rgb_frame, origin xyz=0 0.022 0 rpy=0 0 0
- added joint camera_rgb_optical_joint: type fixed, parent camera_rgb_frame, child camera_rgb_optical_frame, origin xyz=0 0 0 rpy=-1.57079632679 0 -1.57079632679

Commit message: rebuild CARL URDF

File: carl_description/robots/carl.urdf (robot description, URDF)
Before this commit: robot carl, 51 links, 50 joints
Joints:
- joint camera_joint: origin xyz=-0.016 -0.008 0.018 rpy=0 -1.5708 0 -> xyz=-0.016 -0.008 0.018 rpy=0 -1.53 0

Commit message: updated URDF

File: carl_description/robots/carl.urdf (robot description, URDF)
Before this commit: robot carl, 51 links, 50 joints
Joints:
- joint camera_joint: origin xyz=-0.016 -0.008 0.018 rpy=0 -1.53 0 -> xyz=-0.016 -0.008 0.018 rpy=0 -1.54 0
