Commit message: rebuild of URDF

File: carl_description/robots/carl.urdf (robot description, URDF)
Before this commit: robot carl, 51 links, 50 joints
Links:
- removed link BackCover_link
- removed link FrontCover_link
- removed link jaco_large_ring_cover_1
- removed link jaco_large_ring_cover_2
- removed link jaco_large_ring_cover_3
- removed link jaco_link_1
- removed link jaco_link_2
- removed link jaco_link_3
- removed link jaco_link_4
- removed link jaco_link_5
- removed link jaco_link_base
- removed link jaco_link_finger_1
- removed link jaco_link_finger_2
- removed link jaco_link_finger_3
- removed link jaco_link_finger_tip_1
- removed link jaco_link_finger_tip_2
- removed link jaco_link_finger_tip_3
- removed link jaco_link_hand
- removed link jaco_small_ring_cover_1
- removed link jaco_small_ring_cover_2
- removed link jaco_small_ring_cover_3
- added link back_cover_link; collision mesh filename=package://carl_description/meshes/back_cover.stl scale=0.0254 0.0254 0.0254; visual mesh filename=package://carl_description/meshes/back_cover.min.dae scale=0.0254 0.0254 0.0254
- added link front_cover_link; collision mesh filename=package://carl_description/meshes/front_cover.stl scale=0.0254 0.0254 0.0254; visual mesh filename=package://carl_description/meshes/front_cover.min.dae scale=0.0254 0.0254 0.0254
- link asus_lift_link: geometry collision mesh filename=package://carl_description/meshes/camera_lift.stl scale=0.0254 0.0254 0.0254; visual mesh filename=package://carl_description/meshes/camera_lift.min.dae scale=0.0254 0.0254 0.0254
- link asus_mount_link: geometry collision mesh filename=package://carl_description/meshes/camera_mount.stl scale=0.0254 0.0254 0.0254; visual mesh filename=package://carl_description/meshes/camera_mount.min.dae scale=0.0254 0.0254 0.0254
- link asus_servo_arm_link: geometry collision mesh filename=package://carl_description/meshes/servo_arm.stl scale=0.0254 0.0254 0.0254; visual mesh filename=package://carl_description/meshes/servo_arm.min.dae scale=0.0254 0.0254 0.0254
- link asus_servo_link: geometry collision mesh filename=package://carl_description/meshes/servo.stl scale=0.0254 0.0254 0.0254; visual mesh filename=package://carl_description/meshes/servo.min.dae scale=0.0254 0.0254 0.0254
- link asus_servo_mount_link: geometry collision mesh filename=package://carl_description/meshes/servo_mount.stl scale=0.0254 0.0254 0.0254; visual mesh filename=package://carl_description/meshes/servo_mount.min.dae scale=0.0254 0.0254 0.0254
- link base_link: geometry collision mesh filename=package://carl_description/meshes/base.stl scale=0.0254 0.0254 0.0254; visual mesh filename=package://carl_description/meshes/base.min.dae scale=0.0254 0.0254 0.0254
- link camera_link: geometry collision mesh filename=package://carl_description/meshes/asus_xtion_pro_live.stl scale=2.54e-05 2.54e-05 2.54e-05; visual mesh filename=package://carl_description/meshes/asus_xtion_pro_live.min.d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 scale=2.54e-05 2.54e-05 2.54e-05
- link caster_link: geometry collision mesh filename=package://carl_description/meshes/caster.stl scale=0.0254 0.0254 0.0254; visual mesh filename=package://carl_description/meshes/caster.min.dae scale=0.0254 0.0254 0.0254
- link caster_plate_link: geometry collision mesh filename=package://carl_description/meshes/caster_plate.stl scale=0.0254 0.0254 0.0254; visual mesh filename=package://carl_description/meshes/caster_plate.min.dae scale=0.0254 0.0254 0.0254
- link creative_camera_link: geometry collision mesh filename=package://carl_description/meshes/creative_camera.stl scale=0.0254 0.0254 0.0254; visual mesh filename=package://carl_description/meshes/creative_camera.min.dae scale=0.0254 0.0254 0.0254
- link creative_mount_link: geometry collision mesh filename=package://carl_description/meshes/creative_mount.stl scale=0.0254 0.0254 0.0254; visual mesh filename=package://carl_description/meshes/creative_mount.min.dae scale=0.0254 0.0254 0.0254
- link creative_plate_link: geometry collision mesh filename=package://carl_description/meshes/creative_plate.stl scale=0.0254 0.0254 0.0254; visual mesh filename=package://carl_description/meshes/creative_plate.min.dae scale=0.0254 0.0254 0.0254
- link creative_servo_arm_link: geometry collision mesh filename=package://carl_description/meshes/servo_arm.stl scale=0.0254 0.0254 0.0254; visual mesh filename=package://carl_description/meshes/servo_arm.min.dae scale=0.0254 0.0254 0.0254
- link creative_servo_link: geometry collision mesh filename=package://carl_description/meshes/servo.stl scale=0.0254 0.0254 0.0254; visual mesh filename=package://carl_description/meshes/servo.min.dae scale=0.0254 0.0254 0.0254
- link hokuyo_link: geometry collision mesh filename=package://carl_description/meshes/hokuyo.stl; visual mesh filename=package://carl_description/meshes/hokuyo.min.dae
- link jaco_mount_link: geometry collision mesh filename=package://carl_description/meshes/jaco_mount.stl scale=0.0254 0.0254 0.0254; visual mesh filename=package://carl_description/meshes/jaco_mount.min.dae scale=0.0254 0.0254 0.0254
- link left_rear_strut_link: geometry collision mesh filename=package://carl_description/meshes/rear_strut.stl scale=0.0254 0.0254 0.0254; visual mesh filename=package://carl_description/meshes/rear_strut.min.dae scale=0.0254 0.0254 0.0254
- link left_rear_strut_top_link: geometry collision mesh filename=package://carl_description/meshes/rear_strut_top.stl scale=0.0254 0.0254 0.0254; visual mesh filename=package://carl_description/meshes/rear_strut_top.min.dae scale=0.0254 0.0254 0.0254
- link left_side_cover_link: geometry collision mesh filename=package://carl_description/meshes/side_cover.stl scale=0.0254 0.0254 0.0254; visual mesh filename=package://carl_description/meshes/side_cover.min.dae scale=0.0254 0.0254 0.0254
- link left_wheel_link: geometry collision mesh filename=package://carl_description/meshes/wheel.stl scale=0.0254 0.0254 0.0254; visual mesh filename=package://carl_description/meshes/wheel.min.dae scale=0.0254 0.0254 0.0254
- link right_rear_strut_link: geometry collision mesh filename=package://carl_description/meshes/rear_strut.stl scale=0.0254 0.0254 0.0254; visual mesh filename=package://carl_description/meshes/rear_strut.min.dae scale=0.0254 0.0254 0.0254
- link right_rear_strut_top_link: geometry collision mesh filename=package://carl_description/meshes/rear_strut_top.stl scale=0.0254 0.0254 0.0254; visual mesh filename=package://carl_description/meshes/rear_strut_top.min.dae scale=0.0254 0.0254 0.0254
- link right_side_cover_link: geometry collision mesh filename=package://carl_description/meshes/side_cover.stl scale=0.0254 0.0254 0.0254; visual mesh filename=package://carl_description/meshes/side_cover.min.dae scale=0.0254 0.0254 0.0254
- link right_wheel_link: geometry collision mesh filename=package://carl_description/meshes/wheel.stl scale=0.0254 0.0254 0.0254; visual mesh filename=package://carl_description/meshes/wheel.min.dae scale=0.0254 0.0254 0.0254
- link top_plate_link: geometry collision mesh filename=package://carl_description/meshes/top_plate.stl scale=0.0254 0.0254 0.0254; visual mesh filename=package://carl_description/meshes/top_plate.min.dae scale=0.0254 0.0254 0.0254
Joints:
- removed joint asus_lift_asus_servo_mount_joint
- removed joint asus_servo_arm_asus_mount_joint
- removed joint asus_servo_asus_servo_arm_joint
- removed joint asus_servo_mount_asus_servo_joint
- removed joint base_back_cover
- removed joint base_front_cover_joint
- removed joint base_link_caster_plate_joint
- removed joint caster_plate__caster_joint
- removed joint caster_plate_link_hokuyo_joint
- removed joint creative_plate_link_creative_camera_joint
- removed joint creative_servo_arm_creative_plate_joint
- removed joint creative_servo_creative_servo_arm_joint
- removed joint creative_servo_mount_creative_servo_joint
- removed joint jaco_joint_1
- removed joint jaco_joint_2
- removed joint jaco_joint_3
- removed joint jaco_joint_4
- removed joint jaco_joint_5
- removed joint jaco_joint_6
- removed joint jaco_joint_base
- removed joint jaco_joint_finger_1
- removed joint jaco_joint_finger_2
- removed joint jaco_joint_finger_3
- removed joint jaco_joint_finger_tip_1
- removed joint jaco_joint_finger_tip_2
- removed joint jaco_joint_finger_tip_3
- removed joint jaco_large_ring_cover_1_joint
- removed joint jaco_large_ring_cover_2_joint
- removed joint jaco_large_ring_cover_3_joint
- removed joint jaco_large_ring_cover_4_joint
- removed joint jaco_large_ring_cover_5_joint
- removed joint jaco_large_ring_cover_6_joint
- removed joint left_rear_strut_link_left_side_cover_joint
- removed joint left_rear_strut_top_plate_joint
- removed joint right_rear_strut_asus_lift_joint
- removed joint right_rear_strut_link_right_side_cover_joint
- removed joint top_plate_creative_mount_joint
- removed joint top_plate_jaco_mount
- added joint asus_lift_link_asus_servo_mount_link_joint: type fixed, parent asus_lift_link, child asus_servo_mount_link, origin xyz=0 0 0 rpy=1.57079632679 0 0
- added joint asus_servo_arm_link_asus_mount_link_joint: type fixed, parent asus_servo_arm_link, child asus_mount_link, origin xyz=0 -0.053 -0.016 rpy=1.57079632679 0 1.57079632679
- added joint asus_servo_link_asus_servo_arm_link_joint: type continuous, parent asus_servo_link, child asus_servo_arm_link, origin xyz=0 -0.042 0 rpy=1.57079632679 1.57079632679 0, axis 0 0 1
- added joint asus_servo_mount_link_asus_servo_link_joint: type fixed, parent asus_servo_mount_link, child asus_servo_link, origin xyz=0.073 0.013 0.0187 rpy=1.57079632679 0 3.92699082
- added joint base_back_cover_link_joint: type fixed, parent base_link, child back_cover_link, origin xyz=-0.237 0 -0.102 rpy=0 0 0
- added joint base_front_cover_link_joint: type fixed, parent base_link, child front_cover_link, origin xyz=0.247 0 0.242 rpy=0 0 1.57079632679
- added joint base_link_asus_lift_link_joint: type fixed, parent base_link, child asus_lift_link, origin xyz=-0.209 0 1.436 rpy=0 0 0
- added joint base_link_caster_plate_link_joint: type fixed, parent base_link, child caster_plate_link, origin xyz=0.2883 0 0 rpy=0 0 0
- added joint base_link_left_side_cover_link_joint: type fixed, parent base_link, child left_side_cover_link, origin xyz=0.007 0.226 0.345 rpy=0 0 1.57079632679
- added joint base_link_right_side_cover_link_joint: type fixed, parent base_link, child right_side_cover_link, origin xyz=0.007 -0.226 0.345 rpy=0 0 1.57079632679
- added joint base_link_top_plate_link_joint: type fixed, parent base_link, child top_plate_link, origin xyz=0.294 0 0.496 rpy=0 0 0
- added joint caster_plate_link_caster_link_joint: type continuous, parent caster_plate_link, child caster_link, origin xyz=0.0267 0 -0.024 rpy=0 0 0, axis 0 0 1
- added joint caster_plate_link_hokuyo_link_joint: type fixed, parent caster_plate_link, child hokuyo_link, origin xyz=0.07 0 0.035 rpy=0 0 0
- added joint creative_mount_link_creative_servo_link_joint: type fixed, parent creative_mount_link, child creative_servo_link, origin xyz=-0.023 0 -0.01 rpy=1.57079632679 -0.34906585 0
- added joint creative_plate_link_creative_camera_link_joint: type fixed, parent creative_plate_link, child creative_camera_link, origin xyz=0 0.0 0.012 rpy=0 0 0
- added joint creative_servo_arm_link_creative_plate_link_joint: type fixed, parent creative_servo_arm_link, child creative_plate_link, origin xyz=0 -0.057 -0.024 rpy=1.57079632679 1.57079632679 0
- added joint creative_servo_link_creative_servo_arm_link_joint: type continuous, parent creative_servo_link, child creative_servo_arm_link, origin xyz=0 -0.042 0 rpy=1.57079632679 1.57079632679 0, axis 0 0 1
- added joint top_plate_link_creative_mount_link_joint: type fixed, parent top_plate_link, child creative_mount_link, origin xyz=0.07 0 -0.03 rpy=0 0 3.14159265359
- added joint top_plate_link_jaco_mount_link_joint: type fixed, parent top_plate_link, child jaco_mount_link, origin xyz=0 0 -0.130 rpy=0 0 1.57079632679
- joint base_link_left_wheel_joint: origin xyz=0 0.25 0 rpy=-1.5708 0 0 -> xyz=0 0.25 0 rpy=1.57079632679 0 0
- joint base_link_right_rear_strut_joint: origin xyz=-0.222 -0.200 -0.102 rpy=0 0 3.1415926536 -> xyz=-0.222 -0.200 -0.102 rpy=0 0 3.14159265359
- joint base_link_right_wheel_joint: origin xyz=0 -0.25 0 rpy=1.5708 0 0 -> xyz=0 -0.25 0 rpy=-1.57079632679 0 0
- joint camera_joint: origin xyz=-0.016 -0.008 0.018 rpy=0 -1.54 0 -> xyz=-0.016 -0.008 0.018 rpy=0 -1.57079632679 0

Commit message: JACO arm added back

File: carl_description/robots/carl.urdf (robot description, URDF)
Before this commit: robot carl, 32 links, 31 joints
Links:
- added link jaco_large_ring_cover_1; collision mesh filename=package://jaco_description/meshes/jaco_large_ring_cover.stl scale=0.0254 0.0254 0.0254; visual mesh filename=package://jaco_description/meshes/jaco_large_ring_cover.min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 scale=0.0254 0.0254 0.0254
- added link jaco_large_ring_cover_2; collision mesh filename=package://jaco_description/meshes/jaco_large_ring_cover.stl scale=0.0254 0.0254 0.0254; visual mesh filename=package://jaco_description/meshes/jaco_large_ring_cover.min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 scale=0.0254 0.0254 0.0254
- added link jaco_large_ring_cover_3; collision mesh filename=package://jaco_description/meshes/jaco_large_ring_cover.stl scale=0.0254 0.0254 0.0254; visual mesh filename=package://jaco_description/meshes/jaco_large_ring_cover.min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 scale=0.0254 0.0254 0.0254
- added link jaco_link_1; collision mesh filename=package://jaco_description/meshes/jaco_link_1.stl scale=0.0254 0.0254 0.0254; visual mesh filename=package://jaco_description/meshes/jaco_link_1.min.dae scale=0.0254 0.0254 0.0254
- added link jaco_link_2; collision mesh filename=package://jaco_description/meshes/jaco_link_2.stl scale=0.0254 0.0254 0.0254; visual mesh filename=package://jaco_description/meshes/jaco_link_2.min.dae scale=0.0254 0.0254 0.0254
- added link jaco_link_3; collision mesh filename=package://jaco_description/meshes/jaco_link_3.stl scale=0.0254 0.0254 0.0254; visual mesh filename=package://jaco_description/meshes/jaco_link_3.min.dae scale=0.0254 0.0254 0.0254
- added link jaco_link_4; collision mesh filename=package://jaco_description/meshes/jaco_link_4_5.stl scale=0.0254 0.0254 0.0254; visual mesh filename=package://jaco_description/meshes/jaco_link_4_5.min.dae scale=0.0254 0.0254 0.0254
- added link jaco_link_5; collision mesh filename=package://jaco_description/meshes/jaco_link_4_5.stl scale=0.0254 0.0254 0.0254; visual mesh filename=package://jaco_description/meshes/jaco_link_4_5.min.dae scale=0.0254 0.0254 0.0254
- added link jaco_link_base; collision mesh filename=package://jaco_description/meshes/jaco_link_base.stl scale=0.0254 0.0254 0.0254; visual mesh filename=package://jaco_description/meshes/jaco_link_base.min.dae scale=0.0254 0.0254 0.0254
- added link jaco_link_finger_1; collision mesh filename=package://jaco_description/meshes/jaco_link_finger.stl scale=0.0254 0.0254 0.0254; visual mesh filename=package://jaco_description/meshes/jaco_link_finger.min.dae scale=0.0254 0.0254 0.0254
- added link jaco_link_finger_2; collision mesh filename=package://jaco_description/meshes/jaco_link_finger.stl scale=0.0254 0.0254 0.0254; visual mesh filename=package://jaco_description/meshes/jaco_link_finger.min.dae scale=0.0254 0.0254 0.0254
- added link jaco_link_finger_3; collision mesh filename=package://jaco_description/meshes/jaco_link_finger.stl scale=0.0254 0.0254 0.0254; visual mesh filename=package://jaco_description/meshes/jaco_link_finger.min.dae scale=0.0254 0.0254 0.0254
- added link jaco_link_finger_tip_1; collision mesh filename=package://jaco_description/meshes/jaco_link_finger_tip.stl scale=0.0254 0.0254 0.0254; visual mesh filename=package://jaco_description/meshes/jaco_link_finger_tip.min.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 scale=0.0254 0.0254 0.0254
- added link jaco_link_finger_tip_2; collision mesh filename=package://jaco_description/meshes/jaco_link_finger_tip.stl scale=0.0254 0.0254 0.0254; visual mesh filename=package://jaco_description/meshes/jaco_link_finger_tip.min.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 scale=0.0254 0.0254 0.0254
- added link jaco_link_finger_tip_3; collision mesh filename=package://jaco_description/meshes/jaco_link_finger_tip.stl scale=0.0254 0.0254 0.0254; visual mesh filename=package://jaco_description/meshes/jaco_link_finger_tip.min.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 scale=0.0254 0.0254 0.0254
- added link jaco_link_hand; collision mesh filename=package://jaco_description/meshes/jaco_link_hand.stl scale=0.0254 0.0254 0.0254; visual mesh filename=package://jaco_description/meshes/jaco_link_hand.min.dae scale=0.0254 0.0254 0.0254
- added link jaco_small_ring_cover_1; collision mesh filename=package://jaco_description/meshes/jaco_small_ring_cover.stl scale=0.0254 0.0254 0.0254; visual mesh filename=package://jaco_description/meshes/jaco_small_ring_cover.min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 scale=0.0254 0.0254 0.0254
- added link jaco_small_ring_cover_2; collision mesh filename=package://jaco_description/meshes/jaco_small_ring_cover.stl scale=0.0254 0.0254 0.0254; visual mesh filename=package://jaco_description/meshes/jaco_small_ring_cover.min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 scale=0.0254 0.0254 0.0254
- added link jaco_small_ring_cover_3; collision mesh filename=package://jaco_description/meshes/jaco_small_ring_cover.stl scale=0.0254 0.0254 0.0254; visual mesh filename=package://jaco_description/meshes/jaco_small_ring_cover.min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 scale=0.0254 0.0254 0.0254
Joints:
- added joint jaco_joint_1: type revolute, parent jaco_link_base, child jaco_link_1, origin xyz=0 0 0.1535 rpy=3.14159265359 0 0, axis 0 0 1, limit lower=-6.28318530718 upper=6.28318530718 effort=30 velocity=5
- added joint jaco_joint_2: type revolute, parent jaco_link_1, child jaco_link_2, origin xyz=0 0 -0.1185 rpy=-1.57079632679 -1.57079632679 0, axis 0 0 1, limit lower=0 upper=6.28318530718 effort=30 velocity=5
- added joint jaco_joint_3: type revolute, parent jaco_link_2, child jaco_link_3, origin xyz=0.41 0 0 rpy=0 0 3.14159265359, axis 0 0 1, limit lower=0 upper=6.28318530718 effort=30 velocity=5
- added joint jaco_joint_4: type revolute, parent jaco_link_3, child jaco_link_4, origin xyz=0.207 0 -0.01125 rpy=0 -1.57079632679 0, axis 0 0 1, limit lower=-6.28318530718 upper=6.28318530718 effort=30 velocity=5
- added joint jaco_joint_5: type revolute, parent jaco_link_4, child jaco_link_5, origin xyz=0.0343 0 -0.06588 rpy=0 0.959931088597 3.14159265359, axis 0 0 1, limit lower=-6.28318530718 upper=6.28318530718 effort=30 velocity=5
- added joint jaco_joint_6: type revolute, parent jaco_link_5, child jaco_link_hand, origin xyz=0.0343 0 -0.06588 rpy=0 0.959931088597 3.14159265359, axis 0 0 1, limit lower=-6.28318530718 upper=6.28318530718 effort=30 velocity=5
- added joint jaco_joint_base: type fixed, parent jaco_mount_link, child jaco_link_base, origin xyz=0 0 0 rpy=0 0 0, axis 0 0 0, limit lower=-6.28318530718 upper=6.28318530718 effort=30 velocity=5
- added joint jaco_joint_finger_1: type revolute, parent jaco_link_hand, child jaco_link_finger_1, origin xyz=-0.032578 0.0033 -0.12131 rpy=-1.7983 1.117 3.1416, axis 0 0 1, limit lower=0 upper=0.698131700798 effort=30 velocity=5
- added joint jaco_joint_finger_2: type revolute, parent jaco_link_hand, child jaco_link_finger_2, origin xyz=0.027788 0.0206 -0.12131 rpy=-1.5161 1.1459 0.23978, axis 0 0 1, limit lower=0 upper=0.698131700798 effort=30 velocity=5
- added joint jaco_joint_finger_3: type revolute, parent jaco_link_hand, child jaco_link_finger_3, origin xyz=0.027788 -0.0206 -0.12131 rpy=-1.6222 1.117 -0.23615, axis 0 0 1, limit lower=0 upper=0.698131700798 effort=30 velocity=5
- added joint jaco_joint_finger_tip_1: type revolute, parent jaco_link_finger_1, child jaco_link_finger_tip_1, origin xyz=0.044094 -0.0029 0 rpy=0 0 0, axis 0 0 1, limit lower=0 upper=0.698131700798 effort=30 velocity=5
- added joint jaco_joint_finger_tip_2: type revolute, parent jaco_link_finger_2, child jaco_link_finger_tip_2, origin xyz=0.044094 -0.0029 0 rpy=0 0 0, axis 0 0 1, limit lower=0 upper=0.698131700798 effort=30 velocity=5
- added joint jaco_joint_finger_tip_3: type revolute, parent jaco_link_finger_3, child jaco_link_finger_tip_3, origin xyz=0.044094 -0.0029 0 rpy=0 0 0, axis 0 0 1, limit lower=0 upper=0.698131700798 effort=30 velocity=5
- added joint jaco_large_ring_cover_1_joint: type fixed, parent jaco_link_base, child jaco_large_ring_cover_1, origin xyz=0 0 0.1535 rpy=3.14159265359 0 0, axis 0 0 1, limit lower=-6.28318530718 upper=6.28318530718 effort=30 velocity=5
- added joint jaco_large_ring_cover_2_joint: type fixed, parent jaco_link_1, child jaco_large_ring_cover_2, origin xyz=0 0 -0.1185 rpy=-1.57079632679 -1.57079632679 0, axis 0 0 1, limit lower=0 upper=6.28318530718 effort=30 velocity=5
- added joint jaco_large_ring_cover_3_joint: type fixed, parent jaco_link_2, child jaco_large_ring_cover_3, origin xyz=0.41 0 0 rpy=0 0 3.14159265359, axis 0 0 1, limit lower=0 upper=6.28318530718 effort=30 velocity=5
- added joint jaco_large_ring_cover_4_joint: type fixed, parent jaco_link_3, child jaco_small_ring_cover_1, origin xyz=0.207 0 -0.01125 rpy=0 -1.57079632679 0, axis 0 0 1, limit lower=-6.28318530718 upper=6.28318530718 effort=30 velocity=5
- added joint jaco_large_ring_cover_5_joint: type fixed, parent jaco_link_4, child jaco_small_ring_cover_2, origin xyz=0.0343 0 -0.06588 rpy=0 0.959931088597 3.14159265359, axis 0 0 1, limit lower=-6.28318530718 upper=6.28318530718 effort=30 velocity=5
- added joint jaco_large_ring_cover_6_joint: type fixed, parent jaco_link_4, child jaco_small_ring_cover_3, origin xyz=0.0343 0 -0.06588 rpy=0 0.959931088597 3.14159265359, axis 0 0 1, limit lower=-6.28318530718 upper=6.28318530718 effort=30 velocity=5

File: carl_description/robots/carl.urdf.xacro (robot description, xacro)
@@ -2,4 +2,6 @@
 <robot xmlns:xacro="http://www.ros.org/wiki/xacro" name="carl">
   <xacro:include filename="$(find carl_description)/urdf/carl_base/carl_base.urdf.xacro" />
+  <xacro:include filename="$(find jaco_description)/urdf/jaco_arm.urdf.xacro" />
   <xacro:carl_base name="base" />
+  <xacro:jaco_arm  parent="jaco_mount_link" />
 </robot>
