Commit message: fixed rotation of arm

File: carl_description/robots/carl.urdf (robot description, URDF)
Before this commit: robot carl, 51 links, 50 joints
Joints:
- joint jaco_joint_1: origin xyz=0 0 0.1535 rpy=3.14159265359 0 0 -> xyz=0 0 0.1535 rpy=3.14159265359 0 1.412
- joint jaco_joint_2: origin xyz=0 0 -0.1185 rpy=-1.57079632679 -1.57079632679 0 -> xyz=0 0 -0.1185 rpy=-1.57079632679 1.403 0
- joint jaco_joint_3: origin xyz=0.41 0 0 rpy=0 0 3.14159265359 -> xyz=0.41 0 0 rpy=-3.14159265359 0 2.274
- joint jaco_joint_4: origin xyz=0.207 0 -0.01125 rpy=0 -1.57079632679 0 -> xyz=0.207 0 -0.01125 rpy=1.57079632679 0.752 -1.57079632679
- joint jaco_joint_5: origin xyz=0.0343 0 -0.06588 rpy=0 0.959931088597 3.14159265359 -> xyz=0.0343 0 -0.06588 rpy=0.959 -0.045 -1.539
- joint jaco_joint_6: origin xyz=0.0343 0 -0.06588 rpy=0 0.959931088597 3.14159265359 -> xyz=0.0343 0 -0.06588 rpy=0.953 0.139 -1.669
- joint jaco_joint_base: origin xyz=0 0 0 rpy=0 0 0 -> xyz=0 0 0 rpy=0 0 -1.57079632679
- joint jaco_large_ring_cover_1_joint: origin xyz=0 0 0.1535 rpy=3.14159265359 0 0 -> xyz=0 0 0.1535 rpy=3.14159265359 0 1.412
- joint jaco_large_ring_cover_2_joint: origin xyz=0 0 -0.1185 rpy=-1.57079632679 -1.57079632679 0 -> xyz=0 0 -0.1185 rpy=-1.57079632679 1.403 0
- joint jaco_large_ring_cover_3_joint: origin xyz=0.41 0 0 rpy=0 0 3.14159265359 -> xyz=0.41 0 0 rpy=-3.14159265359 0 2.274
- joint jaco_large_ring_cover_4_joint: origin xyz=0.207 0 -0.01125 rpy=0 -1.57079632679 0 -> xyz=0.207 0 -0.01125 rpy=1.57079632679 0.752 -1.57079632679
- joint jaco_large_ring_cover_5_joint: origin xyz=0.0343 0 -0.06588 rpy=0 0.959931088597 3.14159265359 -> xyz=0.0343 0 -0.06588 rpy=0.959 -0.045 -1.539
- joint jaco_large_ring_cover_6_joint: origin xyz=0.0343 0 -0.06588 rpy=0 0.959931088597 3.14159265359 -> xyz=0.0343 0 -0.06588 rpy=0.953 0.139 -1.669; parent jaco_link_4 -> jaco_link_5

File: carl_description/robots/carl.urdf.xacro (robot description, xacro)
@@ -3,5 +3,6 @@
   <xacro:include filename="$(find carl_description)/urdf/carl_base/carl_base.urdf.xacro" />
   <xacro:include filename="$(find jaco_description)/urdf/jaco_arm.urdf.xacro" />
+  <xacro:property name="M_PI" value="3.1415926535897931" />
   <xacro:carl_base name="base" />
-  <xacro:jaco_arm  parent="jaco_mount_link" />
+  <xacro:jaco_arm  parent="jaco_mount_link" xyz="0 0 0" rpy="0 0 -${M_PI/2}" />
 </robot>

Commit message: start position of arm fixed

File: carl_description/robots/carl.urdf (robot description, URDF)
Before this commit: robot carl, 51 links, 50 joints
Joints:
- joint jaco_joint_1: origin xyz=0 0 0.1535 rpy=3.14159265359 0 1.412 -> xyz=0 0 0.1535 rpy=3.14159265359 0 0
- joint jaco_joint_2: origin xyz=0 0 -0.1185 rpy=-1.57079632679 1.403 0 -> xyz=0 0 -0.1185 rpy=-1.57079632679 -1.57079632679 0
- joint jaco_joint_3: origin xyz=0.41 0 0 rpy=-3.14159265359 0 2.274 -> xyz=0.41 0 0 rpy=3.14159265359 0 3.14159265359
- joint jaco_joint_4: origin xyz=0.207 0 -0.01125 rpy=1.57079632679 0.752 -1.57079632679 -> xyz=0.207 0 -0.01125 rpy=0 -1.57079632679 0
- joint jaco_joint_5: origin xyz=0.0343 0 -0.06588 rpy=0.959 -0.045 -1.539 -> xyz=0.0343 0 -0.06588 rpy=0 0.959931088597 3.14159265359
- joint jaco_joint_6: origin xyz=0.0343 0 -0.06588 rpy=0.953 0.139 -1.669 -> xyz=0.0343 0 -0.06588 rpy=0 0.959931088597 3.14159265359
- joint jaco_large_ring_cover_1_joint: origin xyz=0 0 0.1535 rpy=3.14159265359 0 1.412 -> xyz=0 0 0.1535 rpy=3.14159265359 0 0
- joint jaco_large_ring_cover_2_joint: origin xyz=0 0 -0.1185 rpy=-1.57079632679 1.403 0 -> xyz=0 0 -0.1185 rpy=-1.57079632679 -1.57079632679 0
- joint jaco_large_ring_cover_3_joint: origin xyz=0.41 0 0 rpy=-3.14159265359 0 2.274 -> xyz=0.41 0 0 rpy=3.14159265359 0 3.14159265359
- joint jaco_large_ring_cover_4_joint: origin xyz=0.207 0 -0.01125 rpy=1.57079632679 0.752 -1.57079632679 -> xyz=0.207 0 -0.01125 rpy=0 -1.57079632679 0
- joint jaco_large_ring_cover_5_joint: origin xyz=0.0343 0 -0.06588 rpy=0.959 -0.045 -1.539 -> xyz=0.0343 0 -0.06588 rpy=0 0.959931088597 3.14159265359
- joint jaco_large_ring_cover_6_joint: origin xyz=0.0343 0 -0.06588 rpy=0.953 0.139 -1.669 -> xyz=0.0343 0 -0.06588 rpy=0 0.959931088597 3.14159265359

Commit message: ran xacro

File: carl_description/robots/carl.urdf (robot description, URDF)
Before this commit: robot carl, 51 links, 50 joints
Links:
- link asus_lift_link: geometry collision box size=0.027 0.454 0.054; visual mesh filename=package://carl_description/meshes/camera_lift.min.dae scale=0.0254 0.0254 0.0254
- link asus_mount_link: geometry collision box size=0.041 0.2365 0.0032; visual mesh filename=package://carl_description/meshes/camera_mount.min.dae scale=0.0254 0.0254 0.0254
- link asus_servo_arm_link: geometry collision box size=0.029 0.067 0.049; visual mesh filename=package://carl_description/meshes/servo_arm.min.dae scale=0.0254 0.0254 0.0254
- link asus_servo_link: geometry collision box size=0.05 0.0382 0.032; visual mesh filename=package://carl_description/meshes/servo.min.dae scale=0.0254 0.0254 0.0254
- link asus_servo_mount_link: geometry collision box size=0.057 0.0508 0.089; visual mesh filename=package://carl_description/meshes/servo_mount.min.dae scale=0.0254 0.0254 0.0254
- link base_link: geometry collision box size=0.4 0.363 0.12; visual mesh filename=package://carl_description/meshes/base.min.dae scale=0.0254 0.0254 0.0254
- link camera_link: geometry collision box size=0.1799 0.0246 0.0362; visual mesh filename=package://carl_description/meshes/asus_xtion_pro_live.min.d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 scale=2.54e-05 2.54e-05 2.54e-05
- link caster_link: geometry collision box size=0.17 0.0636 0.1858; visual mesh filename=package://carl_description/meshes/caster.min.dae scale=0.0254 0.0254 0.0254
- link caster_plate_link: geometry collision box size=0.16 0.16 0.0949; collision box size=0.3 0.16 0.0949
- link creative_camera_link: geometry collision box size=0.1070 0.02575 0.026; visual mesh filename=package://carl_description/meshes/creative_camera.min.dae scale=0.0254 0.0254 0.0254
- link creative_mount_link: geometry collision box size=0.0298 0.051 0.051; visual mesh filename=package://carl_description/meshes/creative_mount.min.dae scale=0.0254 0.0254 0.0254
- link creative_plate_link: geometry collision box size=0.13975 0.03815 0.00318; visual mesh filename=package://carl_description/meshes/creative_plate.min.dae scale=0.0254 0.0254 0.0254
- link creative_servo_arm_link: geometry collision box size=0.029 0.067 0.049; visual mesh filename=package://carl_description/meshes/servo_arm.min.dae scale=0.0254 0.0254 0.0254
- link creative_servo_link: geometry collision box size=0.05 0.0382 0.032; visual mesh filename=package://carl_description/meshes/servo.min.dae scale=0.0254 0.0254 0.0254
- link front_cover_link: geometry collision box size=0.25 0.068 0.508; collision box size=0.25 0.068 0.508
- link hokuyo_link: geometry collision box size=0.05 0.05 0.08; visual mesh filename=package://carl_description/meshes/hokuyo.min.dae
- link jaco_mount_link: geometry collision box size=0.2286 0.0508 0.0254; visual mesh filename=package://carl_description/meshes/jaco_mount.min.dae scale=0.0254 0.0254 0.0254
- link left_rear_strut_link: geometry collision box size=0.0255 0.052 1.1; visual mesh filename=package://carl_description/meshes/rear_strut.min.dae scale=0.0254 0.0254 0.0254
- link left_rear_strut_top_link: geometry collision box size=0.0255 0.051 0.4572; visual mesh filename=package://carl_description/meshes/rear_strut_top.min.dae scale=0.0254 0.0254 0.0254
- link left_side_cover_link: geometry collision box size=0.0015 0.483 0.289; visual mesh filename=package://carl_description/meshes/side_cover.min.dae scale=0.0254 0.0254 0.0254
- link left_wheel_link: geometry collision cylinder length=0.12 radius=0.25; visual mesh filename=package://carl_description/meshes/wheel.min.dae scale=0.0254 0.0254 0.0254
- link right_rear_strut_link: geometry collision box size=0.0255 0.052 1.1; visual mesh filename=package://carl_description/meshes/rear_strut.min.dae scale=0.0254 0.0254 0.0254
- link right_rear_strut_top_link: geometry collision box size=0.0255 0.051 0.4572; visual mesh filename=package://carl_description/meshes/rear_strut_top.min.dae scale=0.0254 0.0254 0.0254
- link right_side_cover_link: geometry collision box size=0.0015 0.483 0.289; visual mesh filename=package://carl_description/meshes/side_cover.min.dae scale=0.0254 0.0254 0.0254
- link right_wheel_link: geometry collision cylinder length=0.12 radius=0.25; visual mesh filename=package://carl_description/meshes/wheel.min.dae scale=0.0254 0.0254 0.0254
- link top_plate_link: geometry collision box size=0.325 0.14 0.0066; collision box size=0.325 0.14 0.0066

Commit message: fixed rear struts. also rebuild urdf

File: carl_description/robots/carl.urdf (robot description, URDF)
Before this commit: robot carl, 51 links, 50 joints
Links:
- link front_cover_link: geometry collision box size=0.21 0.068 0.508; collision box size=0.21 0.068 0.508
- link left_rear_strut_link: geometry collision box size=0.04 0.052 1.07; visual mesh filename=package://carl_description/meshes/rear_strut.min.dae scale=0.0254 0.0254 0.0254
- link left_rear_strut_top_link: geometry collision box size=0.04 0.051 0.4572; visual mesh filename=package://carl_description/meshes/rear_strut_top.min.dae scale=0.0254 0.0254 0.0254
- link right_rear_strut_link: geometry collision box size=0.04 0.052 1.07; visual mesh filename=package://carl_description/meshes/rear_strut.min.dae scale=0.0254 0.0254 0.0254
- link right_rear_strut_top_link: geometry collision box size=0.04 0.051 0.4572; visual mesh filename=package://carl_description/meshes/rear_strut_top.min.dae scale=0.0254 0.0254 0.0254

File: carl_description/urdf/components/carl_rear_strut.urdf.xacro (robot description, xacro)
@@ -22,7 +22,7 @@
       </visual>
       <collision>
-        <origin xyz="0.005 0.001 0.525" rpy="0 0 0"/>
+        <origin xyz="0 0.001 0.525" rpy="0 0 0"/>
         <geometry>
-          <box size="0.0355 0.052 1.07 "/>
+          <box size="0.04 0.052 1.07 "/>
         </geometry>
       </collision>
@@ -42,7 +42,7 @@
       </visual>
       <collision>
-        <origin xyz="0.005 0 0.229" rpy="0 0 0" />
+        <origin xyz="-0 0 0.229" rpy="0 0 0" />
         <geometry>
-          <box size="0.0355 0.051 0.4572"/>
+          <box size="0.04 0.051 0.4572"/>
         </geometry>
       </collision>
